File: TrackerAVL/TrackerAVL.sch (KiCad schematic (older format))
At the start: 0 parts

Commit message: Cambios en sch
Changed lines of the file:
@@
 $EndSheet
 $Sheet
-S 2100 5750 800  650
-U 5BA56FF8
-F0 "Fuente" 50
-F1 "fuente.sch" 50
-$EndSheet
-$Sheet
-S 2350 2850 500  150
+S 7600 3550 500  150
 U 5BA57001
 F0 "Acelerómetro" 50
@@
 $EndSheet
 $Sheet
-S 2350 2400 500  150
+S 1400 2100 1500 2400
 U 5BA5703C
 F0 "Conectores_IO" 50
@@
 $EndSheet
 $Sheet
-S 2350 3300 500  150
+S 7600 4000 500  150
 U 5BA7C507
 F0 "ON_BOARD_IO" 50
@@
 Wire Wire Line
 	7600 2750 6300 2750
-Text Notes 700  1350 0    71   ~ 14
+Text Notes 8150 1350 0    71   ~ 14
 Pendientes Equipo AVL\n> Transistor a speaker para pitido tipo buzzer.\n> IRF7105 a PWR_MDM.\n> Ver tema i2c, spi para display consola (mux?).\n> UART_DTR (uc20) a GPIO para manejo sleep mode.\n> Ver tema IO An./Dig.
+$Sheet
+S 1400 1000 1500 600
+U 5BA56FF8
+F0 "Fuente" 50
+F1 "fuente.sch" 50
+F2 "VDD_ADC" O R 2900 1300 50
+$EndSheet
 $EndSCHEMATC

Commit message: Cambios en sch
Changed lines of the file:
@@
 $EndDescr
 $Sheet
-S 4300 1000 2000 5400
+S 4700 1000 2000 5400
 U 5BA56FC1
 F0 "CPU" 50
 F1 "cpu.sch" 50
-F2 "UART_TX" O R 6300 2750 50
-F3 "UART_RX" I R 6300 2650 50
+F2 "UART_TX" O R 6700 2750 50
+F3 "UART_RX" I R 6700 2650 50
 $EndSheet
 $Sheet
-S 7600 3550 500  150
+S 8000 3550 500  150
 U 5BA57001
 F0 "Acelerómetro" 50
@@
 $EndSheet
 $Sheet
-S 1400 2100 1500 2400
+S 1800 2100 1500 4000
 U 5BA5703C
 F0 "Conectores_IO" 50
@@
 $EndSheet
 $Sheet
-S 7600 4700 1500 1100
+S 8000 4700 1500 1100
 U 5BA57067
 F0 "Audio" 50
@@
 $EndSheet
 $Sheet
-S 7600 4000 500  150
+S 8000 4000 500  150
 U 5BA7C507
 F0 "ON_BOARD_IO" 50
@@
 $EndSheet
 $Sheet
-S 7600 2000 1500 1100
+S 8000 2000 1500 1100
 U 5BA5700E
 F0 "UC20_PCIe" 50
 F1 "uc20_pcie.sch" 50
-F2 "WAKE_HOST" O L 7600 2150 50
-F3 "PWR_MDM" I L 7600 2950 50
-F4 "UART_TX" O L 7600 2650 50
-F5 "UART_RX" I L 7600 2750 50
-F6 "UART_DTR" I L 7600 2250 50
-F7 "PCM_SYNC" O R 9100 2950 50
-F8 "PCM_IN" I R 9100 2850 50
-F9 "PCM_OUT" O R 9100 2750 50
-F10 "PCM_CLK" O R 9100 2650 50
-F11 "W_DISABLE" I L 7600 2350 50
-F12 "PERST" I L 7600 2450 50
-F13 "I2C_SCL" O R 9100 2550 50
-F14 "I2C_SDA" B R 9100 2450 50
+F2 "WAKE_HOST" O L 8000 2150 50
+F3 "PWR_MDM" I L 8000 2950 50
+F4 "UART_TX" O L 8000 2650 50
+F5 "UART_RX" I L 8000 2750 50
+F6 "UART_DTR" I L 8000 2250 50
+F7 "PCM_SYNC" O R 9500 2950 50
+F8 "PCM_IN" I R 9500 2850 50
+F9 "PCM_OUT" O R 9500 2750 50
+F10 "PCM_CLK" O R 9500 2650 50
+F11 "W_DISABLE" I L 8000 2350 50
+F12 "PERST" I L 8000 2450 50
+F13 "I2C_SCL" O R 9500 2550 50
+F14 "I2C_SDA" B R 9500 2450 50
 $EndSheet
 Wire Wire Line
-	6300 2650 7600 2650
+	6700 2650 8000 2650
 Wire Wire Line
-	7600 2750 6300 2750
-Text Notes 8150 1350 0    71   ~ 14
+	8000 2750 6700 2750
+Text Notes 8100 1350 0    71   ~ 14
 Pendientes Equipo AVL\n> Transistor a speaker para pitido tipo buzzer.\n> IRF7105 a PWR_MDM.\n> Ver tema i2c, spi para display consola (mux?).\n> UART_DTR (uc20) a GPIO para manejo sleep mode.\n> Ver tema IO An./Dig.
 $Sheet
-S 1400 1000 1500 600
+S 1800 1000 1500 600
 U 5BA56FF8
 F0 "Fuente" 50
 F1 "fuente.sch" 50
-F2 "VDD_ADC" O R 2900 1300 50
+F2 "VBAT" I R 3300 1300 50
 $EndSheet
 $EndSCHEMATC

Commit message: Cambios en sch
Parts:
- added H101, H102, H103, H104: MountingHole, MountingHole:MountingHole_3.2mm_M3, symbol Mechanical:MountingHole
Changed lines of the file:
@@
 F2 "VBAT" I R 3300 1300 50
 $EndSheet
+$Comp
+L Mechanical:MountingHole H101
+U 1 1 5BAF3FC6
+P 2000 6900
+F 0 "H101" H 2100 6946 50  0000 L CNN
+F 1 "MountingHole" H 2100 6855 50  0000 L CNN
+F 2 "MountingHole:MountingHole_3.2mm_M3" H 2000 6900 50  0001 C CNN
+F 3 "~" H 2000 6900 50  0001 C CNN
+	1    2000 6900
+	1    0    0    -1
+$EndComp
+$Comp
+L Mechanical:MountingHole H103
+U 1 1 5BAF4006
+P 2800 6900
+F 0 "H103" H 2900 6946 50  0000 L CNN
+F 1 "MountingHole" H 2900 6855 50  0000 L CNN
+F 2 "MountingHole:MountingHole_3.2mm_M3" H 2800 6900 50  0001 C CNN
+F 3 "~" H 2800 6900 50  0001 C CNN
+	1    2800 6900
+	1    0    0    -1
+$EndComp
+$Comp
+L Mechanical:MountingHole H102
+U 1 1 5BAF4050
+P 2000 7200
+F 0 "H102" H 2100 7246 50  0000 L CNN
+F 1 "MountingHole" H 2100 7155 50  0000 L CNN
+F 2 "MountingHole:MountingHole_3.2mm_M3" H 2000 7200 50  0001 C CNN
+F 3 "~" H 2000 7200 50  0001 C CNN
+	1    2000 7200
+	1    0    0    -1
+$EndComp
+$Comp
+L Mechanical:MountingHole H104
+U 1 1 5BAF40B1
+P 2800 7200
+F 0 "H104" H 2900 7246 50  0000 L CNN
+F 1 "MountingHole" H 2900 7155 50  0000 L CNN
+F 2 "MountingHole:MountingHole_3.2mm_M3" H 2800 7200 50  0001 C CNN
+F 3 "~" H 2800 7200 50  0001 C CNN
+	1    2800 7200
+	1    0    0    -1
+$EndComp
 $EndSCHEMATC

Commit message: Cambios en sch y adición de documentación
Parts:
- added F101, F102, F103, F104, F105, F106: Fiducial, Fiducial:Fiducial_1mm_Dia_2mm_Outer, symbol Mechanical:MountingHole
Changed lines of the file:
@@
 Wire Wire Line
 	8000 2750 6700 2750
-Text Notes 8100 1350 0    71   ~ 14
+Text Notes 7800 1450 0    79   ~ 16
 Pendientes Equipo AVL\n> Transistor a speaker para pitido tipo buzzer.\n> IRF7105 a PWR_MDM.\n> Ver tema i2c, spi para display consola (mux?).\n> UART_DTR (uc20) a GPIO para manejo sleep mode.\n> Ver tema IO An./Dig.
 $Sheet
@@
 	1    0    0    -1
 $EndComp
+$Comp
+L Mechanical:MountingHole F101
+U 1 1 5BBA90D0
+P 3800 6900
+F 0 "F101" H 3900 6946 50  0000 L CNN
+F 1 "Fiducial" H 3900 6855 50  0000 L CNN
+F 2 "Fiducial:Fiducial_1mm_Dia_2mm_Outer" H 3800 6900 50  0001 C CNN
+F 3 "~" H 3800 6900 50  0001 C CNN
+	1    3800 6900
+	1    0    0    -1
+$EndComp
+$Comp
+L Mechanical:MountingHole F104
+U 1 1 5BBA95C7
+P 3800 7200
+F 0 "F104" H 3900 7246 50  0000 L CNN
+F 1 "Fiducial" H 3900 7155 50  0000 L CNN
+F 2 "Fiducial:Fiducial_1mm_Dia_2mm_Outer" H 3800 7200 50  0001 C CNN
+F 3 "~" H 3800 7200 50  0001 C CNN
+	1    3800 7200
+	1    0    0    -1
+$EndComp
+$Comp
+L Mechanical:MountingHole F102
+U 1 1 5BBA95EF
+P 4300 6900
+F 0 "F102" H 4400 6946 50  0000 L CNN
+F 1 "Fiducial" H 4400 6855 50  0000 L CNN
+F 2 "Fiducial:Fiducial_1mm_Dia_2mm_Outer" H 4300 6900 50  0001 C CNN
+F 3 "~" H 4300 6900 50  0001 C CNN
+	1    4300 6900
+	1    0    0    -1
+$EndComp
+$Comp
+L Mechanical:MountingHole F103
+U 1 1 5BBA9625
+P 4800 6900
+F 0 "F103" H 4900 6946 50  0000 L CNN
+F 1 "Fiducial" H 4900 6855 50  0000 L CNN
+F 2 "Fiducial:Fiducial_1mm_Dia_2mm_Outer" H 4800 6900 50  0001 C CNN
+F 3 "~" H 4800 6900 50  0001 C CNN
+	1    4800 6900
+	1    0    0    -1
+$EndComp
+$Comp
+L Mechanical:MountingHole F105
+U 1 1 5BBA9655
+P 4300 7200
+F 0 "F105" H 4400 7246 50  0000 L CNN
+F 1 "Fiducial" H 4400 7155 50  0000 L CNN
+F 2 "Fiducial:Fiducial_1mm_Dia_2mm_Outer" H 4300 7200 50  0001 C CNN
+F 3 "~" H 4300 7200 50  0001 C CNN
+	1    4300 7200
+	1    0    0    -1
+$EndComp
+$Comp
+L Mechanical:MountingHole F106
+U 1 1 5BBA967F
+P 4800 7200
+F 0 "F106" H 4900 7246 50  0000 L CNN
+F 1 "Fiducial" H 4900 7155 50  0000 L CNN
+F 2 "Fiducial:Fiducial_1mm_Dia_2mm_Outer" H 4800 7200 50  0001 C CNN
+F 3 "~" H 4800 7200 50  0001 C CNN
+	1    4800 7200
+	1    0    0    -1
+$EndComp

Commit message: Cambios en sch
Connections:
- net labels added: IGN, MIC+, MIC-, SPK+, SPK-, VBAT
- wire segments 2 -> 14
Other:
- note added: "Pendientes Equipo AVL\n> Transistor a speaker para pitido tipo buzzer.\n> IRF7105 a PWR_MDM.\n> Ver tema i2c, spi para display consola (mux?).\n> UART_DTR (uc20) a GPIO para manejo sleep mode.\n> Ver tema IO An./Dig. \n> 0.8mm de Margen y de Ancho de pista. Menor margen: 0.5mm.\n> Ej: MAYER tiene un margen mínimo de 0.3mm, pero no conviene usarlo."
- note added: "SHEET VALIDADA OK"
- note removed: "Pendientes Equipo AVL\n> Transistor a speaker para pitido tipo buzzer.\n> IRF7105 a PWR_MDM.\n> Ver tema i2c, spi para display consola (mux?).\n> UART_DTR (uc20) a GPIO para manejo sleep mode.\n> Ver tema IO An./Dig."
Changed lines of the file:
@@
 $EndDescr
 $Sheet
-S 4700 1000 2000 5400
+S 3700 1000 2000 5400
 U 5BA56FC1
 F0 "CPU" 50
 F1 "cpu.sch" 50
-F2 "UART_TX" O R 6700 2750 50
-F3 "UART_RX" I R 6700 2650 50
-$EndSheet
-$Sheet
-S 8000 3550 500  150
+F2 "UART_TX" O R 5700 2750 50
+F3 "UART_RX" I R 5700 2650 50
+$EndSheet
+$Sheet
+S 6625 950  500  150
 U 5BA57001
 F0 "Acelerómetro" 50
@@
 $EndSheet
 $Sheet
-S 1800 2100 1500 4000
+S 1300 2100 1500 4000
 U 5BA5703C
 F0 "Conectores_IO" 50
@@
 $EndSheet
 $Sheet
-S 8000 4700 1500 1100
+S 9000 1975 1500 1425
 U 5BA57067
 F0 "Audio" 50
 F1 "audio.sch" 50
-$EndSheet
-$Sheet
-S 8000 4000 500  150
+F2 "ADCOUT" O L 9000 2450 50
+F3 "DACIN" I L 9000 2550 50
+F4 "SCLK" I L 9000 2250 50
+F5 "SDIN" B L 9000 2150 50
+F6 "SPK+" O L 9000 2950 50
+F7 "SPK-" O L 9000 3050 50
+F8 "MIC+" I L 9000 3150 50
+F9 "MIC-" I L 9000 3250 50
+F10 "BCLK-MCLK" I L 9000 2750 50
+F11 "FS" I L 9000 2650 50
+$EndSheet
+$Sheet
+S 6625 1350 500  150
 U 5BA7C507
 F0 "ON_BOARD_IO" 50
@@
 $EndSheet
 $Sheet
-S 8000 2000 1500 1100
+S 6600 2000 1500 1100
 U 5BA5700E
 F0 "UC20_PCIe" 50
 F1 "uc20_pcie.sch" 50
-F2 "WAKE_HOST" O L 8000 2150 50
-F3 "PWR_MDM" I L 8000 2950 50
-F4 "UART_TX" O L 8000 2650 50
-F5 "UART_RX" I L 8000 2750 50
-F6 "UART_DTR" I L 8000 2250 50
-F7 "PCM_SYNC" O R 9500 2950 50
-F8 "PCM_IN" I R 9500 2850 50
-F9 "PCM_OUT" O R 9500 2750 50
-F10 "PCM_CLK" O R 9500 2650 50
-F11 "W_DISABLE" I L 8000 2350 50
-F12 "PERST" I L 8000 2450 50
-F13 "I2C_SCL" O R 9500 2550 50
-F14 "I2C_SDA" B R 9500 2450 50
-$EndSheet
-Wire Wire Line
-	6700 2650 8000 2650
-Wire Wire Line
-	8000 2750 6700 2750
-Text Notes 7800 1450 0    79   ~ 16
-Pendientes Equipo AVL\n> Transistor a speaker para pitido tipo buzzer.\n> IRF7105 a PWR_MDM.\n> Ver tema i2c, spi para display consola (mux?).\n> UART_DTR (uc20) a GPIO para manejo sleep mode.\n> Ver tema IO An./Dig.
-$Sheet
-S 1800 1000 1500 600
+F2 "WAKE_HOST" O L 6600 2150 50
+F3 "PWR_MDM" I L 6600 2950 50
+F4 "UART_TX" O L 6600 2650 50
+F5 "UART_RX" I L 6600 2750 50
+F6 "UART_DTR" I L 6600 2250 50
+F7 "PCM_SYNC" O R 8100 2650 50
+F8 "PCM_IN" I R 8100 2450 50
+F9 "PCM_OUT" O R 8100 2550 50
+F10 "PCM_CLK" O R 8100 2750 50
+F11 "W_DISABLE" I L 6600 2350 50
+F12 "PERST" I L 6600 2450 50
+F13 "I2C_SCL" O R 8100 2250 50
+F14 "I2C_SDA" B R 8100 2150 50
+$EndSheet
+Text Notes 6500 4750 0    79   ~ 16
+Pendientes Equipo AVL\n> Transistor a speaker para pitido tipo buzzer.\n> IRF7105 a PWR_MDM.\n> Ver tema i2c, spi para display consola (mux?).\n> UART_DTR (uc20) a GPIO para manejo sleep mode.\n> Ver tema IO An./Dig. \n> 0.8mm de Margen y de Ancho de pista. Menor margen: 0.5mm.\n> Ej: MAYER tiene un margen mínimo de 0.3mm, pero no conviene usarlo.
+$Sheet
+S 1300 1000 1500 600
 U 5BA56FF8
 F0 "Fuente" 50
 F1 "fuente.sch" 50
-F2 "VBAT" I R 3300 1300 50
+F2 "VBAT" I R 2800 1250 50
+F3 "IGN" I R 2800 1350 50
 $EndSheet
 $Comp
@@
 	1    0    0    -1
 $EndComp
+Wire Wire Line
+	6600 2650 5700 2650
+Wire Wire Line
+	6600 2750 5700 2750
+Wire Wire Line
+	8100 2150 9000 2150
+Wire Wire Line
+	9000 2250 8100 2250
+Wire Wire Line
+	9000 2450 8100 2450
+Wire Wire Line
+	9000 2550 8100 2550
+Wire Wire Line
+	9000 2650 8100 2650
+Wire Wire Line
+	9000 2750 8100 2750
+Text Label 8650 2950 0    50   ~ 0
+SPK+
+Text Label 8650 3050 0    50   ~ 0
+SPK-
+Text Label 8650 3150 0    50   ~ 0
+MIC+
+Text Label 8650 3250 0    50   ~ 0
+MIC-
+Text Notes 9000 1850 0    79   ~ 16
+SHEET VALIDADA OK
+Text Notes 1300 900  0    79   ~ 16
+SHEET VALIDADA OK
+Wire Wire Line
+	9000 2950 8650 2950
+Wire Wire Line
+	8650 3050 9000 3050
+Wire Wire Line
+	9000 3150 8650 3150
+Wire Wire Line
+	8650 3250 9000 3250
+Wire Wire Line
+	2800 1250 3150 1250
+Wire Wire Line
+	2800 1350 3150 1350
+Text Label 3150 1250 2    50   ~ 0
+VBAT
+Text Label 3150 1350 2    50   ~ 0
+IGN
 $EndSCHEMATC

Commit message: Cambios en sch
Connections:
- wire segments 14 -> 40
Changed lines of the file:
@@
 $Descr A4 11693 8268
 encoding utf-8
-Sheet 1 8
+Sheet 1 7
 Title ""
 Date ""
@@
 F2 "UART_TX" O R 5700 2750 50
 F3 "UART_RX" I R 5700 2650 50
+F4 "TEC_0" I L 3700 3900 50
+F5 "TEC_1" I L 3700 4000 50
+F6 "TEC_2" I L 3700 4100 50
+F7 "SPI_MISO" I R 5700 3900 50
+F8 "SPI_MOSI" O R 5700 4000 50
+F9 "TEC_3" I L 3700 4200 50
+F10 "I2C_SCL" O L 3700 5400 50
+F11 "I2C_SCA" B L 3700 5500 50
+F12 "DIG_OUT_1" O L 3700 2400 50
+F13 "DIG_OUT_2" O L 3700 2500 50
+F14 "DIG_OUT_0" O L 3700 2300 50
+F15 "AN_IN_0" I L 3700 2700 50
+F16 "AN_IN_1" I L 3700 2800 50
+F17 "AN_IN_2" I L 3700 2900 50
+F18 "DIG_IN_1" I L 3700 3200 50
+F19 "DIG_IN_2" I L 3700 3300 50
+F20 "DIG_IN_0" I L 3700 3100 50
+F21 "GPIO8" B L 3700 4900 50
 $EndSheet
 $Sheet
@@
 F0 "Acelerómetro" 50
 F1 "acelerometro.sch" 50
-$EndSheet
-$Sheet
-S 1300 2100 1500 4000
-U 5BA5703C
-F0 "Conectores_IO" 50
-F1 "conectores_io.sch" 50
 $EndSheet
 $Sheet
@@
 F10 "BCLK-MCLK" I L 9000 2750 50
 F11 "FS" I L 9000 2650 50
-$EndSheet
-$Sheet
-S 6625 1350 500  150
-U 5BA7C507
-F0 "ON_BOARD_IO" 50
-F1 "ON_BOARD_IO.sch" 50
 $EndSheet
 $Sheet
@@
 Text Label 3150 1350 2    50   ~ 0
 IGN
+Text Notes 1300 2000 0    79   ~ 16
+SHEET VALIDADA OK
+$Sheet
+S 1300 2100 1500 3800
+U 5BA5703C
+F0 "Conectores_IO" 50
+F1 "conectores_io.sch" 50
+F2 "AN_IN_1" O R 2800 2800 50
+F3 "AN_IN_2" O R 2800 2900 50
+F4 "DIG_IN_1" O R 2800 3200 50
+F5 "DIG_IN_2" O R 2800 3300 50
+F6 "VBAT" O R 2800 3500 50
+F7 "IGN" O R 2800 3600 50
+F8 "TEC_1" O R 2800 4000 50
+F9 "TEC_2" O R 2800 4100 50
+F10 "TEC_3" O R 2800 4200 50
+F11 "SPK+" I R 2800 4400 50
+F12 "SPK-" I R 2800 4500 50
+F13 "MIC-" O R 2800 4700 50
+F14 "MIC+" O R 2800 4600 50
+F15 "IBUTTON" B R 2800 4900 50
+F16 "DIG_OUT_1" I R 2800 2400 50
+F17 "DIG_OUT_2" I R 2800 2500 50
+F18 "PROG_TX" I R 2800 5100 50
+F19 "PROG_RX" O R 2800 5200 50
+F20 "DISP_1" B R 2800 5500 50
+F21 "DISP_2" B R 2800 5600 50
+F22 "DISP_3" B R 2800 5700 50
+F23 "DIG_OUT_0" I R 2800 2300 50
+F24 "AN_IN_0" O R 2800 2700 50
+F25 "DIG_IN_0" O R 2800 3100 50
+F26 "TEC_0" O R 2800 3900 50
+F27 "DISP_0" B R 2800 5400 50
+$EndSheet
+Wire Wire Line
+	2800 3500 3150 3500
+Wire Wire Line
+	2800 3600 3150 3600
+Text Label 3150 3500 2    50   ~ 0
+VBAT
+Text Label 3150 3600 2    50   ~ 0
+IGN
+Wire Wire Line
+	2800 4400 3150 4400
+Wire Wire Line
+	2800 4500 3150 4500
+Wire Wire Line
+	2800 4600 3150 4600
+Wire Wire Line
+	2800 5100 3150 5100
+Wire Wire Line
+	2800 5200 3150 5200
+Wire Wire Line
+	2800 5600 3150 5600
+Wire Wire Line
+	2800 4700 3150 4700
+Wire Wire Line
+	2800 5700 3150 5700
+Text Label 3150 4400 2    50   ~ 0
+SPK+
+Text Label 3150 4500 2    50   ~ 0
+SPK-
+Text Label 3150 4600 2    50   ~ 0
+MIC+
+Text Label 3150 4700 2    50   ~ 0
+MIC-
+Wire Wire Line
+	2800 3900 3700 3900
+Wire Wire Line
+	2800 4000 3700 4000
+Wire Wire Line
+	2800 4100 3700 4100
+Wire Wire Line
+	2800 4200 3700 4200
+Wire Wire Line
+	2800 2300 3700 2300
+Wire Wire Line
+	2800 2400 3700 2400
+Wire Wire Line
+	2800 2500 3700 2500
+Wire Wire Line
+	2800 2700 3700 2700
+Wire Wire Line
+	2800 2800 3700 2800
+Wire Wire Line
+	2800 2900 3700 2900
+Wire Wire Line
+	2800 3100 3700 3100
+Wire Wire Line
+	2800 3200 3700 3200
+Wire Wire Line
+	2800 3300 3700 3300
+Wire Wire Line
+	2800 5400 3700 5400
+Wire Wire Line
+	2800 5500 3700 5500
+Wire Wire Line
+	2800 4900 3700 4900
 $EndSCHEMATC

Commit message: Cambios en sch
Other:
- note added: "Cuidado que no entre en\nconflicto con display I2C"
- note added: "Pendientes Equipo AVL\n> Transistor a speaker para pitido tipo buzzer.\n> IRF7105 a PWR_MDM.\n> Ver tema i2c, spi para display consola (mux?).\n> UART_DTR (uc20) a GPIO para manejo sleep mode. \n> 0.8mm de Margen y de Ancho de pista. Menor margen: 0.5mm.\n> Ej: MAYER tiene un margen mínimo de 0.3mm, pero no conviene usarlo."
- note removed: "Pendientes Equipo AVL\n> Transistor a speaker para pitido tipo buzzer.\n> IRF7105 a PWR_MDM.\n> Ver tema i2c, spi para display consola (mux?).\n> UART_DTR (uc20) a GPIO para manejo sleep mode.\n> Ver tema IO An./Dig. \n> 0.8mm de Margen y de Ancho de pista. Menor margen: 0.5mm.\n> Ej: MAYER tiene un margen mínimo de 0.3mm, pero no conviene usarlo."
Changed lines of the file:
@@
 F0 "CPU" 50
 F1 "cpu.sch" 50
-F2 "UART_TX" O R 5700 2750 50
-F3 "UART_RX" I R 5700 2650 50
-F4 "TEC_0" I L 3700 3900 50
-F5 "TEC_1" I L 3700 4000 50
-F6 "TEC_2" I L 3700 4100 50
-F7 "SPI_MISO" I R 5700 3900 50
-F8 "SPI_MOSI" O R 5700 4000 50
-F9 "TEC_3" I L 3700 4200 50
-F10 "I2C_SCL" O L 3700 5400 50
-F11 "I2C_SCA" B L 3700 5500 50
-F12 "DIG_OUT_1" O L 3700 2400 50
-F13 "DIG_OUT_2" O L 3700 2500 50
-F14 "DIG_OUT_0" O L 3700 2300 50
-F15 "AN_IN_0" I L 3700 2700 50
-F16 "AN_IN_1" I L 3700 2800 50
-F17 "AN_IN_2" I L 3700 2900 50
-F18 "DIG_IN_1" I L 3700 3200 50
-F19 "DIG_IN_2" I L 3700 3300 50
-F20 "DIG_IN_0" I L 3700 3100 50
-F21 "GPIO8" B L 3700 4900 50
-$EndSheet
-$Sheet
-S 6625 950  500  150
+F2 "TEC_0" I L 3700 3900 50
+F3 "TEC_1" I L 3700 4000 50
+F4 "TEC_2" I L 3700 4100 50
+F5 "SPI_MISO" I L 3700 5800 50
+F6 "SPI_MOSI" O L 3700 5900 50
+F7 "TEC_3" I L 3700 4200 50
+F8 "I2C_SCL" O L 3700 5400 50
+F9 "I2C_SCA" B L 3700 5500 50
+F10 "DIG_OUT_1" O L 3700 2400 50
+F11 "DIG_OUT_2" O L 3700 2500 50
+F12 "DIG_OUT_0" O L 3700 2300 50
+F13 "AN_IN_0" I L 3700 2700 50
+F14 "AN_IN_1" I L 3700 2800 50
+F15 "AN_IN_2" I L 3700 2900 50
+F16 "DIG_IN_1" I L 3700 3200 50
+F17 "DIG_IN_2" I L 3700 3300 50
+F18 "DIG_IN_0" I L 3700 3100 50
+F19 "IBUTTON" B L 3700 4900 50
+F20 "IGN" I L 3700 3600 50
+F21 "VBAT" I L 3700 3500 50
+F22 "U3_TX" O R 5700 2750 50
+F23 "U3_RX" I R 5700 2650 50
+F24 "RS232_TXD" O L 3700 5100 50
+F25 "RS232_RXD" I L 3700 5200 50
+F26 "SPI_SCK" O L 3700 6000 50
+$EndSheet
+$Sheet
+S 6600 3850 1500 850
 U 5BA57001
 F0 "Acelerómetro" 50
 F1 "acelerometro.sch" 50
+F2 "I2C_SCL" I L 6600 4100 50
+F3 "I2C_SDA" B L 6600 4200 50
+F4 "INT" O L 6600 4400 50
 $EndSheet
 $Sheet
@@
 F14 "I2C_SDA" B R 8100 2150 50
 $EndSheet
-Text Notes 6500 4750 0    79   ~ 16
-Pendientes Equipo AVL\n> Transistor a speaker para pitido tipo buzzer.\n> IRF7105 a PWR_MDM.\n> Ver tema i2c, spi para display consola (mux?).\n> UART_DTR (uc20) a GPIO para manejo sleep mode.\n> Ver tema IO An./Dig. \n> 0.8mm de Margen y de Ancho de pista. Menor margen: 0.5mm.\n> Ej: MAYER tiene un margen mínimo de 0.3mm, pero no conviene usarlo.
+Text Notes 6300 6150 0    79   ~ 16
+Pendientes Equipo AVL\n> Transistor a speaker para pitido tipo buzzer.\n> IRF7105 a PWR_MDM.\n> Ver tema i2c, spi para display consola (mux?).\n> UART_DTR (uc20) a GPIO para manejo sleep mode. \n> 0.8mm de Margen y de Ancho de pista. Menor margen: 0.5mm.\n> Ej: MAYER tiene un margen mínimo de 0.3mm, pero no conviene usarlo.
 $Sheet
 S 1300 1000 1500 600
@@
 F27 "DISP_0" B R 2800 5400 50
 $EndSheet
-Wire Wire Line
-	2800 3500 3150 3500
-Wire Wire Line
-	2800 3600 3150 3600
 Text Label 3150 3500 2    50   ~ 0
 VBAT
@@
 Wire Wire Line
 	2800 4600 3150 4600
-Wire Wire Line
-	2800 5100 3150 5100
-Wire Wire Line
-	2800 5200 3150 5200
 Wire Wire Line
 	2800 5600 3150 5600
@@
 Wire Wire Line
 	2800 4900 3700 4900
+Wire Wire Line
+	2800 5100 3700 5100
+Wire Wire Line
+	2800 5200 3700 5200
+Wire Wire Line
+	2800 3500 3700 3500
+Wire Wire Line
+	2800 3600 3700 3600
+Text Notes 7000 4250 0    79   ~ 16
+Cuidado que no entre en\nconflicto con display I2C
+Text Notes 6600 3750 0    79   ~ 16
+SHEET VALIDADA OK
 $EndSCHEMATC

Commit message: Cambios en sch
Connections:
- net labels added: AN_IN_0, AN_IN_1, AN_IN_2, DIG_IN_0, DIG_IN_1, DIG_IN_2, DIG_OUT_0, DIG_OUT_1, DIG_OUT_2, I2C_SCL, I2C_SDA
- wire segments 40 -> 68
Other:
- note added: "FALTA PONER BUFFER!!!!!!!!"
- note added: "Pendientes Equipo AVL\n> Transistor a speaker para pitido tipo buzzer.\n> Ver tema i2c, spi para display consola (mux?).\n> 0.8mm de Margen y de Ancho de pista. Menor margen: 0.5mm.\n> Ej: MAYER tiene un margen mínimo de 0.3mm, pero no conviene usarlo.\n> Tema conectores SMA!, encargué los que van en PCB... sirven??? mmm.."
- note removed: "Cuidado que no entre en\nconflicto con display I2C"
- note removed: "Pendientes Equipo AVL\n> Transistor a speaker para pitido tipo buzzer.\n> IRF7105 a PWR_MDM.\n> Ver tema i2c, spi para display consola (mux?).\n> UART_DTR (uc20) a GPIO para manejo sleep mode. \n> 0.8mm de Margen y de Ancho de pista. Menor margen: 0.5mm.\n> Ej: MAYER tiene un margen mínimo de 0.3mm, pero no conviene usarlo."
