File: TrackerAVL/TrackerAVL.sch (KiCad schematic (older format))
At the start: 10 parts

Commit message: Cambios en sch
Parts:
- added TP?: TestPoint, MountingHole:MountingHole_3.2mm_M3_Pad, symbol Connector:TestPoint
- renumbered F104 to F102, F102 to F103, F105 to F104, F103 to F105
Connections:
- net labels added: GND, TEC_0, TEC_1, TEC_2, TEC_3
- wire segments 68 -> 78
Other:
- note added: "Agujeros de montaje"
- note added: "Fiduciales (3 por capa)"
- note added: "Pendientes Equipo AVL\n> Transistor a speaker para pitido tipo buzzer.\n> Ver tema i2c, spi para display consola (mux?).\n> Asociar huellas"
- note added: "Referencias:\nNM: NOT MOUNTED in PCB"
- note added: "TestPoints"
- note added: "Ver tema buzzer \ny buses I2C/SPI"
- note removed: "FALTA PONER BUFFER!!!!!!!!"
- note removed: "Pendientes Equipo AVL\n> Transistor a speaker para pitido tipo buzzer.\n> Ver tema i2c, spi para display consola (mux?).\n> 0.8mm de Margen y de Ancho de pista. Menor margen: 0.5mm.\n> Ej: MAYER tiene un margen mínimo de 0.3mm, pero no conviene usarlo.\n> Tema conectores SMA!, encargué los que van en PCB... sirven??? mmm.."
- moved on the sheet: F101, F102, F103, F104, F105, F106, H101, H102, H103, H104

Commit message: Cambios en sch
Parts:
- gave numbers to parts that had none: 1
Connections:
- net labels added: SPI_MOSI, SPI_SCK
- wire segments 78 -> 81
Other:
- note added: "Pendientes Equipo AVL\n> Asociar huellas"
- note removed: "Pendientes Equipo AVL\n> Transistor a speaker para pitido tipo buzzer.\n> Ver tema i2c, spi para display consola (mux?).\n> Asociar huellas"
- note removed: "Ver tema buzzer \ny buses I2C/SPI"
Changed lines of the file:
@@
 F30 "SPI_CS1" O L 3500 5700 50
 F31 "BUFFER_OE" O R 5500 6200 50
+F32 "DISPLAY_MODE" O L 3500 5800 50
+F33 "BUZZER" O L 3500 6000 50
 $EndSheet
 $Sheet
@@
 $EndSheet
 Text Notes 8750 4100 0    118  ~ 24
-Pendientes Equipo AVL\n> Transistor a speaker para pitido tipo buzzer.\n> Ver tema i2c, spi para display consola (mux?).\n> Asociar huellas
+Pendientes Equipo AVL\n> Asociar huellas
 $Sheet
 S 1100 900  1500 600
@@
 Text Notes 6400 3800 0    79   ~ 16
 SHEET VALIDADA OK
-Text Label 3050 5300 2    50   ~ 0
+Text Label 2850 5300 0    50   ~ 0
 I2C_SCL
-Text Label 3050 5400 2    50   ~ 0
+Text Label 2850 5400 0    50   ~ 0
 I2C_SDA
 Wire Wire Line
@@
 Wire Wire Line
 	6400 3050 5500 3050
-Text Notes 9050 6400 0    98   ~ 20
+Text Notes 8950 6400 0    98   ~ 20
 Referencias:\nNM: NOT MOUNTED in PCB
 Text Label 3050 3800 2    50   ~ 0
@@
 F18 "PROG_TX" I R 2600 5000 50
 F19 "PROG_RX" O R 2600 5100 50
-F20 "DISP_1" B R 2600 5400 50
-F21 "DISP_2" B R 2600 5500 50
-F22 "DISP_3" B R 2600 5600 50
-F23 "DIG_OUT_0" I R 2600 2200 50
-F24 "AN_IN_0" O R 2600 2600 50
-F25 "DIG_IN_0" O R 2600 3000 50
-F26 "TEC_0" O R 2600 3800 50
-F27 "DISP_0" B R 2600 5300 50
+F20 "DIG_OUT_0" I R 2600 2200 50
+F21 "AN_IN_0" O R 2600 2600 50
+F22 "DIG_IN_0" O R 2600 3000 50
+F23 "TEC_0" O R 2600 3800 50
+F24 "DISP_I2C_SCL" I R 2600 5300 50
+F25 "DISP_I2C_SDA" B R 2600 5400 50
+F26 "DISP_SPI_MOSI" I R 2600 5500 50
+F27 "DISP_SPI_SCK" I R 2600 5600 50
+F28 "DISP_SPI_CS1" I R 2600 5700 50
+F29 "DISPLAY_MODE" I R 2600 5800 50
+F30 "BUZZER" I R 2600 6000 50
 $EndSheet
 Wire Wire Line
@@
 Wire Wire Line
 	6400 6000 5500 6000
-Text Notes 2700 6150 0    118  ~ 24
-Ver tema buzzer \ny buses I2C/SPI
-$Comp
-L Connector:TestPoint TP?
+$Comp
+L Connector:TestPoint TP101
 U 1 1 5BDCE2DE
 P 3800 7000
-F 0 "TP?" H 3858 7074 50  0000 L CNN
+F 0 "TP101" H 3858 7074 50  0000 L CNN
 F 1 "TestPoint" H 3858 7029 50  0001 L CNN
 F 2 "MountingHole:MountingHole_3.2mm_M3_Pad" H 4000 7000 50  0001 C CNN
@@
 Fiduciales (3 por capa)
 $Comp
-L power:GND #PWR?
+L power:GND #PWR0101
 U 1 1 5BDFB84C
 P 3800 7200
-F 0 "#PWR?" H 3800 6950 50  0001 C CNN
+F 0 "#PWR0101" H 3800 6950 50  0001 C CNN
 F 1 "GND" H 3805 7027 50  0000 C CNN
 F 2 "" H 3800 7200 50  0001 C CNN
@@
 Wire Wire Line
 	2600 5600 3500 5600
+Wire Wire Line
+	2600 5700 3500 5700
+Wire Wire Line
+	3500 5800 2600 5800
+Wire Wire Line
+	2600 6000 3500 6000
+Text Label 2850 5500 0    50   ~ 0
+SPI_MOSI
+Text Label 2850 5600 0    50   ~ 0
+SPI_SCK
+Text Notes 6400 750  0    79   ~ 16
+SHEET VALIDADA OK
+Text Notes 3500 750  0    79   ~ 16
+SHEET VALIDADA OK
 $EndSCHEMATC

Commit message: Cambios en pcb
Other:
- note added: "Equipo AVL vRaptor v1.0 https://github.com/MauroMoreyra/EquipoAVL_pcb/"
- note removed: "Pendientes Equipo AVL\n> Asociar huellas"
- note removed: "SHEET VALIDADA OK"
Changed lines of the file:
@@
 Rev "1.0"
 Comp ""
-Comment1 "Ing. Mauro Moreyra"
+Comment1 "Autor: Ing. Mauro Moreyra"
 Comment2 ""
 Comment3 ""
@@
 F11 "FS" I L 8800 1550 50
 $EndSheet
-Text Notes 8750 4100 0    118  ~ 24
-Pendientes Equipo AVL\n> Asociar huellas
+Text Notes 1100 725  0    118  ~ 24
+Equipo AVL vRaptor v1.0 https://github.com/MauroMoreyra/EquipoAVL_pcb/
 $Sheet
 S 1100 900  1500 600
@@
 Text Label 10650 1600 2    50   ~ 0
 MIC-
-Text Notes 8800 750  0    79   ~ 16
-SHEET VALIDADA OK
-Text Notes 1100 800  0    79   ~ 16
-SHEET VALIDADA OK
 Wire Wire Line
 	10300 1300 10650 1300
@@
 Text Label 2950 1250 2    50   ~ 0
 IGN
-Text Notes 1100 1900 0    79   ~ 16
-SHEET VALIDADA OK
 Text Label 3050 3400 2    50   ~ 0
 VBAT
@@
 Wire Wire Line
 	2600 5100 3500 5100
-Text Notes 6400 2400 0    79   ~ 16
-SHEET VALIDADA OK
 $Sheet
 S 6400 900  1500 1100
@@
 Wire Wire Line
 	5500 1250 6400 1250
-Text Notes 6400 3800 0    79   ~ 16
-SHEET VALIDADA OK
 Text Label 2850 5300 0    50   ~ 0
 I2C_SCL
@@
 Wire Wire Line
 	6400 3050 5500 3050
-Text Notes 8950 6400 0    98   ~ 20
+Text Notes 8600 2675 0    118  ~ 24
 Referencias:\nNM: NOT MOUNTED in PCB
 Text Label 3050 3800 2    50   ~ 0
@@
 Text Label 2850 5600 0    50   ~ 0
 SPI_SCK
-Text Notes 6400 750  0    79   ~ 16
-SHEET VALIDADA OK
-Text Notes 3500 750  0    79   ~ 16
-SHEET VALIDADA OK
 $EndSCHEMATC

Commit message: Cambios en pcb y modelos 3d
Parts:
- removed TP101: TestPoint, MountingHole:MountingHole_3.2mm_M3_Pad, symbol Connector:TestPoint
Connections:
- net labels removed: GND
- wire segments 81 -> 80
Other:
- note removed: "TestPoints"
Changed lines of the file:
@@
 Wire Wire Line
 	6400 6000 5500 6000
-$Comp
-L Connector:TestPoint TP101
-U 1 1 5BDCE2DE
-P 3800 7000
-F 0 "TP101" H 3858 7074 50  0000 L CNN
-F 1 "TestPoint" H 3858 7029 50  0001 L CNN
-F 2 "MountingHole:MountingHole_3.2mm_M3_Pad" H 4000 7000 50  0001 C CNN
-F 3 "~" H 4000 7000 50  0001 C CNN
-	1    3800 7000
-	1    0    0    -1
-$EndComp
 Text Notes 1100 6750 0    59   ~ 12
 Agujeros de montaje
 Text Notes 2250 6750 0    59   ~ 12
 Fiduciales (3 por capa)
-$Comp
-L power:GND #PWR0101
-U 1 1 5BDFB84C
-P 3800 7200
-F 0 "#PWR0101" H 3800 6950 50  0001 C CNN
-F 1 "GND" H 3805 7027 50  0000 C CNN
-F 2 "" H 3800 7200 50  0001 C CNN
-F 3 "" H 3800 7200 50  0001 C CNN
-	1    3800 7200
-	1    0    0    -1
-$EndComp
-Wire Wire Line
-	3800 7000 3800 7200
-Text Notes 3750 6750 0    59   ~ 12
-TestPoints
 Wire Wire Line
 	2600 5500 3500 5500

Commit message: Cambios en README, ahora incluye información de versiones
Parts:
- H101, H102, H103, H104: footprint MountingHole:MountingHole_3.2mm_M3 -> MountingHole:MountingHole_3.2mm_M3_Pad_Thin
Changed lines of the file:
@@
 F 0 "H101" H 1300 6946 50  0000 L CNN
 F 1 "MountingHole" H 1300 6855 50  0000 L CNN
-F 2 "MountingHole:MountingHole_3.2mm_M3" H 1200 6900 50  0001 C CNN
+F 2 "MountingHole:MountingHole_3.2mm_M3_Pad_Thin" H 1200 6900 50  0001 C CNN
 F 3 "~" H 1200 6900 50  0001 C CNN
 	1    1200 6900
@@
 F 0 "H103" H 1300 7346 50  0000 L CNN
 F 1 "MountingHole" H 1300 7255 50  0000 L CNN
-F 2 "MountingHole:MountingHole_3.2mm_M3" H 1200 7300 50  0001 C CNN
+F 2 "MountingHole:MountingHole_3.2mm_M3_Pad_Thin" H 1200 7300 50  0001 C CNN
 F 3 "~" H 1200 7300 50  0001 C CNN
 	1    1200 7300
@@
 F 0 "H102" H 1300 7146 50  0000 L CNN
 F 1 "MountingHole" H 1300 7055 50  0000 L CNN
-F 2 "MountingHole:MountingHole_3.2mm_M3" H 1200 7100 50  0001 C CNN
+F 2 "MountingHole:MountingHole_3.2mm_M3_Pad_Thin" H 1200 7100 50  0001 C CNN
 F 3 "~" H 1200 7100 50  0001 C CNN
 	1    1200 7100
@@
 F 0 "H104" H 1300 7546 50  0000 L CNN
 F 1 "MountingHole" H 1300 7455 50  0000 L CNN
-F 2 "MountingHole:MountingHole_3.2mm_M3" H 1200 7500 50  0001 C CNN
+F 2 "MountingHole:MountingHole_3.2mm_M3_Pad_Thin" H 1200 7500 50  0001 C CNN
 F 3 "~" H 1200 7500 50  0001 C CNN
 	1    1200 7500
