File: TrackerAVL/audio.sch (KiCad schematic (older format))
At the start: 1 part

Commit message: Cambios en sch
Parts:
- removed U?: NAU8814, nau8814:NAU8814_QFN-24_4x4mm_Pitch0.5mm_EPAD, symbol nau8814:NAU8814
- added U?: NAU8814, nau8814:NAU8814_QFN-24_4x4mm_Pitch0.5mm_EPAD, symbol nau8814:NAU8814
Changed lines of the file:
@@
 $Comp
 L nau8814:NAU8814 U?
-U 1 1 5BA81B55
+U 1 1 5BA9B2C5
 P 5550 3500
 F 0 "U?" H 6441 3553 60  0000 L CNN

Commit message: Cambios en sch
Parts:
- gave numbers to parts that had none: 1
Changed lines of the file:
@@
 $EndDescr
 $Comp
-L nau8814:NAU8814 U?
+L nau8814:NAU8814 U501
 U 1 1 5BA9B2C5
 P 5550 3500
-F 0 "U?" H 6441 3553 60  0000 L CNN
+F 0 "U501" H 6441 3553 60  0000 L CNN
 F 1 "NAU8814" H 6441 3447 60  0000 L CNN
 F 2 "nau8814:NAU8814_QFN-24_4x4mm_Pitch0.5mm_EPAD" H 5550 3500 60  0001 C CNN

Commit message: Cambios en sch y adición de documentación
Parts:
- added C? (x6): 4.7uF, symbol Device:C
- added C? (x4): 1uF, symbol Device:C
- added R? (x2): 1K2, symbol Device:R
Connections:
- net labels added: ADCOUT, AUX, BCLK, CSb-GPIO, DACIN, FS, GND, MCLK, MIC+, MIC-, MODE, MOUT, SCLK, SDIN, SPKOUT+, SPKOUT-, VDDSPK, VREF
- wire segments 0 -> 69
Other:
- note added: "Referencia: circuito de aplicación (pag. 106 de datasheet NAU8814).\n\n1) Ver si hay que poner capacitores de 0.1uF en paralelo a los de 4.7uF."
- note removed: "Ver página 106 de datasheet NAU8814 (Typical Application)."

Commit message: Cambios en sch y add docs
Parts:
- removed C? (x5): 4.7uF, symbol Device:C
- removed C? (x4): 1uF, symbol Device:C
- removed R? (x2): 1K2, symbol Device:R
- added C? (x5): 0.1uF, symbol Device:C
- added C? (x6): 4.7uF, symbol Device:C
- added C? (x2): 10pF, symbol Device:C
- added C? (x2): 33pF, symbol Device:C
- added C? (x2): 1uF, symbol Device:C
- added C?: 10nF, symbol Device:C
- added C?: 20pF, symbol Device:C
- added R? (x2): 1K2, symbol Device:R
- added R? (x2): 1K, symbol Device:R
- added R?: 0R, symbol Device:R
- added R? (x4): 22R, symbol Device:R
- added R? (x4): 10K, symbol Device:R
Connections:
- net labels added: +1V8, +3.3V, GNDA, MICBIAS, MICN, MICP, SPK+, SPK-, VDDA
- net labels removed: AUX, CSb-GPIO, MCLK, MODE, MOUT, SPKOUT+, SPKOUT-, VDDSPK, VREF
- wire segments 69 -> 139
- no-connect marks 0 -> 2
Other:
- note added: "Bus I2C UC20"
- note added: "Bus PCM UC20"
- note added: "Close to mic connector"
- note added: "Referencias:\nNAU8814 Audio codec.pdf (pag. 106)\nUC20_Reference_Design_20130712"
- note removed: "Referencia: circuito de aplicación (pag. 106 de datasheet NAU8814).\n\n1) Ver si hay que poner capacitores de 0.1uF en paralelo a los de 4.7uF."

Commit message: Cambios en sch
Connections:
- net labels added: BCLK-MCLK
- net labels removed: BCLK
Changed lines of the file:
@@
 Text HLabel 2575 5050 0    50   Input ~ 0
 DACIN
-Text HLabel 2575 5175 0    50   BiDi ~ 0
+Text HLabel 2575 5175 0    50   Input ~ 0
 FS
 Text HLabel 2575 5300 0    50   Input ~ 0
-BCLK
+BCLK-MCLK
 Text HLabel 5450 4075 2    50   Input ~ 0
 SCLK

Commit message: Cambios en sch
Parts:
- gave numbers to parts that had none: 33
Changed lines of the file:
@@
 $Descr A4 11693 8268
 encoding utf-8
-Sheet 5 7
+Sheet 5 8
 Title ""
 Date ""
@@
 $EndComp
 $Comp
-L Device:C C?
+L Device:C C404
 U 1 1 5BC14982
 P 2400 4175
-F 0 "C?" H 2450 4275 50  0000 L CNN
+F 0 "C404" H 2450 4275 50  0000 L CNN
 F 1 "4.7uF" H 2450 4075 50  0000 L CNN
 F 2 "" H 2438 4025 50  0001 C CNN
@@
 	2400 4325 2400 4425
 $Comp
-L Device:C C?
+L Device:C C403
 U 1 1 5BC349CB
 P 2100 4175
-F 0 "C?" H 2150 4275 50  0000 L CNN
+F 0 "C403" H 2150 4275 50  0000 L CNN
 F 1 "0.1uF" H 2150 4075 50  0000 L CNN
 F 2 "" H 2138 4025 50  0001 C CNN
@@
 	2100 4425 2400 4425
 $Comp
-L Device:C C?
+L Device:C C402
 U 1 1 5BC378D2
 P 1800 4175
-F 0 "C?" H 1850 4275 50  0000 L CNN
+F 0 "C402" H 1850 4275 50  0000 L CNN
 F 1 "4.7uF" H 1850 4075 50  0000 L CNN
 F 2 "" H 1838 4025 50  0001 C CNN
@@
 $EndComp
 $Comp
-L Device:C C?
+L Device:C C401
 U 1 1 5BC37914
 P 1500 4175
-F 0 "C?" H 1550 4275 50  0000 L CNN
+F 0 "C401" H 1550 4275 50  0000 L CNN
 F 1 "0.1uF" H 1550 4075 50  0000 L CNN
 F 2 "" H 1538 4025 50  0001 C CNN
@@
 $EndComp
 $Comp
-L Device:C C?
+L Device:C C414
 U 1 1 5BC37956
 P 7375 1975
-F 0 "C?" H 7425 2075 50  0000 L CNN
+F 0 "C414" H 7425 2075 50  0000 L CNN
 F 1 "4.7uF" H 7425 1875 50  0000 L CNN
 F 2 "" H 7413 1825 50  0001 C CNN
@@
 $EndComp
 $Comp
-L Device:C C?
+L Device:C C410
 U 1 1 5BC3799C
 P 7075 1975
-F 0 "C?" H 7125 2075 50  0000 L CNN
+F 0 "C410" H 7125 2075 50  0000 L CNN
 F 1 "0.1uF" H 7125 1875 50  0000 L CNN
 F 2 "" H 7113 1825 50  0001 C CNN
@@
 Connection ~ 1800 3875
 $Comp
-L Device:C C?
+L Device:C C407
 U 1 1 5BC5BE43
 P 4025 2275
-F 0 "C?" V 4075 2175 50  0000 C CNN
+F 0 "C407" V 4075 2175 50  0000 C CNN
 F 1 "4.7uF" V 4075 2425 50  0000 C CNN
 F 2 "" H 4063 2125 50  0001 C CNN
@@
 $EndComp
 $Comp
-L Device:C C?
+L Device:C C406
 U 1 1 5BC5BEA3
 P 4025 2075
-F 0 "C?" V 4075 1975 50  0000 C CNN
+F 0 "C406" V 4075 1975 50  0000 C CNN
 F 1 "0.1uF" V 4075 2225 50  0000 C CNN
 F 2 "" H 4063 1925 50  0001 C CNN
@@
 $EndComp
 $Comp
-L Device:C C?
+L Device:C C411
 U 1 1 5BC8E196
 P 7225 3300
-F 0 "C?" H 7275 3400 50  0000 L CNN
+F 0 "C411" H 7275 3400 50  0000 L CNN
 F 1 "4.7uF" H 7275 3200 50  0000 L CNN
 F 2 "" H 7263 3150 50  0001 C CNN
@@
 $EndComp
 $Comp
-L Device:C C?
+L Device:C C409
 U 1 1 5BC8E1EA
 P 6925 3300
-F 0 "C?" H 6975 3400 50  0000 L CNN
+F 0 "C409" H 6975 3400 50  0000 L CNN
 F 1 "0.1uF" H 6975 3200 50  0000 L CNN
 F 2 "" H 6963 3150 50  0001 C CNN
@@
 	2550 3425 2550 3475
 $Comp
-L Device:C C?
+L Device:C C418
 U 1 1 5BCDC5C8
 P 9625 4950
-F 0 "C?" H 9675 5050 50  0000 L CNN
+F 0 "C418" H 9675 5050 50  0000 L CNN
 F 1 "10pF" H 9675 4850 50  0000 L CNN
 F 2 "" H 9663 4800 50  0001 C CNN
@@
 $EndComp
 $Comp
-L Device:C C?
+L Device:C C419
 U 1 1 5BCDC65A
 P 9925 4950
-F 0 "C?" H 9975 5050 50  0000 L CNN
+F 0 "C419" H 9975 5050 50  0000 L CNN
 F 1 "33pF" H 9975 4850 50  0000 L CNN
 F 2 "" H 9963 4800 50  0001 C CNN
@@
 	9925 4800 9925 4500
 $Comp
-L Device:C C?
+L Device:C C420
 U 1 1 5BCE2157
 P 10325 4950
-F 0 "C?" H 10375 5050 50  0000 L CNN
+F 0 "C420" H 10375 5050 50  0000 L CNN
 F 1 "4.7uF" H 10375 4850 50  0000 L CNN
 F 2 "" H 10363 4800 50  0001 C CNN
@@
 	7225 3550 7225 3650
 $Comp
-L Device:C C?
+L Device:C C412
 U 1 1 5BD112E6
 P 7225 4100
-F 0 "C?" V 7275 4000 50  0000 C CNN
+F 0 "C412" V 7275 4000 50  0000 C CNN
 F 1 "1uF" V 7275 4250 50  0000 C CNN
 F 2 "" H 7263 3950 50  0001 C CNN
@@
 $EndComp
 $Comp
-L Device:C C?
+L Device:C C413
 U 1 1 5BD1165D
 P 7225 4500
-F 0 "C?" V 7275 4400 50  0000 C CNN
+F 0 "C413" V 7275 4400 50  0000 C CNN
 F 1 "1uF" V 7275 4650 50  0000 C CNN
 F 2 "" H 7263 4350 50  0001 C CNN
@@
 $EndComp
 $Comp
-L Device:C C?
+L Device:C C415
 U 1 1 5BD11BF1
 P 8075 4300
-F 0 "C?" H 8175 4200 50  0000 C CNN
+F 0 "C415" H 8175 4200 50  0000 C CNN
 F 1 "10nF" H 8175 4400 50  0000 C CNN
 F 2 "" H 8113 4150 50  0001 C CNN
@@
 	7375 4500 7725 4500
 $Comp
-L Device:R R?
+L Device:R R411
 U 1 1 5BD28920
 P 7725 3900
-F 0 "R?" H 7795 3946 50  0000 L CNN
+F 0 "R411" H 7795 3946 50  0000 L CNN
 F 1 "1K2" H 7795 3855 50  0000 L CNN
 F 2 "" V 7655 3900 50  0001 C CNN
@@
 	7725 4050 7725 4100
 $Comp
-L Device:R R?
+L Device:R R410
 U 1 1 5BD2C760
 P 7725 3475
-F 0 "R?" H 7795 3521 50  0000 L CNN
+F 0 "R410" H 7795 3521 50  0000 L CNN
 F 1 "1K" H 7795 3430 50  0000 L CNN
 F 2 "" V 7655 3475 50  0001 C CNN
@@
 $EndComp
 $Comp
-L Device:R R?
+L Device:R R412
 U 1 1 5BD2C7B4
 P 7725 4700
-F 0 "R?" H 7795 4746 50  0000 L CNN
+F 0 "R412" H 7795 4746 50  0000 L CNN
 F 1 "1K2" H 7795 4655 50  0000 L CNN
 F 2 "" V 7655 4700 50  0001 C CNN
@@
 $EndComp
 $Comp
-L Device:R R?
+L Device:R R413
 U 1 1 5BD2C816
 P 7725 5100
-F 0 "R?" H 7795 5146 50  0000 L CNN
+F 0 "R413" H 7795 5146 50  0000 L CNN
 F 1 "1K" H 7795 5055 50  0000 L CNN
 F 2 "" V 7655 5100 50  0001 C CNN
@@
 	7725 4100 8775 4100
 $Comp
-L Device:C C?
+L Device:C C416
 U 1 1 5BDB5708
 P 8775 4950
-F 0 "C?" H 8825 5050 50  0000 L CNN
+F 0 "C416" H 8825 5050 50  0000 L CNN
 F 1 "10pF" H 8825 4850 50  0000 L CNN
 F 2 "" H 8813 4800 50  0001 C CNN
@@
 $EndComp
 $Comp
-L Device:C C?
+L Device:C C417
 U 1 1 5BDB5798
 P 9075 4950
-F 0 "C?" H 9125 5050 50  0000 L CNN
+F 0 "C417" H 9125 5050 50  0000 L CNN
 F 1 "33pF" H 9125 4850 50  0000 L CNN
 F 2 "" H 9113 4800 50  0001 C CNN
@@
 	8775 4100 9075 4100
 $Comp
-L Device:R R?
+L Device:R R409
 U 1 1 5BDCA93E
 P 6725 1675
-F 0 "R?" V 6825 1550 50  0000 L CNN
+F 0 "R409" V 6825 1550 50  0000 L CNN
 F 1 "0R" V 6825 1725 50  0000 L CNN
 F 2 "" V 6655 1675 50  0001 C CNN
@@
 Connection ~ 2100 3975
 $Comp
-L Device:R R?
+L Device:R R402
 U 1 1 5BE58835
 P 2925 5050
-F 0 "R?" V 2875 5175 50  0000 L CNN
+F 0 "R402" V 2875 5175 50  0000 L CNN
 F 1 "22R" V 2875 4775 50  0000 L CNN
 F 2 "" V 2855 5050 50  0001 C CNN
@@
 $EndComp
 $Comp
-L Device:R R?
+L Device:R R401
 U 1 1 5BE6C53C
 P 2925 4925
-F 0 "R?" V 2875 5050 50  0000 L CNN
+F 0 "R401" V 2875 5050 50  0000 L CNN
 F 1 "22R" V 2875 4650 50  0000 L CNN
 F 2 "" V 2855 4925 50  0001 C CNN
@@
 $EndComp
 $Comp
-L Device:R R?
+L Device:R R403
 U 1 1 5BE8557D
 P 2925 5175
-F 0 "R?" V 2875 5300 50  0000 L CNN
+F 0 "R403" V 2875 5300 50  0000 L CNN
 F 1 "22R" V 2875 4900 50  0000 L CNN
 F 2 "" V 2855 5175 50  0001 C CNN
@@
 $EndComp
 $Comp
-L Device:R R?
+L Device:R R404
 U 1 1 5BE8F89C
 P 2925 5300
-F 0 "R?" V 2875 5425 50  0000 L CNN
+F 0 "R404" V 2875 5425 50  0000 L CNN
 F 1 "22R" V 2875 5025 50  0000 L CNN
 F 2 "" V 2855 5300 50  0001 C CNN
@@
 	3650 4675 3650 5300
 $Comp
-L Device:R R?
+L Device:R R405
 U 1 1 5BEB58EB
 P 3850 4925
-F 0 "R?" H 3920 4971 50  0000 L CNN
+F 0 "R405" H 3920 4971 50  0000 L CNN
 F 1 "10K" H 3920 4880 50  0000 L CNN
 F 2 "" V 3780 4925 50  0001 C CNN
@@
 Connection ~ 3650 5300
 $Comp
-L Device:C C?
+L Device:C C405
 U 1 1 5BEEDB3B
 P 3650 5525
-F 0 "C?" H 3675 5625 50  0000 L CNN
+F 0 "C405" H 3675 5625 50  0000 L CNN
 F 1 "20pF" H 3675 5425 50  0000 L CNN
 F 2 "" H 3688 5375 50  0001 C CNN
@@
 Bus I2C UC20
 $Comp
-L Device:R R?
+L Device:R R408
 U 1 1 5BF2D2AB
 P 5200 3775
-F 0 "R?" H 5270 3821 50  0000 L CNN
+F 0 "R408" H 5270 3821 50  0000 L CNN
 F 1 "10K" H 5270 3730 50  0000 L CNN
 F 2 "" V 5130 3775 50  0001 C CNN
@@
 $EndComp
 $Comp
-L Device:R R?
+L Device:R R407
 U 1 1 5BF2D7DE
 P 4925 3775
-F 0 "R?" H 4995 3821 50  0000 L CNN
+F 0 "R407" H 4995 3821 50  0000 L CNN
 F 1 "10K" H 4995 3730 50  0000 L CNN
 F 2 "" V 4855 3775 50  0001 C CNN
@@
 	4925 4075 5450 4075
 $Comp
-L Device:R R?
+L Device:R R406
 U 1 1 5BF42823
 P 4600 4300
-F 0 "R?" H 4670 4346 50  0000 L CNN
+F 0 "R406" H 4670 4346 50  0000 L CNN
 F 1 "10K" H 4670 4255 50  0000 L CNN
 F 2 "" V 4530 4300 50  0001 C CNN
@@
 	3750 2275 3750 2975
 $Comp
-L Device:C C?
+L Device:C C408
 U 1 1 5BFDDC6A
 P 4025 2475
-F 0 "C?" V 4075 2375 50  0000 C CNN
+F 0 "C408" V 4075 2375 50  0000 C CNN
 F 1 "4.7uF" V 4075 2625 50  0000 C CNN
 F 2 "" H 4063 2325 50  0001 C CNN
