File: TrackerAVL/audio.sch (KiCad schematic (older format))
At the start: 34 parts, among them U401 NAU8814

Commit message: Cambios en pcb
Parts:
- JP401: footprint Jumper:SolderJumper-2_P1.3mm_Bridged_Pad1.0x1.5mm -> NetTie:NetTie-2_SMD_Pad0.5mm
Changed lines of the file:
@@
 F 0 "JP401" H 5600 5864 50  0000 C CNN
 F 1 "Jumper" H 5600 5773 50  0000 C CNN
-F 2 "Jumper:SolderJumper-2_P1.3mm_Bridged_Pad1.0x1.5mm" H 5600 5600 50  0001 C CNN
+F 2 "NetTie:NetTie-2_SMD_Pad0.5mm" H 5600 5600 50  0001 C CNN
 F 3 "~" H 5600 5600 50  0001 C CNN
 	1    5600 5600
