File: TrackerAVL/fuente.sch (KiCad schematic (older format))
At the start: 0 parts

Commit message: Cambios en sch
Parts:
- added C? (x2): 10uF, Libreria_EDU_CIAA_NXP:c_1206_tantalio, symbol Device:CP
- added C?: 100nF, Libreria_EDU_CIAA_NXP:c_0805, symbol Device:C
- added D?: SMAZ5V6, Libreria_EDU_CIAA_NXP:SOD123F, symbol TrackerAVL:ZENER
- added FB? (x2): HZ0805E601R-10, Libreria_EDU_CIAA_NXP:SM0805, symbol edu-ciaa-nxp:FILTER
- added U?: NCP1117ST33T3G, Libreria_EDU_CIAA_NXP:SOT223, symbol TrackerAVL:NCP1117ST33T3G
Connections:
- net labels added: +3.3V, +3.3VADC, +5V, GND, GNDA, VBAT
- wire segments 0 -> 25
Other:
- note added: "Nets de PWR para ADC"

Commit message: Cambios en sch
Other:
- note added: "EVALUAR FUENTE... Poner mc34063 o switching similar?\no un regulador lineal? Validar tensión máx de entrada."
Changed lines of the file:
@@
 Wire Notes Line
 	6900 4800 7950 4800
+Text Notes 4150 2450 0    59   ~ 0
+EVALUAR FUENTE... Poner mc34063 o switching similar?\no un regulador lineal? Validar tensión máx de entrada.
 $EndSCHEMATC

Commit message: Cambios en sch
Parts:
- added C803: 100nF, Libreria_EDU_CIAA_NXP:c_0805, symbol Device:C
- added C804: 1000uF 50V, symbol Device:CP
- added D801: PMEG3020EH, Libreria_EDU_CIAA_NXP:DO-214AA(SMB), symbol edu-ciaa-nxp:DIODESCH
- added F801: Polyfuse, symbol Device:Polyfuse
- added RV801: Varistor, symbol Device:Varistor
- added U802: LD1085_D²PAK, Package_TO_SOT_SMD:SOT-223-3_TabPin2, symbol Regulator_Linear:LD1117S50TR_SOT223
- gave numbers to parts that had none: 7
Connections:
- wire segments 25 -> 59
Other:
- note removed: "EVALUAR FUENTE... Poner mc34063 o switching similar?\no un regulador lineal? Validar tensión máx de entrada."

Commit message: Cambios en sch y adición de documentación
Parts:
- added R801: 10K, symbol Device:R
- added U803: IRF7105, Libreria_EDU_CIAA_NXP:SOIC-8, symbol EquipoAVL:IRF7105
Connections:
- net labels added: +BATT, IGN
- wire segments 59 -> 82
Other:
- note added: "Testear circuito con 12V ign.\nRevisar, si tengo solo 3.3v en toda la placa, \nentonces saco la parte de la fuente de 3.3v\n(parte de abajo de este sch)."
Changed lines of the file:
@@
 Text Notes 7100 3500 0    59   ~ 0
 Nets de PWR para ADC
-Text HLabel 3550 2100 0    50   Input ~ 0
+Text HLabel 1650 1800 0    50   Input ~ 0
 VBAT
 Wire Wire Line
@@
 L edu-ciaa-nxp:DIODESCH D801
 U 1 1 5BAC5FAB
-P 3950 2100
-F 0 "D801" H 3950 2293 40  0000 C CNN
-F 1 "PMEG3020EH" H 3950 2217 40  0000 C CNN
-F 2 "Libreria_EDU_CIAA_NXP:DO-214AA(SMB)" H 3950 2232 60  0001 C CNN
-F 3 "" H 3950 2100 60  0000 C CNN
-	1    3950 2100
+P 1950 2600
+F 0 "D801" H 1950 2793 40  0000 C CNN
+F 1 "PMEG3020EH" H 1950 2717 40  0000 C CNN
+F 2 "Libreria_EDU_CIAA_NXP:DO-214AA(SMB)" H 1950 2732 60  0001 C CNN
+F 3 "" H 1950 2600 60  0000 C CNN
+	1    1950 2600
 	1    0    0    -1
 $EndComp
@@
 L Device:Polyfuse F801
 U 1 1 5BAC60A8
-P 4500 2100
-F 0 "F801" V 4725 2100 50  0000 C CNN
-F 1 "Polyfuse" V 4634 2100 50  0000 C CNN
-F 2 "" H 4550 1900 50  0001 L CNN
-F 3 "~" H 4500 2100 50  0001 C CNN
-	1    4500 2100
+P 2450 2600
+F 0 "F801" V 2675 2600 50  0000 C CNN
+F 1 "Polyfuse" V 2584 2600 50  0000 C CNN
+F 2 "" H 2500 2400 50  0001 L CNN
+F 3 "~" H 2450 2600 50  0001 C CNN
+	1    2450 2600
 	0    -1   -1   0
 $EndComp
-Wire Wire Line
-	3550 2100 3750 2100
 Wire Wire Line
 	4150 2100 4350 2100
@@
 Wire Wire Line
 	3450 3900 3450 4050
+Text HLabel 1650 1700 0    50   Input ~ 0
+IGN
+$Comp
+L EquipoAVL:IRF7105 U803
+U 1 1 5BBADAEA
+P 2950 1700
+F 0 "U803" H 2950 2067 50  0000 C CNN
+F 1 "IRF7105" H 2950 1976 50  0000 C CNN
+F 2 "Libreria_EDU_CIAA_NXP:SOIC-8" H 2950 1700 50  0001 C CNN
+F 3 "" H 2950 1700 50  0001 C CNN
+	1    2950 1700
+	1    0    0    -1
+$EndComp
+$Comp
+L Device:R R?
+U 1 1 5BBB5359
+P 2000 1900
+AR Path="/5BA5700E/5BBB5359" Ref="R?"  Part="1"
+AR Path="/5BA56FF8/5BBB5359" Ref="R801"  Part="1"
+F 0 "R801" V 2100 1950 50  0000 L CNN
+F 1 "10K" V 2100 1750 50  0000 L CNN
+F 2 "" V 1930 1900 50  0001 C CNN
+F 3 "~" H 2000 1900 50  0001 C CNN
+	1    2000 1900
+	0    1    1    0
+$EndComp
+Wire Wire Line
+	1650 1800 1800 1800
+Wire Wire Line
+	2150 1900 2500 1900
+Wire Wire Line
+	1850 1900 1800 1900
+Wire Wire Line
+	1800 1900 1800 1800
+Connection ~ 1800 1800
+Wire Wire Line
+	1800 1800 2550 1800
+Wire Wire Line
+	3750 2100 3650 2100
+Wire Wire Line
+	3650 2100 3650 1900
+Wire Wire Line
+	3350 1800 3650 1800
+Wire Wire Line
+	3350 1900 3650 1900
+Connection ~ 3650 1900
+Wire Wire Line
+	3650 1900 3650 1800
+Wire Wire Line
+	3350 1600 3400 1600
+Wire Wire Line
+	3400 1600 3400 1700
+Wire Wire Line
+	3400 2100 2500 2100
+Wire Wire Line
+	2500 2100 2500 1900
+Connection ~ 2500 1900
+Wire Wire Line
+	2500 1900 2550 1900
+Wire Wire Line
+	3350 1700 3400 1700
+Connection ~ 3400 1700
+Wire Wire Line
+	3400 1700 3400 2100
+$Comp
+L power:GND #PWR0101
+U 1 1 5BC0B5DC
+P 2500 1450
+F 0 "#PWR0101" H 2500 1200 50  0001 C CNN
+F 1 "GND" H 2505 1277 50  0000 C CNN
+F 2 "" H 2500 1450 50  0001 C CNN
+F 3 "" H 2500 1450 50  0001 C CNN
+	1    2500 1450
+	-1   0    0    1
+$EndComp
+Wire Wire Line
+	2550 1600 2500 1600
+Wire Wire Line
+	2500 1600 2500 1450
+Wire Wire Line
+	1650 1700 2550 1700
+Text Notes 1550 1050 0    79   ~ 16
+Testear circuito con 12V ign.\nRevisar, si tengo solo 3.3v en toda la placa, \nentonces saco la parte de la fuente de 3.3v\n(parte de abajo de este sch).
+$Comp
+L power:+BATT #PWR?
+U 1 1 5BC0FCB4
+P 3650 1450
+F 0 "#PWR?" H 3650 1300 50  0001 C CNN
+F 1 "+BATT" H 3665 1623 50  0000 C CNN
+F 2 "" H 3650 1450 50  0001 C CNN
+F 3 "" H 3650 1450 50  0001 C CNN
+	1    3650 1450
+	1    0    0    -1
+$EndComp
+Wire Wire Line
+	3650 1450 3650 1500
+Connection ~ 3650 1800
+$Comp
+L edu-ciaa-nxp:PWR_FLAG #FLG?
+U 1 1 5BC11B0E
+P 3900 1400
+F 0 "#FLG?" H 3900 1495 30  0001 C CNN
+F 1 "PWR_FLAG" H 3900 1608 30  0000 C CNN
+F 2 "" H 3900 1400 60  0000 C CNN
+F 3 "" H 3900 1400 60  0000 C CNN
+	1    3900 1400
+	1    0    0    -1
+$EndComp
+Wire Wire Line
+	3900 1400 3900 1500
+Wire Wire Line
+	3900 1500 3650 1500
+Connection ~ 3650 1500
+Wire Wire Line
+	3650 1500 3650 1800
 $EndSCHEMATC

Commit message: Cambios en sch
Parts:
- removed C802, C805: 10uF, Libreria_EDU_CIAA_NXP:c_1206_tantalio, symbol Device:CP
- removed U801: NCP1117ST33T3G, Libreria_EDU_CIAA_NXP:SOT223, symbol TrackerAVL:NCP1117ST33T3G
- added C? (x3): 4.7uF 6.3V, Libreria_EDU_CIAA_NXP:c_0805, symbol Device:C
- added U?: NCP114ASN180T1G, symbol NCP114:NCP114SN
- D801: Desc (none) -> DIODE SCHOTTKY 30V 2A SOD123F
- F801: value Polyfuse -> 60R300XF; Desc (none) -> PTC RESET FUSE 60V 3A RADIAL
- RV801: value Varistor -> 30VDC
- U802: value LD1085_D²PAK -> LD1085D2T33R
- U803: value IRF7105 -> STS8C5H30L
Connections:
- net labels added: +1V8
- net labels removed: +5V
- wire segments 82 -> 80
Other:
- note added: "Señales de POWER generadas:\n+3.3V\n+3.3VADC\n+1.8V\n+BATT\nGND\nGNDA\n"
- note removed: "Testear circuito con 12V ign.\nRevisar, si tengo solo 3.3v en toda la placa, \nentonces saco la parte de la fuente de 3.3v\n(parte de abajo de este sch)."
- moved on the sheet: U802

Commit message: Cambios en sch
Parts:
- gave numbers to parts that had none: 4
Changed lines of the file:
@@
 $Descr A4 11693 8268
 encoding utf-8
-Sheet 6 7
+Sheet 5 8
 Title ""
 Date ""
@@
 Wire Wire Line
 	1800 2550 2700 2550
-Text Notes 5050 1650 0    79   ~ 16
+Text Notes 1600 1750 0    79   ~ 16
 Señales de POWER generadas:\n+3.3V\n+3.3VADC\n+1.8V\n+BATT\nGND\nGNDA\n
 $Comp
@@
 $EndComp
 $Comp
-L Device:C C?
+L Device:C C502
 U 1 1 5BCB6C25
 P 6900 2750
-F 0 "C?" H 7015 2796 50  0000 L CNN
+F 0 "C502" H 7015 2796 50  0000 L CNN
 F 1 "4.7uF 6.3V" H 7015 2705 50  0000 L CNN
 F 2 "Libreria_EDU_CIAA_NXP:c_0805" H 6938 2600 50  0001 C CNN
@@
 	3800 2300 3800 2500
 $Comp
-L NCP114:NCP114SN U?
+L NCP114:NCP114SN U502
 U 1 1 5BCD771B
 P 6300 4100
-F 0 "U?" H 6300 4375 50  0000 C CNN
+F 0 "U502" H 6300 4375 50  0000 C CNN
 F 1 "NCP114ASN180T1G" H 6300 4284 50  0000 C CNN
 F 2 "" H 6300 4100 50  0001 C CNN
@@
 	7200 3850 7200 4050
 $Comp
-L Device:C C?
+L Device:C C503
 U 1 1 5BCEE528
 P 6900 4250
-F 0 "C?" H 7015 4296 50  0000 L CNN
+F 0 "C503" H 7015 4296 50  0000 L CNN
 F 1 "4.7uF 6.3V" H 7015 4205 50  0000 L CNN
 F 2 "Libreria_EDU_CIAA_NXP:c_0805" H 6938 4100 50  0001 C CNN
@@
 Connection ~ 5600 4500
 $Comp
-L Device:C C?
+L Device:C C501
 U 1 1 5BD0EA83
 P 5600 4250
-F 0 "C?" H 5750 4250 50  0000 L CNN
+F 0 "C501" H 5750 4250 50  0000 L CNN
 F 1 "4.7uF 6.3V" H 5650 4150 50  0000 L CNN
 F 2 "Libreria_EDU_CIAA_NXP:c_0805" H 5638 4100 50  0001 C CNN
