File: TrackerAVL/conectores_io.sch (KiCad schematic (older format))
At the start: 3 parts

Commit message: Cambios en sch
Other:
- note added: "PWR Display"
Changed lines of the file:
@@
 $Descr A4 11693 8268
 encoding utf-8
-Sheet 5 8
+Sheet 4 8
 Title ""
 Date ""
@@
 Wire Wire Line
 	6100 2400 6700 2400
-Text HLabel 6700 1900 2    50   Output ~ 0
+Text HLabel 6700 1900 2    50   Input ~ 0
 DIG_OUT_1
-Text HLabel 6700 2000 2    50   Output ~ 0
+Text HLabel 6700 2000 2    50   Input ~ 0
 DIG_OUT_3
-Text HLabel 6700 2100 2    50   Output ~ 0
+Text HLabel 6700 2100 2    50   Input ~ 0
 DIG_OUT_3
-Text HLabel 6700 2200 2    50   Input ~ 0
+Text HLabel 6700 2200 2    50   Output ~ 0
 AN_IN_1
-Text HLabel 6700 2300 2    50   Input ~ 0
+Text HLabel 6700 2300 2    50   Output ~ 0
 AN_IN_2
-Text HLabel 6700 2400 2    50   Input ~ 0
+Text HLabel 6700 2400 2    50   Output ~ 0
 AN_IN_3
-Text HLabel 5000 2000 0    50   Input ~ 0
+Text HLabel 5000 2000 0    50   Output ~ 0
 DIG_IN_1
-Text HLabel 5000 2100 0    50   Input ~ 0
+Text HLabel 5000 2100 0    50   Output ~ 0
 DIG_IN_2
-Text HLabel 5000 2200 0    50   Input ~ 0
+Text HLabel 5000 2200 0    50   Output ~ 0
 DIG_IN_3
 Wire Wire Line
@@
 Text HLabel 5000 5000 0    50   Input ~ 0
 PROG_RX
+Wire Notes Line
+	4950 2950 3500 2950
+Text Notes 3500 2950 0    59   ~ 0
+PWR Display
 $EndSCHEMATC

Commit message: Cambios en sch
Parts:
- gave numbers to parts that had none: 3
Changed lines of the file:
@@
 $EndDescr
 $Comp
-L Connector_Generic:Conn_02x07_Top_Bottom J?
+L Connector_Generic:Conn_02x07_Top_Bottom J401
 U 1 1 5BA83A7B
 P 5800 2100
-F 0 "J?" H 5850 1700 50  0000 C CNN
+F 0 "J401" H 5850 1700 50  0000 C CNN
 F 1 "Conn_02x07_Odd_Even" H 5850 1600 50  0000 C CNN
 F 2 "Connector_Molex_MM:Molex_Micro-Fit_3.0_43045-1406_2x07-1MP_P3.00mm_Horizontal" H 5800 2100 50  0001 C CNN
@@
 $EndComp
 $Comp
-L Connector_Generic:Conn_01x04 J?
+L Connector_Generic:Conn_01x04 J403
 U 1 1 5BA83B5F
 P 5800 4900
-F 0 "J?" H 5880 4892 50  0000 L CNN
+F 0 "J403" H 5880 4892 50  0000 L CNN
 F 1 "Conn_01x04" H 5880 4801 50  0000 L CNN
 F 2 "Connector_Molex_MM:Molex_Pico_SPOX_87438-0443_1x04" H 5800 4900 50  0001 C CNN
@@
 $EndComp
 $Comp
-L Connector_Generic:Conn_01x15 J?
+L Connector_Generic:Conn_01x15 J402
 U 1 1 5BA83CA7
 P 5800 3600
-F 0 "J?" H 5880 3642 50  0000 L CNN
+F 0 "J402" H 5880 3642 50  0000 L CNN
 F 1 "Conn_01x15" H 5880 3551 50  0000 L CNN
 F 2 "Connector_Molex_MM:Molex_Pico_SPOX_87438-0443_1x15" H 5800 3600 50  0001 C CNN
@@
 GND_CONN_1
 $Comp
-L power:GND #PWR?
+L power:GND #PWR0401
 U 1 1 5BA977C8
 P 5050 1300
-F 0 "#PWR?" H 5050 1050 50  0001 C CNN
+F 0 "#PWR0401" H 5050 1050 50  0001 C CNN
 F 1 "GND" H 5055 1127 50  0000 C CNN
 F 2 "" H 5050 1300 50  0001 C CNN

Commit message: Cambios en sch
Connections:
- wire segments 39 -> 41
Changed lines of the file:
@@
 Text Notes 3500 2950 0    59   ~ 0
 PWR Display
+$Comp
+L power:PWR_FLAG #FLG?
+U 1 1 5BCF30C6
+P 4850 950
+F 0 "#FLG?" H 4850 1025 50  0001 C CNN
+F 1 "PWR_FLAG" H 4850 1124 50  0000 C CNN
+F 2 "" H 4850 950 50  0001 C CNN
+F 3 "~" H 4850 950 50  0001 C CNN
+	1    4850 950
+	1    0    0    -1
+$EndComp
+Wire Wire Line
+	4850 950  4850 1000
+Wire Wire Line
+	4850 1000 5050 1000
+Connection ~ 5050 1000
+Text HLabel 4550 3500 0    50   Output ~ 0
+DISP_1
+Text HLabel 4550 3600 0    50   Output ~ 0
+DISP_2
+Text HLabel 4550 3700 0    50   Output ~ 0
+DISP_3
+Text HLabel 4550 3800 0    50   Output ~ 0
+DISP_4
 $EndSCHEMATC

Commit message: Cambios en sch
Connections:
- net labels added: +3.3V, AN_IN_0, DIG_IN_0, DIG_OUT_0, DIG_OUT_2, DISP_0, TEC_0
- net labels removed: AN_INPUT_1, AN_INPUT_2, AN_INPUT_3, AN_IN_3, DIG_INPUT_1, DIG_INPUT_2, DIG_INPUT_3, DIG_IN_3, DIG_OUTPUT_1, DIG_OUTPUT_2, DIG_OUTPUT_3, DIG_OUT_3, DISP_4, TEC_4, VCC_CONSOLA
- wire segments 41 -> 42
Other:
- note added: "Audio consola"
- note added: "Display consola"
- note added: "Entradas analógicas"
- note added: "Entradas digitales"
- note added: "IButton consola"
- note added: "Interfaz consola"
- note added: "Interfaz de serial"
- note added: "Interfaz principal"
- note added: "Interfaz programación"
- note added: "Salidas digitales"
- note added: "Señal de ignición"
- note added: "Teclas consola"
- note added: "Tensión de batería"
- moved on the sheet: J401, J402, J403

Commit message: Cambios en sch
Parts:
- added D801, D802, D803, D804, D805: PESD5V0L1UA, Diode_THT:D_DO-201AE_P15.24mm_Horizontal, symbol Diode:1.5KExxA
- renumbered J401 to J801, J402 to J802, J403 to J803
Connections:
- net DISP_0: now also D805.1 (A1)
- net DISP_1: now also D804.1 (A1)
- net DISP_2: now also D803.1 (A1)
- net DISP_3: now also D802.1 (A1)
- net GND: now also D801.2 (A2), D802.2 (A2), D803.2 (A2), D804.2 (A2), D805.2 (A2)
- net IBUTTON: now also D801.1 (A1)
Other:
- note added: "Protecciones IO"
- note removed: "Interfaz de serial"
Changed lines of the file:
@@
 $Descr A4 11693 8268
 encoding utf-8
-Sheet 6 8
+Sheet 8 8
 Title ""
 Date ""
@@
 $EndDescr
 $Comp
-L Connector_Generic:Conn_02x07_Top_Bottom J401
+L Connector_Generic:Conn_02x07_Top_Bottom J801
 U 1 1 5BA83A7B
 P 5800 1950
-F 0 "J401" H 5850 1550 50  0000 C CNN
+F 0 "J801" H 5850 1550 50  0000 C CNN
 F 1 "Conn_02x07_Odd_Even" H 5850 1450 50  0000 C CNN
 F 2 "Connector_Molex_MM:Molex_Micro-Fit_3.0_43045-1406_2x07-1MP_P3.00mm_Horizontal" H 5800 1950 50  0001 C CNN
@@
 $EndComp
 $Comp
-L Connector_Generic:Conn_01x04 J403
+L Connector_Generic:Conn_01x04 J803
 U 1 1 5BA83B5F
 P 5800 5200
-F 0 "J403" H 5880 5192 50  0000 L CNN
+F 0 "J803" H 5880 5192 50  0000 L CNN
 F 1 "Conn_01x04" H 5880 5101 50  0000 L CNN
 F 2 "Connector_Molex_MM:Molex_Pico_SPOX_87438-0443_1x04" H 5800 5200 50  0001 C CNN
@@
 $EndComp
 $Comp
-L Connector_Generic:Conn_01x15 J402
+L Connector_Generic:Conn_01x15 J802
 U 1 1 5BA83CA7
 P 5800 3700
-F 0 "J402" H 5880 3742 50  0000 L CNN
+F 0 "J802" H 5880 3742 50  0000 L CNN
 F 1 "Conn_01x15" H 5880 3651 50  0000 L CNN
 F 2 "Connector_Molex_MM:Molex_Pico_SPOX_87438-0443_1x15" H 5800 3700 50  0001 C CNN
@@
 GND_CONN_1
 $Comp
-L power:GND #PWR0401
+L power:GND #PWR0801
 U 1 1 5BA977C8
-P 9350 2700
-F 0 "#PWR0401" H 9350 2450 50  0001 C CNN
-F 1 "GND" H 9355 2527 50  0000 C CNN
-F 2 "" H 9350 2700 50  0001 C CNN
-F 3 "" H 9350 2700 50  0001 C CNN
-	1    9350 2700
-	1    0    0    -1
-$EndComp
-Text Label 9900 2400 2    50   ~ 0
+P 1800 2000
+F 0 "#PWR0801" H 1800 1750 50  0001 C CNN
+F 1 "GND" H 1805 1827 50  0000 C CNN
+F 2 "" H 1800 2000 50  0001 C CNN
+F 3 "" H 1800 2000 50  0001 C CNN
+	1    1800 2000
+	1    0    0    -1
+$EndComp
+Text Label 2350 1700 2    50   ~ 0
 GND_CONN_1
 Wire Wire Line
-	9350 2400 9900 2400
+	1800 1700 2350 1700
 Text Label 5050 3000 0    50   ~ 0
 VCC_CONN_2
@@
 IGN
 Wire Wire Line
-	9350 2500 9900 2500
-Wire Wire Line
-	9350 2600 9900 2600
-Wire Wire Line
-	9350 2400 9350 2500
-Wire Wire Line
-	9350 2500 9350 2600
-Connection ~ 9350 2500
-Wire Wire Line
-	9350 2600 9350 2700
-Connection ~ 9350 2600
-Text Label 9900 2500 2    50   ~ 0
+	1800 1800 2350 1800
+Wire Wire Line
+	1800 1900 2350 1900
+Wire Wire Line
+	1800 1700 1800 1800
+Wire Wire Line
+	1800 1800 1800 1900
+Connection ~ 1800 1800
+Wire Wire Line
+	1800 1900 1800 2000
+Connection ~ 1800 1900
+Text Label 2350 1800 2    50   ~ 0
 GND_CONN_2
-Text Label 9900 2600 2    50   ~ 0
+Text Label 2350 1900 2    50   ~ 0
 GND_CONN_3
 Wire Wire Line
@@
 PWR Display
 $Comp
-L power:PWR_FLAG #FLG0102
+L power:PWR_FLAG #FLG0801
 U 1 1 5BCF30C6
-P 9150 2350
-F 0 "#FLG0102" H 9150 2425 50  0001 C CNN
-F 1 "PWR_FLAG" H 9150 2524 50  0000 C CNN
-F 2 "" H 9150 2350 50  0001 C CNN
-F 3 "~" H 9150 2350 50  0001 C CNN
-	1    9150 2350
-	1    0    0    -1
-$EndComp
-Wire Wire Line
-	9150 2350 9150 2400
-Wire Wire Line
-	9150 2400 9350 2400
-Connection ~ 9350 2400
+P 1600 1650
+F 0 "#FLG0801" H 1600 1725 50  0001 C CNN
+F 1 "PWR_FLAG" H 1600 1824 50  0000 C CNN
+F 2 "" H 1600 1650 50  0001 C CNN
+F 3 "~" H 1600 1650 50  0001 C CNN
+	1    1600 1650
+	1    0    0    -1
+$EndComp
+Wire Wire Line
+	1600 1650 1600 1700
+Wire Wire Line
+	1600 1700 1800 1700
+Connection ~ 1800 1700
 Text HLabel 5000 3700 0    50   BiDi ~ 0
 DISP_1
@@
 DISP_0
 Wire Notes Line
-	4950 3550 3500 3550
+	3500 3550 4950 3550
 Text Notes 3500 3550 0    59   ~ 0
 Teclas consola
@@
 Text Notes 8200 2300 2    59   ~ 0
 Entradas analógicas
-Wire Notes Line
-	4950 5350 3500 5350
-Text Notes 3500 5350 0    59   ~ 0
-Interfaz de serial
 Text Notes 5350 1500 0    79   ~ 16
 Interfaz principal
@@
 Interfaz programación
 $Comp
-L power:+3.3V #PWR0149
+L power:+3.3V #PWR0802
 U 1 1 5BCDA499
 P 4850 2900
-F 0 "#PWR0149" H 4850 2750 50  0001 C CNN
+F 0 "#PWR0802" H 4850 2750 50  0001 C CNN
 F 1 "+3.3V" H 4865 3073 50  0000 C CNN
 F 2 "" H 4850 2900 50  0001 C CNN
@@
 Wire Wire Line
 	4850 3000 5600 3000
+$Comp
+L Diode:1.5KExxA D?
+U 1 1 5BDE240C
+P 7900 3800
+AR Path="/5BA56FC1/5BDE240C" Ref="D?"  Part="1"
+AR Path="/5BD5C4FD/5BDE240C" Ref="D?"  Part="1"
+AR Path="/5BA5703C/5BDE240C" Ref="D801"  Part="1"
+F 0 "D801" H 7900 3900 50  0000 L CNN
+F 1 "PESD5V0L1UA" H 7650 3700 50  0000 L CNN
+F 2 "Diode_THT:D_DO-201AE_P15.24mm_Horizontal" H 7900 3600 50  0001 C CNN
+F 3 "https://www.vishay.com/docs/88301/15ke.pdf" H 7850 3800 50  0001 C CNN
+	1    7900 3800
+	0    1    1    0
+$EndComp
+Text Label 5050 3600 0    50   ~ 0
+DISP_0
+Text Label 5050 3700 0    50   ~ 0
+DISP_1
+Text Label 5050 3800 0    50   ~ 0
+DISP_2
+Text Label 5050 3900 0    50   ~ 0
+DISP_3
+Text Label 5050 4400 0    50   ~ 0
+IBUTTON
+$Comp
+L Diode:1.5KExxA D?
+U 1 1 5BD351A1
+P 8200 3800
+AR Path="/5BA56FC1/5BD351A1" Ref="D?"  Part="1"
+AR Path="/5BD5C4FD/5BD351A1" Ref="D?"  Part="1"
+AR Path="/5BA5703C/5BD351A1" Ref="D802"  Part="1"
+F 0 "D802" H 8200 3900 50  0000 L CNN
+F 1 "PESD5V0L1UA" H 7950 3700 50  0000 L CNN
+F 2 "Diode_THT:D_DO-201AE_P15.24mm_Horizontal" H 8200 3600 50  0001 C CNN
+F 3 "https://www.vishay.com/docs/88301/15ke.pdf" H 8150 3800 50  0001 C CNN
+	1    8200 3800
+	0    1    1    0
+$EndComp
+$Comp
+L Diode:1.5KExxA D?
+U 1 1 5BD351C7
+P 8500 3800
+AR Path="/5BA56FC1/5BD351C7" Ref="D?"  Part="1"
+AR Path="/5BD5C4FD/5BD351C7" Ref="D?"  Part="1"
+AR Path="/5BA5703C/5BD351C7" Ref="D803"  Part="1"
+F 0 "D803" H 8500 3900 50  0000 L CNN
+F 1 "PESD5V0L1UA" H 8250 3700 50  0000 L CNN
+F 2 "Diode_THT:D_DO-201AE_P15.24mm_Horizontal" H 8500 3600 50  0001 C CNN
+F 3 "https://www.vishay.com/docs/88301/15ke.pdf" H 8450 3800 50  0001 C CNN
+	1    8500 3800
+	0    1    1    0
+$EndComp
+$Comp
+L Diode:1.5KExxA D?
+U 1 1 5BD351EB
+P 8800 3800
+AR Path="/5BA56FC1/5BD351EB" Ref="D?"  Part="1"
+AR Path="/5BD5C4FD/5BD351EB" Ref="D?"  Part="1"
+AR Path="/5BA5703C/5BD351EB" Ref="D804"  Part="1"
+F 0 "D804" H 8800 3900 50  0000 L CNN
+F 1 "PESD5V0L1UA" H 8550 3700 50  0000 L CNN
+F 2 "Diode_THT:D_DO-201AE_P15.24mm_Horizontal" H 8800 3600 50  0001 C CNN
+F 3 "https://www.vishay.com/docs/88301/15ke.pdf" H 8750 3800 50  0001 C CNN
+	1    8800 3800
+	0    1    1    0
+$EndComp
+$Comp
+L Diode:1.5KExxA D?
+U 1 1 5BD35211
+P 9100 3800
+AR Path="/5BA56FC1/5BD35211" Ref="D?"  Part="1"
+AR Path="/5BD5C4FD/5BD35211" Ref="D?"  Part="1"
+AR Path="/5BA5703C/5BD35211" Ref="D805"  Part="1"
+F 0 "D805" H 9100 3900 50  0000 L CNN
+F 1 "PESD5V0L1UA" H 8850 3700 50  0000 L CNN
+F 2 "Diode_THT:D_DO-201AE_P15.24mm_Horizontal" H 9100 3600 50  0001 C CNN
+F 3 "https://www.vishay.com/docs/88301/15ke.pdf" H 9050 3800 50  0001 C CNN
+	1    9100 3800
+	0    1    1    0
+$EndComp
+$Comp
+L power:GND #PWR0803
+U 1 1 5BD35291
+P 7900 4200
+F 0 "#PWR0803" H 7900 3950 50  0001 C CNN
+F 1 "GND" H 7905 4027 50  0000 C CNN
+F 2 "" H 7900 4200 50  0001 C CNN
+F 3 "" H 7900 4200 50  0001 C CNN
+	1    7900 4200
+	1    0    0    -1
+$EndComp
+Wire Wire Line
+	7900 3950 7900 4100
+Wire Wire Line
+	7900 4100 8200 4100
+Wire Wire Line
+	8200 4100 8200 3950
+Connection ~ 7900 4100
+Wire Wire Line
+	7900 4100 7900 4200
+Wire Wire Line
+	8200 4100 8500 4100
+Wire Wire Line
+	8500 4100 8500 3950
+Connection ~ 8200 4100
+Wire Wire Line
+	8500 4100 8800 4100
+Wire Wire Line
+	8800 4100 8800 3950
+Connection ~ 8500 4100
+Wire Wire Line
+	8800 4100 9100 4100
+Wire Wire Line
+	9100 4100 9100 3950
+Connection ~ 8800 4100
+Wire Wire Line
+	7900 3650 7900 3500
+Text Label 7450 3100 0    50   ~ 0
+DISP_0
+Wire Wire Line
+	7450 3500 7900 3500
+Text Notes 7850 2850 0    79   ~ 16
+Protecciones IO
+Wire Wire Line
+	8200 3650 8200 3400
+Wire Wire Line
+	8200 3400 7450 3400
+Wire Wire Line
+	7450 3300 8500 3300
+Wire Wire Line
+	8500 3300 8500 3650
+Wire Wire Line
+	7450 3200 8800 3200
+Wire Wire Line
+	8800 3200 8800 3650
+Wire Wire Line
+	7450 3100 9100 3100
+Wire Wire Line
+	9100 3100 9100 3650
+Text Label 7450 3200 0    50   ~ 0
+DISP_1
+Text Label 7450 3300 0    50   ~ 0
+DISP_2
+Text Label 7450 3400 0    50   ~ 0
+DISP_3
+Text Label 7450 3500 0    50   ~ 0
+IBUTTON
 $EndSCHEMATC

Commit message: Cambios en sch
Parts:
- added U801: 74HC4053, symbol 74xx:74HC4053
Connections:
- net +3V3: now also U801.16 (VCC)
- net DISP_0: now also U801.14 (An)
- net DISP_1: now also U801.15 (Bn)
- net DISP_2: now also U801.4 (Cn)
- net GND: now also U801.6 (~E), U801.7 (VEE), U801.8 (GND)
- net DISP_3 renamed BUZZER
- new net DISPLAY_MODE: U801.10 (S1), U801.11 (S0), U801.9 (S2)
- new net DISP_I2C_SCL: U801.12 (A0)
- new net DISP_I2C_SDA: U801.2 (B0)
- new net DISP_SPI_CS1: U801.3 (C1)
- new net DISP_SPI_MOSI: U801.1 (B1)
- new net DISP_SPI_SCK: U801.13 (A1)
- no-connect marks 0 -> 1
Other:
- note added: "Buzzer consola"
- note added: "DM = 0 / DM = 1"
- note added: "I2C_SCL / SPI_SCK"
- note added: "I2C_SDA / SPI_MOSI"
- note added: "Lógica de switcheo de buses I2C/SPI\n(según protocolo del display)"
- note added: "NC / SPI_CS1"
- moved on the sheet: D801, D802, D803, D804, D805, J801, J803
