File: TrackerAVL/conectores_io.sch (KiCad schematic (older format))
At the start: 9 parts, among them J801 Conn_02x07_Odd_Even, J802 Conn_01x15, J803 Conn_01x04, U801 74HC4053

Commit message: Cambios en sch
Parts:
- D801, D802, D803, D804, D805: footprint Diode_THT:D_DO-201AE_P15.24mm_Horizontal -> Diode_SMD:D_SOD-323_HandSoldering
- U801: footprint (none) -> Package_SO:TSSOP-16_4.4x5mm_P0.65mm
Changed lines of the file:
@@
 encoding utf-8
 Sheet 8 8
-Title ""
-Date ""
-Rev ""
+Title "Equipo AVL - vRaptor"
+Date "2018-10-30"
+Rev "1.0"
 Comp ""
-Comment1 ""
+Comment1 "Ing. Mauro Moreyra"
 Comment2 ""
 Comment3 ""
@@
 F 0 "D801" H 7900 3700 50  0000 L CNN
 F 1 "PESD5V0L1UA" H 7650 3500 50  0000 L CNN
-F 2 "Diode_THT:D_DO-201AE_P15.24mm_Horizontal" H 7900 3400 50  0001 C CNN
+F 2 "Diode_SMD:D_SOD-323_HandSoldering" H 7900 3400 50  0001 C CNN
 F 3 "https://www.vishay.com/docs/88301/15ke.pdf" H 7850 3600 50  0001 C CNN
 	1    7900 3600
@@
 F 0 "D802" H 8200 3700 50  0000 L CNN
 F 1 "PESD5V0L1UA" H 7950 3500 50  0000 L CNN
-F 2 "Diode_THT:D_DO-201AE_P15.24mm_Horizontal" H 8200 3400 50  0001 C CNN
+F 2 "Diode_SMD:D_SOD-323_HandSoldering" H 8200 3400 50  0001 C CNN
 F 3 "https://www.vishay.com/docs/88301/15ke.pdf" H 8150 3600 50  0001 C CNN
 	1    8200 3600
@@
 F 0 "D803" H 8500 3700 50  0000 L CNN
 F 1 "PESD5V0L1UA" H 8250 3500 50  0000 L CNN
-F 2 "Diode_THT:D_DO-201AE_P15.24mm_Horizontal" H 8500 3400 50  0001 C CNN
+F 2 "Diode_SMD:D_SOD-323_HandSoldering" H 8500 3400 50  0001 C CNN
 F 3 "https://www.vishay.com/docs/88301/15ke.pdf" H 8450 3600 50  0001 C CNN
 	1    8500 3600
@@
 F 0 "D804" H 8800 3700 50  0000 L CNN
 F 1 "PESD5V0L1UA" H 8550 3500 50  0000 L CNN
-F 2 "Diode_THT:D_DO-201AE_P15.24mm_Horizontal" H 8800 3400 50  0001 C CNN
+F 2 "Diode_SMD:D_SOD-323_HandSoldering" H 8800 3400 50  0001 C CNN
 F 3 "https://www.vishay.com/docs/88301/15ke.pdf" H 8750 3600 50  0001 C CNN
 	1    8800 3600
@@
 F 0 "D805" H 9100 3700 50  0000 L CNN
 F 1 "PESD5V0L1UA" H 8850 3500 50  0000 L CNN
-F 2 "Diode_THT:D_DO-201AE_P15.24mm_Horizontal" H 9100 3400 50  0001 C CNN
+F 2 "Diode_SMD:D_SOD-323_HandSoldering" H 9100 3400 50  0001 C CNN
 F 3 "https://www.vishay.com/docs/88301/15ke.pdf" H 9050 3600 50  0001 C CNN
 	1    9100 3600
@@
 F 0 "U801" H 2500 6300 50  0000 C CNN
 F 1 "74HC4053" H 2100 6300 50  0000 C CNN
-F 2 "" H 2400 5400 50  0001 C CNN
+F 2 "Package_SO:TSSOP-16_4.4x5mm_P0.65mm" H 2400 5400 50  0001 C CNN
 F 3 "http://www.ti.com/lit/ds/symlink/cd74hct4051.pdf" H 2400 5400 50  0001 C CNN
 	1    2400 5800

Commit message: Cambios en pcb
Other:
- note added: "DISPLAY_MODE (DM)"
Changed lines of the file:
@@
 Text Notes 3400 5400 0    50   ~ 0
 DM = 0 / DM = 1
+Text Notes 3400 5300 0    50   ~ 0
+DISPLAY_MODE (DM)
 $EndSCHEMATC

Commit message: Cambios en pcb y modelos 3d
Parts:
- U801: footprint Package_SO:TSSOP-16_4.4x5mm_P0.65mm -> Package_SO:SOIC-16_3.9x9.9mm_P1.27mm
Changed lines of the file:
@@
 F 0 "U801" H 2500 6300 50  0000 C CNN
 F 1 "74HC4053" H 2100 6300 50  0000 C CNN
-F 2 "Package_SO:TSSOP-16_4.4x5mm_P0.65mm" H 2400 5400 50  0001 C CNN
+F 2 "Package_SO:SOIC-16_3.9x9.9mm_P1.27mm" H 2400 5400 50  0001 C CNN
 F 3 "http://www.ti.com/lit/ds/symlink/cd74hct4051.pdf" H 2400 5400 50  0001 C CNN
 	1    2400 5800

Commit message: Cambios en pcb
Parts:
- U801: symbol 74xx:74HC4053 -> TrackerAVL-rescue:74HC4053-74xx
Changed lines of the file:
@@
 DISPLAY_MODE
 $Comp
-L 74xx:74HC4053 U801
+L TrackerAVL-rescue:74HC4053-74xx U801
 U 1 1 5BDADD1C
 P 2400 5800
