File: TrackerAVL/cpu.sch (KiCad schematic (older format))
At the start: 1 part

Commit message: Cambios en sch
Parts:
- gave numbers to parts that had none: 1
Changed lines of the file:
@@
 NoConn ~ 6700 8800
 $Comp
-L power:GND #PWR?
+L power:GND #PWR0201
 U 1 1 5BAA5B3A
 P 7650 10000
-F 0 "#PWR?" H 7650 9750 50  0001 C CNN
+F 0 "#PWR0201" H 7650 9750 50  0001 C CNN
 F 1 "GND" H 7655 9827 50  0000 C CNN
 F 2 "" H 7650 10000 50  0001 C CNN
@@
 Connection ~ 7850 9800
 $Comp
-L power:GNDA #PWR?
+L power:GNDA #PWR0202
 U 1 1 5BAAC763
 P 8050 10000
-F 0 "#PWR?" H 8050 9750 50  0001 C CNN
+F 0 "#PWR0202" H 8050 9750 50  0001 C CNN
 F 1 "GNDA" H 8055 9827 50  0000 C CNN
 F 2 "" H 8050 10000 50  0001 C CNN
@@
 RTCX1
 $Comp
-L TrackerAVL:LPC4337JBD144 U?
+L TrackerAVL:LPC4337JBD144 U201
 U 1 1 5BA579FD
 P 7650 6450
-F 0 "U?" H 8650 3550 60  0000 C CNN
+F 0 "U201" H 8650 3550 60  0000 C CNN
 F 1 "LPC4337JBD144" H 8950 3450 60  0000 C CNN
-F 2 "" H 7550 10400 60  0000 C CNN
+F 2 "" H 7550 10400 60  0001 C CNN
 F 3 "" H 7550 10400 60  0000 C CNN
 	1    7650 6450

Commit message: Cambios en sch
Parts:
- added R? (x2): 2K2, symbol Device:R
Connections:
- net labels added: +3.3V, I2C_SCA, I2C_SCL
- wire segments 24 -> 34
- no-connect marks 60 -> 62
Changed lines of the file:
@@
 	1    0    0    -1
 $EndComp
+Text HLabel 10500 7100 2    50   Output ~ 0
+I2C_SCL
+$Comp
+L Device:R R?
+U 1 1 5BD137D9
+P 10300 6900
+F 0 "R?" V 10400 6800 50  0000 L CNN
+F 1 "2K2" V 10300 6800 50  0000 L CNN
+F 2 "" V 10230 6900 50  0001 C CNN
+F 3 "~" H 10300 6900 50  0001 C CNN
+	1    10300 6900
+	1    0    0    -1
+$EndComp
+Text HLabel 10500 7200 2    50   BiDi ~ 0
+I2C_SCA
+Wire Wire Line
+	10500 7100 10300 7100
+Wire Wire Line
+	9400 7200 10100 7200
+$Comp
+L Device:R R?
+U 1 1 5BD13DA2
+P 10100 6900
+F 0 "R?" V 10200 6800 50  0000 L CNN
+F 1 "2K2" V 10100 6800 50  0000 L CNN
+F 2 "" V 10030 6900 50  0001 C CNN
+F 3 "~" H 10100 6900 50  0001 C CNN
+	1    10100 6900
+	1    0    0    -1
+$EndComp
+$Comp
+L power:+3.3V #PWR?
+U 1 1 5BD13ECF
+P 10300 6650
+F 0 "#PWR?" H 10300 6500 50  0001 C CNN
+F 1 "+3.3V" H 10315 6823 50  0000 C CNN
+F 2 "" H 10300 6650 50  0001 C CNN
+F 3 "" H 10300 6650 50  0001 C CNN
+	1    10300 6650
+	1    0    0    -1
+$EndComp
+Wire Wire Line
+	10300 6650 10300 6700
+Wire Wire Line
+	10300 6700 10100 6700
+Wire Wire Line
+	10100 6700 10100 6750
+Connection ~ 10300 6700
+Wire Wire Line
+	10300 6700 10300 6750
+Wire Wire Line
+	10300 7050 10300 7100
+Connection ~ 10300 7100
+Wire Wire Line
+	10300 7100 9400 7100
+Wire Wire Line
+	10100 7050 10100 7200
+Connection ~ 10100 7200
+Wire Wire Line
+	10100 7200 10500 7200
+NoConn ~ 9400 6800
+NoConn ~ 9400 6900
 $EndSCHEMATC

Commit message: Cambios en sch
Connections:
- net labels added: AN_IN_0, AN_IN_1, AN_IN_2, DIG_IN_0, DIG_IN_1, DIG_IN_2, DIG_OUT_0, DIG_OUT_1, DIG_OUT_2, GPIO8, TEC_0, TEC_1, TEC_2, TEC_3
- net labels removed: LED1, LED2, LED3, PULS_0, PULS_1, PULS_2, PULS_3
- wire segments 34 -> 35
Other:
- note added: "LEDS\n"
Changed lines of the file:
@@
 $Descr A3 16535 11693
 encoding utf-8
-Sheet 2 8
+Sheet 2 7
 Title ""
 Date ""
@@
 NoConn ~ 6700 1850
 Text HLabel 6300 2350 0    50   Input ~ 0
-PULS_0
+TEC_0
 Text HLabel 6300 2450 0    50   Input ~ 0
-PULS_1
+TEC_1
 Text HLabel 6300 2550 0    50   Input ~ 0
-PULS_2
+TEC_2
 Text HLabel 6300 2650 0    50   Input ~ 0
 SPI_MISO
@@
 SPI_MOSI
 Text HLabel 6300 2950 0    50   Input ~ 0
-PULS_3
+TEC_3
 Wire Wire Line
 	6700 2350 6300 2350
@@
 NoConn ~ 6700 5300
 NoConn ~ 6700 5400
-Text HLabel 6300 5500 0    50   Output ~ 0
-LED1
-Text HLabel 6300 5600 0    50   Output ~ 0
-LED2
-Text HLabel 6300 5700 0    50   Output ~ 0
-LED3
 Wire Wire Line
 	6700 5500 6300 5500
@@
 NoConn ~ 9400 6800
 NoConn ~ 9400 6900
+Text HLabel 14000 2600 2    50   Output ~ 0
+DIG_OUT_1
+Text HLabel 14000 2700 2    50   Output ~ 0
+DIG_OUT_2
+Text HLabel 14000 2500 2    50   Output ~ 0
+DIG_OUT_0
+Wire Notes Line
+	6100 5500 6100 5700
+Text Notes 6000 5650 2    50   ~ 0
+LEDS\n
+Text HLabel 14000 3000 2    50   Input ~ 0
+AN_IN_0
+Text HLabel 14000 3100 2    50   Input ~ 0
+AN_IN_1
+Text HLabel 14000 3200 2    50   Input ~ 0
+AN_IN_2
+Text HLabel 14000 3550 2    50   Input ~ 0
+DIG_IN_1
+Text HLabel 14000 3650 2    50   Input ~ 0
+DIG_IN_2
+Text HLabel 14000 3450 2    50   Input ~ 0
+DIG_IN_0
+Text HLabel 9800 3850 2    50   BiDi ~ 0
+GPIO8
+Wire Wire Line
+	9400 3850 9800 3850
 $EndSCHEMATC

Commit message: Cambios en sch
Parts:
- added C? (x31): 100nF, symbol Device:C
- added C?: 10uF, symbol Device:C
- added C? (x4): 20pF, symbol Device:C
- added D? (x3): BZT52C36, Diode_SMD:D_SOD-123, symbol Diode:BZT52Bxx
- added D? (x7): PESD5V0L1UA, Diode_THT:D_DO-201AE_P15.24mm_Horizontal, symbol Diode:1.5KExxA
- added D?: LED ROJO, symbol Device:LED_ALT
- added D?: LED AZUL, symbol Device:LED_ALT
- added D?: LED VERDE, symbol Device:LED_ALT
- added FB? (x2): MI0805M221R-10, symbol TrackerAVL:FILTER
- added JP?: JP, symbol Device:Jumper_NO_Small
- added P?: uC_debug, symbol TrackerAVL:CONN_5X2
- added Q? (x3): 2N7002P, Package_TO_SOT_SMD:SOT-23, symbol Transistor_FET:2N7002
- added Q? (x4): DTC043ZEBTL, symbol Transistor_BJT:DTC143Z
- added R? (x9): 10K, symbol Device:R
- added R? (x3): 1K2, symbol Device:R
- added R? (x3): 680, symbol Device:R
- added R? (x4): 1K, symbol Device:R
- added R?: 10K 1%, symbol Device:R
- added R?: 1210 1%, symbol Device:R
- added R?: 10M, symbol Device:R
- added R?: 100K, symbol Device:R
- added U?: MAX3221, symbol Interface_UART:MAX3221
- added X?: 32.768K, 4SOJ, symbol TrackerAVL:CRYSTAL_4Pin_Mini_GND
- added X?: 12MHz, 4-SMD,_No_Lead_(DFN,_LCC), symbol TrackerAVL:SMD_Sealing_Glass_Crystal
Connections:
- net labels added: +3.3VADC, ADC0_1, ADC0_2, ADC0_3, ADC0_4, GPIO0, GPIO1, GPIO2, GPIO3, GPIO4, GPIO5, GPIO6, IBUTTON, IGN, LED1, LED2, LED3, RESET, RS232_RXD, RS232_TXD, SPI_SCK, TCK, TDI, TDO, TEC1, TEC2, TEC3, TEC4, TMS, U2_RXD, U2_TXD, U3_RX, U3_TX, VBAT, nRESET
- net labels removed: UART_RX, UART_TX
- wire segments 35 -> 401
- no-connect marks 62 -> 87
Other:
- note added: "CAN_RD"
- note added: "CAN_TD"
- note added: "Cada cap lo más cerca posible del pin de PWR del uC"
- note added: "Circuito de reset"
- note added: "Circuitos osciladores"
- note added: "Conexión de batería\nde backup para RTC"
- note added: "Configurar GPIO con pullup interno"
- note added: "DAC"
- note added: "ENET_CRS_DV"
- note added: "ENET_MDC"
- note added: "ENET_MDIO"
- note added: "ENET_REF_CLK"
- note added: "ENET_RXD0"
- note added: "ENET_RXD1"
- note added: "ENET_TXD0"
- note added: "ENET_TXD1"
- note added: "ENET_TX_EN"
- note added: "Entradas analógicas"
- note added: "Entradas de teclas de consola"
- note added: "Entradas digitales\n(con detección de conexión a masa)"
- note added: "Entradas sensado Tensión de batería (30Vmax)\ny sensado digital Ignición"
- note added: "GPIO7"
- note added: "ISP"
- note added: "Interfaz RS232 p/ configuración por terminal"
- note added: "Interfaz de debug"
- note added: "LCD1"
- note added: "LCD2"
- note added: "LCD3"
- note added: "LCD4"
- note added: "LCD_RS"
- note added: "LCD__EN"
- note added: "LED0_B"
- note added: "LED0_G"
- note added: "LED0_R"
- note added: "LEDs indicadores de estado:\n1. Power-on equipo (rojo)\n2. Estado conexión GSM (azul)\n3. Estado conexión GPS (verde)"
- note added: "Not mounted"
- note added: "RS485_DIR"
- note added: "RS485_RXD"
- note added: "RS485_TXD"
- note added: "Salidas digitales \n(tipo open-drain)"
- note added: "TEC_COL0"
- note added: "TEC_COL1"
- note added: "TEC_COL2"
- note added: "TEC_F0"
- note added: "TEC_F1"
- note added: "TEC_F2"
- note added: "TEC_F3"
- note added: "USB_DM"
- note added: "USB_DP"
- note added: "USB_ID"
- note added: "USB_PPWR"
- note added: "USB_PWR_FAULT"
- note added: "USB_VBUS"
- note added: "WAKEUP0"
- note removed: "LEDS\n"

Commit message: Cambios en sch
Parts:
- removed C? (x6): 100nF, symbol Device:C
- removed D? (x3): BZT52C36, Diode_SMD:D_SOD-123, symbol Diode:BZT52Bxx
- removed D? (x7): PESD5V0L1UA, Diode_THT:D_DO-201AE_P15.24mm_Horizontal, symbol Diode:1.5KExxA
- removed Q? (x3): 2N7002P, Package_TO_SOT_SMD:SOT-23, symbol Transistor_FET:2N7002
- removed Q?: DTC043ZEBTL, symbol Transistor_BJT:DTC143Z
- removed R? (x3): 10K, symbol Device:R
- removed R? (x3): 1K2, symbol Device:R
- removed R?: 10K 1%, symbol Device:R
- removed R?: 1210 1%, symbol Device:R
- added JP202, JP203: SolderJumper_2_Open, Jumper:SolderJumper-2_P1.3mm_Open_Pad1.0x1.5mm, symbol Jumper:SolderJumper_2_Open
- added R211: 10K, symbol Device:R
- added U203: STS8C5H30L, Libreria_EDU_CIAA_NXP:SOIC-8, symbol EquipoAVL:IRF7105
- gave numbers to parts that had none: 60
Connections:
- net labels added: GPIO7, MPU_INT, PERST, PWR_MDM, SLEEP_MDM, SPI_CS1
- net labels removed: SPI_MISO
- wire segments 401 -> 319
Other:
- note added: "Control de SLEEP MODE\ndel módulo UC20"
- note added: "Lógica de ON/OFF módulo UC20"
- note added: "SPI_MISO"
- note added: "Si se opta por secuencia de reset\nmediante señal PERST# y no me-\ndiante PWR_MDM, se deben cor-\ntocircuitear JP202 y JP203, y no \nse deben montar R211 y U203A."
- note removed: "Entradas analógicas"
- note removed: "Entradas digitales\n(con detección de conexión a masa)"
- note removed: "Entradas sensado Tensión de batería (30Vmax)\ny sensado digital Ignición"
- note removed: "GPIO7"
- note removed: "Salidas digitales \n(tipo open-drain)"
- moved on the sheet: C201, C202, C203, C204, C205, C206, C207, C208, C209, C210, C211, C212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

Commit message: Cambios en sch
Parts:
- X201: footprint 4-SMD,_No_Lead_(DFN,_LCC) -> (none)
- X202: footprint 4SOJ -> (none)
- renumbered U202 to U201, U201 to U202
Connections:
- net labels added: BUFFER_OE, LED0_G, LED0_R
- no-connect marks 87 -> 85
Other:
- note removed: "LED0_G"
- note removed: "LED0_R"

Commit message: Cambios en sch
Parts:
- added D204: 1N4148, symbol TrackerAVL:DIODE
- U202: symbol TrackerAVL:LPC4337JBD144 -> edu-ciaa-nxp:LPC4337JBD144
Connections:
- net labels added: BUZZER, DISPLAY_MODE, LED0_B, RESET_DBG
- net labels removed: RESET
- wire segments 319 -> 324
- no-connect marks 85 -> 84
Other:
- note added: "Control de SLEEP MODE del módulo UC20"
- note added: "Selección de bus I2C o SPI del display"
- note added: "Señal de interrupción del MPU"
- note removed: "Control de SLEEP MODE\ndel módulo UC20"
- note removed: "LED0_B"
Changed lines of the file:
@@
 NoConn ~ 6700 3900
 NoConn ~ 6700 4000
-NoConn ~ 6700 4950
 NoConn ~ 6700 5250
 NoConn ~ 6700 5350
@@
 RTCX1
 $Comp
-L TrackerAVL:LPC4337JBD144 U202
+L edu-ciaa-nxp:LPC4337JBD144 U202
 U 1 1 5BA579FD
 P 7650 6700
@@
 Text Notes 8200 10500 0    79   ~ 16
 Not mounted
-Text Notes 6200 4950 0    50   ~ 0
-LED0_B
-Wire Notes Line
-	6650 4950 6200 4950
 Text Notes 6100 4600 0    50   ~ 0
 ENET_TXD1
@@
 	2200 1500 2200 1600
 Connection ~ 2200 1600
-Text Label 3350 1400 2    50   ~ 0
+Text Label 3450 1400 2    50   ~ 0
 TMS
-Text Label 3350 1500 2    50   ~ 0
+Text Label 3450 1500 2    50   ~ 0
 TCK
-Text Label 3350 1700 2    50   ~ 0
+Text Label 3450 1700 2    50   ~ 0
 TDI
-Text Label 3350 1800 2    50   ~ 0
-RESET
-Text Label 3350 1600 2    50   ~ 0
+Text Label 3450 1800 2    50   ~ 0
+RESET_DBG
+Text Label 3450 1600 2    50   ~ 0
 TDO
-Wire Wire Line
-	3100 1400 3350 1400
-Wire Wire Line
-	3100 1500 3350 1500
-Wire Wire Line
-	3100 1600 3350 1600
-Wire Wire Line
-	3100 1700 3350 1700
-Wire Wire Line
-	3100 1800 3350 1800
 Text HLabel 10000 8200 2    50   Input ~ 0
 AN_IN_1
@@
 Wire Wire Line
 	2600 8150 2600 8250
-Wire Wire Line
-	2600 8250 2100 8250
-Text Label 2100 8250 0    50   ~ 0
+Text Label 1300 8250 0    50   ~ 0
 nRESET
 $Comp
@@
 Wire Wire Line
 	6100 5750 6700 5750
-Text Notes 4450 5750 0    59   ~ 0
-Control de SLEEP MODE\ndel módulo UC20
-Wire Notes Line
-	5550 5750 4450 5750
+Text Notes 3650 5750 0    59   ~ 0
+Control de SLEEP MODE del módulo UC20
 Text HLabel 6100 5850 0    50   Input ~ 0
 MPU_INT
@@
 Text Label 6200 4850 0    50   ~ 0
 LED0_G
+Text HLabel 6100 5950 0    50   Output ~ 0
+DISPLAY_MODE
+Text Notes 3650 5950 0    59   ~ 0
+Selección de bus I2C o SPI del display
+Wire Notes Line
+	3650 5750 5550 5750
+Wire Notes Line
+	3650 5950 5450 5950
+Text Notes 3650 5850 0    59   ~ 0
+Señal de interrupción del MPU
+Wire Notes Line
+	3650 5850 5450 5850
+Text HLabel 6100 4950 0    50   Output ~ 0
+BUZZER
+Wire Wire Line
+	6100 4950 6700 4950
+Text Label 6200 4950 0    50   ~ 0
+LED0_B
+$Comp
+L TrackerAVL:DIODE D204
+U 1 1 5BE8D671
+P 1850 8000
+F 0 "D204" V 1888 7922 40  0000 R CNN
+F 1 "1N4148" V 1812 7922 40  0000 R CNN
+F 2 "" H 1850 8000 60  0000 C CNN
+F 3 "" H 1850 8000 60  0000 C CNN
+	1    1850 8000
+	0    -1   -1   0
+$EndComp
+Wire Wire Line
+	1850 7800 1850 7750
+Text Label 1300 7750 0    50   ~ 0
+RESET_DBG
+Wire Wire Line
+	1300 8250 1850 8250
+Wire Wire Line
+	1850 8200 1850 8250
+Connection ~ 1850 8250
+Wire Wire Line
+	1850 8250 2600 8250
+Wire Wire Line
+	1300 7750 1850 7750
+Wire Wire Line
+	3100 1800 3450 1800
+Wire Wire Line
+	3100 1400 3450 1400
+Wire Wire Line
+	3100 1500 3450 1500
+Wire Wire Line
+	3100 1600 3450 1600
+Wire Wire Line
+	3100 1700 3450 1700
 $EndSCHEMATC

Commit message: Cambios en sch
Changed lines of the file:
@@
 Wire Wire Line
 	3100 1700 3450 1700
+$Comp
+L power:PWR_FLAG #FLG0102
+U 1 1 5BDAFC0B
+P 14500 5125
+F 0 "#FLG0102" H 14500 5200 50  0001 C CNN
+F 1 "PWR_FLAG" H 14500 5299 50  0000 C CNN
+F 2 "" H 14500 5125 50  0001 C CNN
+F 3 "~" H 14500 5125 50  0001 C CNN
+	1    14500 5125
+	1    0    0    -1
+$EndComp
+Wire Wire Line
+	14500 5125 14500 5200
 $EndSCHEMATC
