File: TrackerAVL/cpu.sch (KiCad schematic (older format))
At the start: 66 parts, among them P201 uC_debug, Q201 DTC043ZEBTL, Q202 DTC043ZEBTL, Q203 DTC043ZEBTL, U201 MAX3221, U202 LPC4337JBD144, U203 STS8C5H30L, X201 12MHz, X202 32.768K

Commit message: Cambios en sch
Parts:
- C201, C202, C203, C204, C205, C206, C207, C208, C209, C210, C211, C212, C213, C214, C215, C216, C217, C218, C219, C220, C221, C222, C223, C224, C225, C227, C228, C229, C230: footprint (none) -> Capacitor_SMD:C_0805_2012Metric_Pad1.15x1.40mm_HandSolder
- C226: value 10uF -> 10uF 10V; footprint (none) -> Capacitor_SMD:C_1206_3216Metric_Pad1.42x1.75mm_HandSolder
- D201, D202, D203: footprint (none) -> LED_SMD:LED_0805_2012Metric_Pad1.15x1.40mm_HandSolder
- D204: footprint (none) -> Diode_SMD:D_SOD-123
- FB201, FB202: footprint (none) -> Inductor_SMD:L_0805_2012Metric_Pad1.15x1.40mm_HandSolder
- JP201: footprint (none) -> Connector_PinHeader_2.54mm:PinHeader_1x02_P2.54mm_Vertical
- P201: footprint (none) -> Libreria_EDU_CIAA_NXP:Pin_Array_5x2_1.27mm_SMD
- R201, R202, R203, R204, R205, R206, R207, R208, R209, R210, R211, R212, R213, R214, R215, R216, R217, R218: footprint (none) -> Resistor_SMD:R_0805_2012Metric_Pad1.15x1.40mm_HandSolder
- U201: footprint (none) -> Package_SO:SSOP-16_5.3x6.2mm_P0.65mm
- U202: footprint (none) -> Libreria_EDU_CIAA_NXP:LQFP144-M05
- U203: footprint Libreria_EDU_CIAA_NXP:SOIC-8 -> Package_SO:SOIC-8_3.9x4.9mm_P1.27mm
- X201: footprint (none) -> Libreria_EDU_CIAA_NXP:FA238V-XTAL
- X202: footprint (none) -> EquipoAVL:32.768-XTAL-SMD

Commit message: EquipoAVL-vRaptor1.0 sch-finalizado
Parts:
- Q201, Q202, Q203: footprint (none) -> EquipoAVL:SOT-523_(SOT-416)
Changed lines of the file:
@@
 F 0 "Q201" H 12487 2846 50  0000 L CNN
 F 1 "DTC043ZEBTL" H 12487 2755 50  0000 L CNN
-F 2 "" H 12300 2800 50  0001 L CNN
+F 2 "EquipoAVL:SOT-523_(SOT-416)" H 12300 2800 50  0001 L CNN
 F 3 "" H 12300 2800 50  0001 L CNN
 	1    12300 2800
@@
 F 0 "Q202" H 13887 2846 50  0000 L CNN
 F 1 "DTC043ZEBTL" H 13887 2755 50  0000 L CNN
-F 2 "" H 13700 2800 50  0001 L CNN
+F 2 "EquipoAVL:SOT-523_(SOT-416)" H 13700 2800 50  0001 L CNN
 F 3 "" H 13700 2800 50  0001 L CNN
 	1    13700 2800
@@
 F 0 "Q203" H 15287 2846 50  0000 L CNN
 F 1 "DTC043ZEBTL" H 15287 2755 50  0000 L CNN
-F 2 "" H 15100 2800 50  0001 L CNN
+F 2 "EquipoAVL:SOT-523_(SOT-416)" H 15100 2800 50  0001 L CNN
 F 3 "" H 15100 2800 50  0001 L CNN
 	1    15100 2800

Commit message: Cambios en pcb
Parts:
- removed X202: 32.768K, EquipoAVL:32.768-XTAL-SMD, symbol TrackerAVL:CRYSTAL_4Pin_Mini_GND
- added X202: 32.768K, EquipoAVL:32.768-XTAL-SMD, symbol Device:Crystal
Connections:
- no-connect marks 84 -> 82
Changed lines of the file:
@@
 	6650 8150 6200 8150
-$Comp
-L TrackerAVL:CRYSTAL_4Pin_Mini_GND X202
-U 1 1 5C75239A
-P 3800 6450
-F 0 "X202" V 3846 6349 50  0000 R CNN
-F 1 "32.768K" V 3755 6349 50  0000 R CNN
-F 2 "EquipoAVL:32.768-XTAL-SMD" H 3800 6450 60  0001 C CNN
-F 3 "" H 3800 6450 60  0000 C CNN
-F 4 "535-9166-1-ND" H 4300 6850 60  0001 C CNN "Digikey/Mouser"
-F 5 "Abracon Corporation" H 4000 6550 60  0001 C CNN "Fabricante"
-F 6 "ABS25-32.768KHZ-T" H 4100 6650 60  0001 C CNN "Nro parte"
-F 7 "CRYSTAL 32.768KHZ 12.5PF" H 4000 6350 60  0001 C CNN "Descripcion"
-	1    3800 6450
-	0    -1   -1   0
-$EndComp
-NoConn ~ 3650 6400
-NoConn ~ 3650 6500
 $Comp
 L Device:C C208
@@
 Wire Wire Line
 	14500 5125 14500 5200
+$Comp
+L Device:Crystal X202
+U 1 1 5BD9F233
+P 3800 6450
+F 0 "X202" V 3754 6581 50  0000 L CNN
+F 1 "32.768K" V 3845 6581 50  0000 L CNN
+F 2 "EquipoAVL:32.768-XTAL-SMD" H 3800 6450 50  0001 C CNN
+F 3 "~" H 3800 6450 50  0001 C CNN
+	1    3800 6450
+	0    1    1    0
+$EndComp
 $EndSCHEMATC

Commit message: Cambios en pcb
Connections:
- net DISPLAY_MODE: now also U202.96 (P2_7); no longer Q203.1 (B), U202.106 (P2_12)
- net MPU_INT: now also U202.95 (P2_6); no longer Q202.1 (B), U202.105 (P2_11)
- net RS232_RXD: no longer U202.88 (P2_4)
- net RS232_TXD: no longer U202.87 (P2_3)
- net SLEEP_MDM: now also U202.91 (P2_5); no longer Q201.1 (B), U202.104 (P2_10)
- new net LED1: Q201.1 (B), U202.104 (P2_10)
- new net LED2: Q202.1 (B), U202.105 (P2_11)
- new net LED3: Q203.1 (B), U202.106 (P2_12)
- new net U3_RX: U202.88 (P2_4)
- new net U3_TX: U202.87 (P2_3)
- no-connect marks 82 -> 79
Other:
- note added: "ADC0_1"
- note added: "ADC0_2"
- note added: "ADC0_3"
- note added: "ADC0_4"
- note added: "GPIO0"
- note added: "GPIO1"
- note added: "GPIO2"
- note added: "GPIO3"
- note added: "GPIO4"
- note added: "GPIO5"
- note added: "GPIO6"
- note added: "GPIO8"
- note added: "LED0_B"
- note added: "LED0_G"
- note added: "LED0_R"
- note added: "RS232_RXD"
- note added: "RS232_TXD"
Changed lines of the file:
@@
 NoConn ~ 6700 3900
 NoConn ~ 6700 4000
-NoConn ~ 6700 5250
-NoConn ~ 6700 5350
-NoConn ~ 6700 5450
 NoConn ~ 6700 5550
 NoConn ~ 6700 5650
@@
 Text HLabel 10000 4100 2    50   BiDi ~ 0
 IBUTTON
-Text Label 9900 4100 2    50   ~ 0
-GPIO8
 Text Notes 12100 4100 2    59   ~ 0
 Configurar GPIO con pullup interno
-Text Label 9900 3800 2    50   ~ 0
-GPIO5
-Text Label 9900 3700 2    50   ~ 0
-GPIO4
-Text Label 9900 3600 2    50   ~ 0
-GPIO3
 NoConn ~ 9400 3500
-Text Label 9900 3400 2    50   ~ 0
-GPIO2
-Text Label 9900 3300 2    50   ~ 0
-GPIO1
-Text Label 9900 3000 2    50   ~ 0
-GPIO0
 Text Notes 12100 3600 2    59   ~ 0
 Configurar GPIO con pullup interno
@@
 Text Notes 12100 3800 2    59   ~ 0
 Configurar GPIO con pullup interno
-Text Label 9900 8200 2    50   ~ 0
-ADC0_2
-Text Label 9900 8100 2    50   ~ 0
-ADC0_1
-Text Label 9900 8300 2    50   ~ 0
-ADC0_3
 Wire Wire Line
 	9400 4100 10000 4100
@@
 Text HLabel 10000 8400 2    50   Input ~ 0
 VBAT
-Text Label 9900 8400 2    50   ~ 0
-ADC0_4
-Text Label 9900 3900 2    50   ~ 0
-GPIO6
 Text Notes 12100 3900 2    59   ~ 0
 Configurar GPIO con pullup interno
-Text Label 6200 5050 0    50   ~ 0
-RS232_TXD
-Text Label 6200 5150 0    50   ~ 0
-RS232_RXD
 Text Notes 6200 6300 0    50   ~ 0
 CAN_RD
@@
 Wire Wire Line
 	9400 4000 9900 4000
-Text Label 9900 4000 2    50   ~ 0
-GPIO7
 Text Label 12500 5100 0    50   ~ 0
 GPIO7
@@
 Wire Notes Line
 	11750 6350 14200 6350
-Text HLabel 6100 5750 0    50   Output ~ 0
-SLEEP_MDM
-Wire Wire Line
-	6100 5750 6700 5750
-Text Notes 3650 5750 0    59   ~ 0
+Text Notes 3650 5250 0    59   ~ 0
 Control de SLEEP MODE del módulo UC20
-Text HLabel 6100 5850 0    50   Input ~ 0
-MPU_INT
-Wire Wire Line
-	6100 5850 6700 5850
 Wire Wire Line
 	6100 3000 6700 3000
@@
 Text HLabel 10000 3000 2    50   Output ~ 0
 SPI_CS1
-Wire Wire Line
-	6100 5950 6700 5950
-Text Label 6200 4750 0    50   ~ 0
-LED0_R
 Text HLabel 6100 4750 0    50   Output ~ 0
 BUFFER_OE
@@
 Wire Wire Line
 	6100 4850 6700 4850
-Text Label 6200 4850 0    50   ~ 0
-LED0_G
-Text HLabel 6100 5950 0    50   Output ~ 0
-DISPLAY_MODE
-Text Notes 3650 5950 0    59   ~ 0
+Text Notes 3650 5450 0    59   ~ 0
 Selección de bus I2C o SPI del display
 Wire Notes Line
-	3650 5750 5550 5750
-Wire Notes Line
-	3650 5950 5450 5950
-Text Notes 3650 5850 0    59   ~ 0
+	3650 5250 5550 5250
+Wire Notes Line
+	3650 5450 5450 5450
+Text Notes 3650 5350 0    59   ~ 0
 Señal de interrupción del MPU
 Wire Notes Line
-	3650 5850 5450 5850
+	3650 5350 5450 5350
 Text HLabel 6100 4950 0    50   Output ~ 0
 BUZZER
 Wire Wire Line
 	6100 4950 6700 4950
-Text Label 6200 4950 0    50   ~ 0
-LED0_B
 $Comp
 L TrackerAVL:DIODE D204
@@
 	0    1    1    0
 $EndComp
+Text Notes 6200 5050 0    50   ~ 0
+RS232_TXD
+Text Notes 6200 5150 0    50   ~ 0
+RS232_RXD
+Text HLabel 6100 5250 0    50   Output ~ 0
+SLEEP_MDM
+Wire Wire Line
+	6100 5250 6700 5250
+Text HLabel 6100 5350 0    50   Input ~ 0
+MPU_INT
+Wire Wire Line
+	6100 5350 6700 5350
+Wire Wire Line
+	6100 5450 6700 5450
+Text HLabel 6100 5450 0    50   Output ~ 0
+DISPLAY_MODE
+Wire Wire Line
+	6700 5750 6200 5750
+Wire Wire Line
+	6700 5850 6200 5850
+Wire Wire Line
+	6200 5950 6700 5950
+Text Notes 6200 4750 0    50   ~ 0
+LED0_R
+Text Notes 6200 4850 0    50   ~ 0
+LED0_G
+Text Notes 6200 4950 0    50   ~ 0
+LED0_B
+Text Notes 9900 8100 2    50   ~ 0
+ADC0_1
+Text Notes 9900 8200 2    50   ~ 0
+ADC0_2
+Text Notes 9900 8300 2    50   ~ 0
+ADC0_3
+Text Notes 9900 8400 2    50   ~ 0
+ADC0_4
+Text Notes 9900 3000 2    50   ~ 0
+GPIO0
+Text Notes 9900 3300 2    50   ~ 0
+GPIO1
+Text Notes 9900 3400 2    50   ~ 0
+GPIO2
+Text Notes 9900 3600 2    50   ~ 0
+GPIO3
+Text Notes 9900 3700 2    50   ~ 0
+GPIO4
+Text Notes 9900 3800 2    50   ~ 0
+GPIO5
+Text Notes 9900 3900 2    50   ~ 0
+GPIO6
+Text Notes 9900 4100 2    50   ~ 0
+GPIO8
+Text Label 9900 4000 2    50   ~ 0
+GPIO7
 $EndSCHEMATC

Commit message: Cambios en pcb
Parts:
- D204: symbol TrackerAVL:DIODE -> TrackerAVL-rescue:DIODE-TrackerAVL
- FB201, FB202: symbol TrackerAVL:FILTER -> TrackerAVL-rescue:FILTER-TrackerAVL
- P201: symbol TrackerAVL:CONN_5X2 -> TrackerAVL-rescue:CONN_5X2-TrackerAVL
- U202: symbol edu-ciaa-nxp:LPC4337JBD144 -> TrackerAVL-rescue:LPC4337JBD144-edu-ciaa-nxp
- U203: symbol EquipoAVL:IRF7105 -> TrackerAVL-rescue:IRF7105-EquipoAVL
- X201: symbol TrackerAVL:SMD_Sealing_Glass_Crystal -> TrackerAVL-rescue:SMD_Sealing_Glass_Crystal-TrackerAVL
Changed lines of the file:
@@
 RTCX1
 $Comp
-L edu-ciaa-nxp:LPC4337JBD144 U202
+L TrackerAVL-rescue:LPC4337JBD144-edu-ciaa-nxp U202
 U 1 1 5BA579FD
 P 7650 6700
@@
 Circuitos osciladores
 $Comp
-L TrackerAVL:SMD_Sealing_Glass_Crystal X201
+L TrackerAVL-rescue:SMD_Sealing_Glass_Crystal-TrackerAVL X201
 U 1 1 5C804AF8
 P 2000 6450
@@
 	1300 6450 1500 6450
 $Comp
-L TrackerAVL:FILTER FB201
+L TrackerAVL-rescue:FILTER-TrackerAVL FB201
 U 1 1 5C915198
 P 6150 8950
@@
 Not mounted
 $Comp
-L TrackerAVL:FILTER FB202
+L TrackerAVL-rescue:FILTER-TrackerAVL FB202
 U 1 1 5CA81561
 P 8850 10050
@@
 	9400 6250 9900 6250
 $Comp
-L TrackerAVL:CONN_5X2 P201
+L TrackerAVL-rescue:CONN_5X2-TrackerAVL P201
 U 1 1 5C85D5A7
 P 2700 1600
@@
 	12100 4100 10450 4100
 $Comp
-L EquipoAVL:IRF7105 U?
+L TrackerAVL-rescue:IRF7105-EquipoAVL U?
 U 1 1 5C1F8653
 P 13800 5100
@@
 	6100 4950 6700 4950
 $Comp
-L TrackerAVL:DIODE D204
+L TrackerAVL-rescue:DIODE-TrackerAVL D204
 U 1 1 5BE8D671
 P 1850 8000
