File: TrackerAVL/uc20_pcie.sch (KiCad schematic (older format))
At the start: 6 parts

Commit message: Cambios en sch
Parts:
- gave numbers to parts that had none: 6
Other:
- moved on the sheet: R703, R704, R705
Changed lines of the file:
@@
 $Descr A4 11693 8268
 encoding utf-8
-Sheet 8 8
+Sheet 7 8
 Title ""
 Date ""
@@
 $EndDescr
 $Comp
-L mpcie:MPCIE-Socket U?
+L mpcie:MPCIE-Socket U701
 U 1 1 5BA7E0EE
 P 5900 3250
-F 0 "U?" H 5900 4793 60  0000 C CNN
+F 0 "U701" H 5900 4793 60  0000 C CNN
 F 1 "MPCIE-Socket" H 5900 4687 60  0000 C CNN
 F 2 "mpcie:mpcie-socket" H 5900 4581 60  0000 C CNN
@@
 NoConn ~ 6550 2400
 $Comp
-L power:GND #PWR?
+L power:GND #PWR0701
 U 1 1 5BA8AA56
 P 1200 1500
-F 0 "#PWR?" H 1200 1250 50  0001 C CNN
+F 0 "#PWR0701" H 1200 1250 50  0001 C CNN
 F 1 "GND" H 1205 1327 50  0000 C CNN
 F 2 "" H 1200 1500 50  0001 C CNN
@@
 	4350 4700 5250 4700
 $Comp
-L Device:R R?
+L Device:R R701
 U 1 1 5BAB0D64
 P 9550 1400
-F 0 "R?" H 9620 1446 50  0000 L CNN
+F 0 "R701" H 9620 1446 50  0000 L CNN
 F 1 "10K" H 9620 1355 50  0000 L CNN
 F 2 "" V 9480 1400 50  0001 C CNN
@@
 $EndComp
 $Comp
-L Device:R R?
+L Device:R R703
 U 1 1 5BAB0EDA
-P 9850 1400
-F 0 "R?" H 9920 1446 50  0000 L CNN
-F 1 "10K" H 9920 1355 50  0000 L CNN
-F 2 "" V 9780 1400 50  0001 C CNN
-F 3 "~" H 9850 1400 50  0001 C CNN
-	1    9850 1400
-	1    0    0    -1
-$EndComp
-$Comp
-L Device:R R?
+P 9900 1400
+F 0 "R703" H 9970 1446 50  0000 L CNN
+F 1 "10K" H 9970 1355 50  0000 L CNN
+F 2 "" V 9830 1400 50  0001 C CNN
+F 3 "~" H 9900 1400 50  0001 C CNN
+	1    9900 1400
+	1    0    0    -1
+$EndComp
+$Comp
+L Device:R R705
 U 1 1 5BAB0F0C
-P 10150 1400
-F 0 "R?" H 10220 1446 50  0000 L CNN
-F 1 "10K" H 10220 1355 50  0000 L CNN
-F 2 "" V 10080 1400 50  0001 C CNN
-F 3 "~" H 10150 1400 50  0001 C CNN
-	1    10150 1400
+P 10250 1400
+F 0 "R705" H 10320 1446 50  0000 L CNN
+F 1 "10K" H 10320 1355 50  0000 L CNN
+F 2 "" V 10180 1400 50  0001 C CNN
+F 3 "~" H 10250 1400 50  0001 C CNN
+	1    10250 1400
 	1    0    0    -1
 $EndComp
@@
 Wire Wire Line
 	9550 1600 9050 1600
-Wire Wire Line
-	9850 1550 9850 1700
-Wire Wire Line
-	10150 1550 10150 1800
 Text Label 9050 1600 0    50   ~ 0
 WAKE
@@
 Text Label 9050 1800 0    50   ~ 0
 PERST
-Wire Wire Line
-	10150 1150 10150 1250
-Wire Wire Line
-	9850 1150 9850 1250
 Wire Wire Line
 	9550 1150 9550 1250
@@
 I2C_SCL
 $Comp
-L Device:R R?
+L Device:R R702
 U 1 1 5BAC7583
 P 9550 2500
-F 0 "R?" H 9620 2546 50  0000 L CNN
+F 0 "R702" H 9620 2546 50  0000 L CNN
 F 1 "10K" H 9620 2455 50  0000 L CNN
 F 2 "" V 9480 2500 50  0001 C CNN
@@
 $EndComp
 $Comp
-L Device:R R?
+L Device:R R704
 U 1 1 5BAC758A
-P 9850 2500
-F 0 "R?" H 9920 2546 50  0000 L CNN
-F 1 "10K" H 9920 2455 50  0000 L CNN
-F 2 "" V 9780 2500 50  0001 C CNN
-F 3 "~" H 9850 2500 50  0001 C CNN
-	1    9850 2500
+P 9900 2500
+F 0 "R704" H 9970 2546 50  0000 L CNN
+F 1 "10K" H 9970 2455 50  0000 L CNN
+F 2 "" V 9830 2500 50  0001 C CNN
+F 3 "~" H 9900 2500 50  0001 C CNN
+	1    9900 2500
 	1    0    0    -1
 $EndComp
@@
 Wire Wire Line
 	9550 2700 9050 2700
-Wire Wire Line
-	9850 2650 9850 2800
 Text Label 9050 2800 0    50   ~ 0
 I2C_SCL
-Wire Wire Line
-	9850 2250 9850 2350
 Wire Wire Line
 	9550 2250 9550 2350
@@
 	8950 2850 9650 2850
 $Comp
-L power:+1V8 #PWR?
+L power:+1V8 #PWR0703
 U 1 1 5BAD062F
 P 9050 2250
-F 0 "#PWR?" H 9050 2100 50  0001 C CNN
+F 0 "#PWR0703" H 9050 2100 50  0001 C CNN
 F 1 "+1V8" H 9200 2300 50  0000 C CNN
 F 2 "" H 9050 2250 50  0001 C CNN
@@
 	8950 1000 8950 1850
 $Comp
-L power:+3.3V #PWR?
+L power:+3.3V #PWR0702
 U 1 1 5BAD7224
 P 9050 1150
-F 0 "#PWR?" H 9050 1000 50  0001 C CNN
+F 0 "#PWR0702" H 9050 1000 50  0001 C CNN
 F 1 "+3.3V" H 9200 1200 50  0000 C CNN
 F 2 "" H 9050 1150 50  0001 C CNN
@@
 	1    0    0    -1
 $EndComp
-Wire Wire Line
-	9850 1150 10150 1150
-Connection ~ 9850 1150
-Wire Wire Line
-	9550 1150 9850 1150
 Connection ~ 9550 1150
-Wire Wire Line
-	9050 1800 10150 1800
-Wire Wire Line
-	9050 1700 9850 1700
-Wire Wire Line
-	9550 2250 9850 2250
 Connection ~ 9550 2250
-Wire Wire Line
-	9050 2800 9850 2800
 Text Label 9050 2700 0    50   ~ 0
 I2C_SDA
@@
 Text Notes 6850 4300 0    118  ~ 0
 FALTA DEFINIR
+Wire Wire Line
+	10250 1150 10250 1250
+Wire Wire Line
+	9550 1150 9900 1150
+Wire Wire Line
+	10250 1550 10250 1800
+Wire Wire Line
+	9050 1800 10250 1800
+Wire Wire Line
+	9900 1550 9900 1700
+Wire Wire Line
+	9050 1700 9900 1700
+Wire Wire Line
+	9900 1250 9900 1150
+Connection ~ 9900 1150
+Wire Wire Line
+	9900 1150 10250 1150
+Wire Wire Line
+	9900 2250 9900 2350
+Wire Wire Line
+	9550 2250 9900 2250
+Wire Wire Line
+	9900 2650 9900 2800
+Wire Wire Line
+	9050 2800 9900 2800
 $EndSCHEMATC

Commit message: Cambios en sch y adición de documentación
Connections:
- no-connect marks 18 -> 22
Other:
- note added: "SIM Holder ya está sobre\nel módulo UC20, por lo\ntanto estas salidas no se\nconectan"
- note removed: "FALTA DEFINIR"
Changed lines of the file:
@@
 Comment4 ""
 $EndDescr
-$Comp
-L mpcie:MPCIE-Socket U701
-U 1 1 5BA7E0EE
-P 5900 3250
-F 0 "U701" H 5900 4793 60  0000 C CNN
-F 1 "MPCIE-Socket" H 5900 4687 60  0000 C CNN
-F 2 "mpcie:mpcie-socket" H 5900 4581 60  0000 C CNN
-F 3 "" H 6000 2250 60  0000 C CNN
-	1    5900 3250
-	1    0    0    -1
-$EndComp
 Text HLabel 4350 4700 0    50   Output ~ 0
 WAKE_HOST
@@
 Text Notes 7650 3500 0    59   ~ 0
 Señales de control
-Text Notes 6850 4300 0    118  ~ 0
-FALTA DEFINIR
 Wire Wire Line
 	10250 1150 10250 1250
@@
 Wire Wire Line
 	9050 2800 9900 2800
+$Comp
+L mpcie:MPCIE-Socket U701
+U 1 1 5BA7E0EE
+P 5900 3250
+F 0 "U701" H 5900 4793 60  0000 C CNN
+F 1 "MPCIE-Socket" H 5900 4687 60  0000 C CNN
+F 2 "mpcie:mpcie-socket" H 5900 4581 60  0000 C CNN
+F 3 "" H 6000 2250 60  0000 C CNN
+	1    5900 3250
+	1    0    0    -1
+$EndComp
+NoConn ~ 6550 4100
+NoConn ~ 6550 4200
+NoConn ~ 6550 4300
+NoConn ~ 6550 4400
+Text Notes 7300 4350 0    59   ~ 0
+SIM Holder ya está sobre\nel módulo UC20, por lo\ntanto estas salidas no se\nconectan
+Wire Notes Line
+	6600 3950 8500 3950
+Wire Notes Line
+	6600 4500 8500 4500
+Wire Notes Line
+	8500 3950 8500 4500
 $EndSCHEMATC

Commit message: Cambios en sch
Connections:
- net W_DISABLE: no longer U701.20 (~W_DISABLE)
- net WAKE_HOST: no longer names the net of U701.1 (~WAKE)
- net WAKE_HOST: no longer R701.2
- new net WAKE: R701.2
- no-connect marks 22 -> 24
Other:
- note added: "Señal para despertar al uC (no usado)"
- note added: "W_DISABLE"
- note removed: "Señal para despertar al uC"
Changed lines of the file:
@@
 $Descr A4 11693 8268
 encoding utf-8
-Sheet 7 7
+Sheet 7 8
 Title ""
 Date ""
@@
 Comment4 ""
 $EndDescr
-Text HLabel 4350 4700 0    50   Output ~ 0
-WAKE_HOST
 NoConn ~ 5250 4600
 NoConn ~ 5250 4500
@@
 Text Notes 3100 4000 0    59   ~ 0
 Comunicación serial
-Text Notes 3100 4600 0    59   ~ 0
-Señal para despertar al uC
+Text Notes 3100 4700 0    59   ~ 0
+Señal para despertar al uC (no usado)
 Wire Wire Line
 	6550 2100 7050 2100
@@
 	5250 2100 4350 2100
 Wire Wire Line
-	6550 3700 7450 3700
-Wire Wire Line
 	6550 3600 7450 3600
-Text HLabel 7450 3700 2    50   Input ~ 0
-W_DISABLE
 Text HLabel 7450 3600 2    50   Input ~ 0
 PERST
 Text Label 6700 3600 0    50   ~ 0
 PERST
-Text Label 6700 3700 0    50   ~ 0
-W_DISABLE
-Text Label 4750 4700 0    50   ~ 0
-WAKE
-Wire Wire Line
-	4350 4700 5250 4700
 $Comp
 L Device:R R701
@@
 NoConn ~ 6550 2900
 Wire Notes Line
-	4350 4750 3100 4750
-Wire Notes Line
-	3100 4750 3100 4600
-Wire Notes Line
-	3100 4600 4350 4600
-Wire Notes Line
 	4350 4250 3100 4250
 Wire Notes Line
@@
 Wire Notes Line
 	8500 3950 8500 4500
+NoConn ~ 5250 4700
+Wire Notes Line
+	3100 4700 5200 4700
+NoConn ~ 6550 3700
+Wire Notes Line
+	6600 3700 7050 3700
+Text Notes 7050 3700 2    50   ~ 0
+W_DISABLE
 $EndSCHEMATC

Commit message: Cambios en sch
Parts:
- removed R701, R705: 10K, symbol Device:R
- renumbered R703 to R601, R702 to R602, R704 to R603, U701 to U601
Connections:
- net W_DISABLE: now also U601.20 (~W_DISABLE)
- no-connect marks 24 -> 23
Other:
- note removed: "W_DISABLE"
- moved on the sheet: R601
Changed lines of the file:
@@
 $Descr A4 11693 8268
 encoding utf-8
-Sheet 7 8
+Sheet 6 8
 Title ""
 Date ""
@@
 NoConn ~ 6550 2400
 $Comp
-L power:GND #PWR0701
+L power:GND #PWR0601
 U 1 1 5BA8AA56
 P 1200 1500
-F 0 "#PWR0701" H 1200 1250 50  0001 C CNN
+F 0 "#PWR0601" H 1200 1250 50  0001 C CNN
 F 1 "GND" H 1205 1327 50  0000 C CNN
 F 2 "" H 1200 1500 50  0001 C CNN
@@
 Text Notes 3100 4000 0    59   ~ 0
 Comunicación serial
-Text Notes 3100 4700 0    59   ~ 0
-Señal para despertar al uC (no usado)
 Wire Wire Line
 	6550 2100 7050 2100
@@
 PERST
 $Comp
-L Device:R R701
-U 1 1 5BAB0D64
-P 9550 1400
-F 0 "R701" H 9620 1446 50  0000 L CNN
-F 1 "10K" H 9620 1355 50  0000 L CNN
-F 2 "" V 9480 1400 50  0001 C CNN
-F 3 "~" H 9550 1400 50  0001 C CNN
-	1    9550 1400
-	1    0    0    -1
-$EndComp
-$Comp
-L Device:R R703
+L Device:R R601
 U 1 1 5BAB0EDA
-P 9900 1400
-F 0 "R703" H 9970 1446 50  0000 L CNN
-F 1 "10K" H 9970 1355 50  0000 L CNN
-F 2 "" V 9830 1400 50  0001 C CNN
-F 3 "~" H 9900 1400 50  0001 C CNN
-	1    9900 1400
-	1    0    0    -1
-$EndComp
-$Comp
-L Device:R R705
-U 1 1 5BAB0F0C
-P 10250 1400
-F 0 "R705" H 10320 1446 50  0000 L CNN
-F 1 "10K" H 10320 1355 50  0000 L CNN
-F 2 "" V 10180 1400 50  0001 C CNN
-F 3 "~" H 10250 1400 50  0001 C CNN
-	1    10250 1400
-	1    0    0    -1
-$EndComp
-Wire Wire Line
-	9050 1150 9550 1150
-Wire Wire Line
-	9550 1550 9550 1600
-Wire Wire Line
-	9550 1600 9050 1600
-Text Label 9050 1600 0    50   ~ 0
-WAKE
+P 9500 1400
+F 0 "R601" H 9570 1446 50  0000 L CNN
+F 1 "10K" H 9570 1355 50  0000 L CNN
+F 2 "" V 9430 1400 50  0001 C CNN
+F 3 "~" H 9500 1400 50  0001 C CNN
+	1    9500 1400
+	1    0    0    -1
+$EndComp
 Text Label 9050 1700 0    50   ~ 0
 W_DISABLE
-Text Label 9050 1800 0    50   ~ 0
-PERST
-Wire Wire Line
-	9550 1150 9550 1250
-Text Notes 8950 1000 0    59   ~ 0
+Text Notes 8950 950  0    59   ~ 0
 Pull-ups +3.3V
 NoConn ~ 6550 3300
@@
 I2C_SCL
 $Comp
-L Device:R R702
+L Device:R R602
 U 1 1 5BAC7583
 P 9550 2500
-F 0 "R702" H 9620 2546 50  0000 L CNN
+F 0 "R602" H 9620 2546 50  0000 L CNN
 F 1 "10K" H 9620 2455 50  0000 L CNN
 F 2 "" V 9480 2500 50  0001 C CNN
@@
 $EndComp
 $Comp
-L Device:R R704
+L Device:R R603
 U 1 1 5BAC758A
 P 9900 2500
-F 0 "R704" H 9970 2546 50  0000 L CNN
+F 0 "R603" H 9970 2546 50  0000 L CNN
 F 1 "10K" H 9970 2455 50  0000 L CNN
 F 2 "" V 9830 2500 50  0001 C CNN
@@
 $EndComp
 Wire Wire Line
-	9050 2250 9550 2250
-Wire Wire Line
 	9550 2650 9550 2700
 Wire Wire Line
@@
 Wire Wire Line
 	9550 2250 9550 2350
-Text Notes 8950 2100 0    59   ~ 0
+Text Notes 8950 2050 0    59   ~ 0
 Pull-ups +1.8V
 Wire Notes Line
-	8950 1000 9650 1000
-Wire Notes Line
-	8950 1850 9650 1850
-Wire Notes Line
-	8950 2100 9650 2100
+	8950 950  9650 950
+Wire Notes Line
+	8950 2050 9650 2050
 Wire Notes Line
 	8950 2850 9650 2850
 $Comp
-L power:+1V8 #PWR0703
+L power:+1V8 #PWR0603
 U 1 1 5BAD062F
-P 9050 2250
-F 0 "#PWR0703" H 9050 2100 50  0001 C CNN
-F 1 "+1V8" H 9200 2300 50  0000 C CNN
-F 2 "" H 9050 2250 50  0001 C CNN
-F 3 "" H 9050 2250 50  0001 C CNN
-	1    9050 2250
-	1    0    0    -1
-$EndComp
-Wire Notes Line
-	8950 1000 8950 1850
-$Comp
-L power:+3.3V #PWR0702
+P 9550 2200
+F 0 "#PWR0603" H 9550 2050 50  0001 C CNN
+F 1 "+1V8" H 9700 2250 50  0000 C CNN
+F 2 "" H 9550 2200 50  0001 C CNN
+F 3 "" H 9550 2200 50  0001 C CNN
+	1    9550 2200
+	1    0    0    -1
+$EndComp
+$Comp
+L power:+3.3V #PWR0602
 U 1 1 5BAD7224
-P 9050 1150
-F 0 "#PWR0702" H 9050 1000 50  0001 C CNN
-F 1 "+3.3V" H 9200 1200 50  0000 C CNN
-F 2 "" H 9050 1150 50  0001 C CNN
-F 3 "" H 9050 1150 50  0001 C CNN
-	1    9050 1150
-	1    0    0    -1
-$EndComp
-Connection ~ 9550 1150
-Connection ~ 9550 2250
+P 9500 1100
+F 0 "#PWR0602" H 9500 950 50  0001 C CNN
+F 1 "+3.3V" H 9650 1150 50  0000 C CNN
+F 2 "" H 9500 1100 50  0001 C CNN
+F 3 "" H 9500 1100 50  0001 C CNN
+	1    9500 1100
+	1    0    0    -1
+$EndComp
 Text Label 9050 2700 0    50   ~ 0
 I2C_SDA
-Wire Notes Line
-	8950 2850 8950 2100
 NoConn ~ 6550 2800
 NoConn ~ 6550 2900
@@
 Señales de control
 Wire Wire Line
-	10250 1150 10250 1250
-Wire Wire Line
-	9550 1150 9900 1150
-Wire Wire Line
-	10250 1550 10250 1800
-Wire Wire Line
-	9050 1800 10250 1800
-Wire Wire Line
-	9900 1550 9900 1700
-Wire Wire Line
-	9050 1700 9900 1700
-Wire Wire Line
-	9900 1250 9900 1150
-Connection ~ 9900 1150
-Wire Wire Line
-	9900 1150 10250 1150
+	9050 1700 9500 1700
 Wire Wire Line
 	9900 2250 9900 2350
@@
 	9050 2800 9900 2800
 $Comp
-L mpcie:MPCIE-Socket U701
+L mpcie:MPCIE-Socket U601
 U 1 1 5BA7E0EE
 P 5900 3250
-F 0 "U701" H 5900 4793 60  0000 C CNN
-F 1 "MPCIE-Socket" H 5900 4687 60  0000 C CNN
-F 2 "mpcie:mpcie-socket" H 5900 4581 60  0000 C CNN
+F 0 "U601" H 5850 4700 60  0000 C CNN
+F 1 "MPCIE-Socket" H 5850 4600 60  0000 C CNN
+F 2 "mpcie:mpcie-socket" H 5900 4581 60  0001 C CNN
 F 3 "" H 6000 2250 60  0000 C CNN
 	1    5900 3250
@@
 Wire Notes Line
 	8500 3950 8500 4500
+Text Label 7050 3700 2    50   ~ 0
+W_DISABLE
+Wire Wire Line
+	7050 3700 6550 3700
 NoConn ~ 5250 4700
 Wire Notes Line
 	3100 4700 5200 4700
-NoConn ~ 6550 3700
-Wire Notes Line
-	6600 3700 7050 3700
-Text Notes 7050 3700 2    50   ~ 0
-W_DISABLE
+Text Notes 3100 4700 0    59   ~ 0
+Señal para despertar al uC (no usado)
+Wire Wire Line
+	9500 1550 9500 1700
+Wire Wire Line
+	9550 2250 9550 2200
+Connection ~ 9550 2250
+Wire Wire Line
+	9500 1100 9500 1250
+Wire Notes Line
+	8950 2050 8950 2850
+Wire Notes Line
+	8950 950  8950 1750
+Wire Notes Line
+	8950 1750 9650 1750
 $EndSCHEMATC

Commit message: Cambios en sch
Parts:
- R601, R602, R603: footprint (none) -> Resistor_SMD:R_0805_2012Metric_Pad1.15x1.40mm_HandSolder
- U601: footprint mpcie:mpcie-socket -> mpcie:mpcie-socket-latch
Changed lines of the file:
@@
 encoding utf-8
 Sheet 6 8
-Title ""
-Date ""
-Rev ""
+Title "Equipo AVL - vRaptor"
+Date "2018-10-30"
+Rev "1.0"
 Comp ""
-Comment1 ""
+Comment1 "Ing. Mauro Moreyra"
 Comment2 ""
 Comment3 ""
@@
 F 0 "R601" H 9570 1446 50  0000 L CNN
 F 1 "10K" H 9570 1355 50  0000 L CNN
-F 2 "" V 9430 1400 50  0001 C CNN
+F 2 "Resistor_SMD:R_0805_2012Metric_Pad1.15x1.40mm_HandSolder" V 9430 1400 50  0001 C CNN
 F 3 "~" H 9500 1400 50  0001 C CNN
 	1    9500 1400
@@
 F 0 "R602" H 9620 2546 50  0000 L CNN
 F 1 "10K" H 9620 2455 50  0000 L CNN
-F 2 "" V 9480 2500 50  0001 C CNN
+F 2 "Resistor_SMD:R_0805_2012Metric_Pad1.15x1.40mm_HandSolder" V 9480 2500 50  0001 C CNN
 F 3 "~" H 9550 2500 50  0001 C CNN
 	1    9550 2500
@@
 F 0 "R603" H 9970 2546 50  0000 L CNN
 F 1 "10K" H 9970 2455 50  0000 L CNN
-F 2 "" V 9830 2500 50  0001 C CNN
+F 2 "Resistor_SMD:R_0805_2012Metric_Pad1.15x1.40mm_HandSolder" V 9830 2500 50  0001 C CNN
 F 3 "~" H 9900 2500 50  0001 C CNN
 	1    9900 2500
@@
 F 0 "U601" H 5850 4700 60  0000 C CNN
 F 1 "MPCIE-Socket" H 5850 4600 60  0000 C CNN
-F 2 "mpcie:mpcie-socket" H 5900 4581 60  0001 C CNN
+F 2 "mpcie:mpcie-socket-latch" H 5900 4581 60  0001 C CNN
 F 3 "" H 6000 2250 60  0000 C CNN
 	1    5900 3250

Commit message: Cambios en pcb
Changed lines of the file:
@@
 Text HLabel 7450 3600 2    50   Input ~ 0
-PERST
-Text Label 6700 3600 0    50   ~ 0
 PERST
 $Comp
