File: TrackerAVL/uc20_pcie.sch (KiCad schematic (older format))
At the start: 4 parts, among them U601 MPCIE-Socket

Commit message: Cambios en pcb
Parts:
- U601: symbol mpcie:MPCIE-Socket -> TrackerAVL-rescue:MPCIE-Socket-mpcie
Changed lines of the file:
@@
 	9050 2800 9900 2800
 $Comp
-L mpcie:MPCIE-Socket U601
+L TrackerAVL-rescue:MPCIE-Socket-mpcie U601
 U 1 1 5BA7E0EE
 P 5900 3250
