File: TrackerAVL/acelerometro.sch (KiCad schematic (older format))
At the start: 0 parts

Commit message: Cambios en sch
Parts:
- added C? (x3): 100nF, symbol Device:C
- added C?: 2.2nF, symbol Device:C
- added U?: MPU-6050, Sensor_Motion:InvenSense_QFN-24_4x4mm_P0.5mm, symbol Sensor_Motion:MPU-6050
Connections:
- new net: C?.1, U?.10 (REGOUT)
- new net: C?.1, U?.20 (CPOUT)
- new net +3V3: C?.1, C?.1, U?.13 (VDD), U?.8 (VDDIO)
- new net GND: C?.2, C?.2, C?.2, C?.2, U?.1 (CLKIN), U?.11 (FSYNC), U?.18 (GND), U?.9 (AD0)
- new net I2C_SCL: U?.23 (SCL)
- new net I2C_SDA: U?.24 (SDA)
- new net INT: U?.12 (INT)
- no-connect marks 0 -> 2
Other:
- note added: "Circuito acelerómetro MPU-6050\nProvee datos de:\n> Acelerómetro\n> Giróscopo\n> Temperatura"
Changed lines of the file:
@@
 Comment4 ""
 $EndDescr
+$Comp
+L Sensor_Motion:MPU-6050 U?
+U 1 1 5DB41454
+P 5700 3200
+F 0 "U?" H 5800 2650 50  0000 C CNN
+F 1 "MPU-6050" H 5400 2650 50  0000 C CNN
+F 2 "Sensor_Motion:InvenSense_QFN-24_4x4mm_P0.5mm" H 5700 2400 50  0001 C CNN
+F 3 "https://store.invensense.com/datasheets/invensense/MPU-6050_DataSheet_V3%204.pdf" H 5700 3050 50  0001 C CNN
+	1    5700 3200
+	1    0    0    -1
+$EndComp
+$Comp
+L Device:C C?
+U 1 1 5DB41F13
+P 5200 2100
+AR Path="/5BA56FC1/5DB41F13" Ref="C?"  Part="1"
+AR Path="/5BA57001/5DB41F13" Ref="C?"  Part="1"
+F 0 "C?" H 5200 2200 39  0000 L CNN
+F 1 "100nF" H 5200 2000 39  0000 L CNN
+F 2 "" H 5238 1950 50  0001 C CNN
+F 3 "~" H 5200 2100 50  0001 C CNN
+	1    5200 2100
+	1    0    0    -1
+$EndComp
+$Comp
+L power:GND #PWR?
+U 1 1 5DB41FBA
+P 5200 2350
+F 0 "#PWR?" H 5200 2100 50  0001 C CNN
+F 1 "GND" H 5205 2177 50  0000 C CNN
+F 2 "" H 5200 2350 50  0001 C CNN
+F 3 "" H 5200 2350 50  0001 C CNN
+	1    5200 2350
+	1    0    0    -1
+$EndComp
+Wire Wire Line
+	5200 2250 5200 2350
+$Comp
+L power:GND #PWR?
+U 1 1 5DB420BD
+P 5700 4000
+F 0 "#PWR?" H 5700 3750 50  0001 C CNN
+F 1 "GND" H 5705 3827 50  0000 C CNN
+F 2 "" H 5700 4000 50  0001 C CNN
+F 3 "" H 5700 4000 50  0001 C CNN
+	1    5700 4000
+	1    0    0    -1
+$EndComp
+Wire Wire Line
+	5700 4000 5700 3900
+$Comp
+L power:GND #PWR?
+U 1 1 5DB4256C
+P 4900 4000
+F 0 "#PWR?" H 4900 3750 50  0001 C CNN
+F 1 "GND" H 4905 3827 50  0000 C CNN
+F 2 "" H 4900 4000 50  0001 C CNN
+F 3 "" H 4900 4000 50  0001 C CNN
+	1    4900 4000
+	1    0    0    -1
+$EndComp
+Wire Wire Line
+	5000 3500 4900 3500
+Wire Wire Line
+	5000 3400 4900 3400
+Wire Wire Line
+	4900 3400 4900 3500
+Connection ~ 4900 3500
+Text HLabel 4200 3000 0    50   Input ~ 0
+I2C_SCL
+Text HLabel 4200 2900 0    50   BiDi ~ 0
+I2C_SDA
+Wire Wire Line
+	5000 2900 4200 2900
+Wire Wire Line
+	5000 3000 4200 3000
+$Comp
+L power:+3.3V #PWR?
+U 1 1 5DB43AB6
+P 5600 1850
+F 0 "#PWR?" H 5600 1700 50  0001 C CNN
+F 1 "+3.3V" H 5615 2023 50  0000 C CNN
+F 2 "" H 5600 1850 50  0001 C CNN
+F 3 "" H 5600 1850 50  0001 C CNN
+	1    5600 1850
+	1    0    0    -1
+$EndComp
+Wire Wire Line
+	5600 1850 5600 1900
+Connection ~ 5600 1900
+Wire Wire Line
+	5600 1900 5600 2500
+Wire Wire Line
+	5800 2500 5800 1900
+Wire Wire Line
+	5800 1900 5600 1900
+$Comp
+L Device:C C?
+U 1 1 5DB44A9E
+P 6200 2100
+AR Path="/5BA56FC1/5DB44A9E" Ref="C?"  Part="1"
+AR Path="/5BA57001/5DB44A9E" Ref="C?"  Part="1"
+F 0 "C?" H 6200 2200 39  0000 L CNN
+F 1 "100nF" H 6200 2000 39  0000 L CNN
+F 2 "" H 6238 1950 50  0001 C CNN
+F 3 "~" H 6200 2100 50  0001 C CNN
+	1    6200 2100
+	1    0    0    -1
+$EndComp
+$Comp
+L power:GND #PWR?
+U 1 1 5DB44AE2
+P 6200 2350
+F 0 "#PWR?" H 6200 2100 50  0001 C CNN
+F 1 "GND" H 6205 2177 50  0000 C CNN
+F 2 "" H 6200 2350 50  0001 C CNN
+F 3 "" H 6200 2350 50  0001 C CNN
+	1    6200 2350
+	1    0    0    -1
+$EndComp
+Wire Wire Line
+	6200 2350 6200 2250
+Wire Wire Line
+	6200 1950 6200 1900
+Wire Wire Line
+	6200 1900 5800 1900
+Connection ~ 5800 1900
+Wire Wire Line
+	5600 1900 5200 1900
+Wire Wire Line
+	5200 1900 5200 1950
+Text HLabel 7200 2900 2    50   Output ~ 0
+INT
+Wire Wire Line
+	6400 2900 7200 2900
+Wire Wire Line
+	5000 3100 4900 3100
+Wire Wire Line
+	4900 3100 4900 3400
+Connection ~ 4900 3400
+NoConn ~ 6400 3100
+NoConn ~ 6400 3200
+$Comp
+L Device:C C?
+U 1 1 5DB47214
+P 6500 3750
+AR Path="/5BA56FC1/5DB47214" Ref="C?"  Part="1"
+AR Path="/5BA57001/5DB47214" Ref="C?"  Part="1"
+F 0 "C?" H 6500 3850 39  0000 L CNN
+F 1 "100nF" H 6500 3650 39  0000 L CNN
+F 2 "" H 6538 3600 50  0001 C CNN
+F 3 "~" H 6500 3750 50  0001 C CNN
+	1    6500 3750
+	1    0    0    -1
+$EndComp
+$Comp
+L Device:C C?
+U 1 1 5DB47258
+P 6800 3750
+AR Path="/5BA56FC1/5DB47258" Ref="C?"  Part="1"
+AR Path="/5BA57001/5DB47258" Ref="C?"  Part="1"
+F 0 "C?" H 6800 3850 39  0000 L CNN
+F 1 "2.2nF" H 6800 3650 39  0000 L CNN
+F 2 "" H 6838 3600 50  0001 C CNN
+F 3 "~" H 6800 3750 50  0001 C CNN
+	1    6800 3750
+	1    0    0    -1
+$EndComp
+Wire Wire Line
+	6400 3500 6500 3500
+Wire Wire Line
+	6500 3500 6500 3600
+$Comp
+L power:GND #PWR?
+U 1 1 5DB47429
+P 6500 4000
+F 0 "#PWR?" H 6500 3750 50  0001 C CNN
+F 1 "GND" H 6505 3827 50  0000 C CNN
+F 2 "" H 6500 4000 50  0001 C CNN
+F 3 "" H 6500 4000 50  0001 C CNN
+	1    6500 4000
+	1    0    0    -1
+$EndComp
+Wire Wire Line
+	6500 4000 6500 3900
+Wire Wire Line
+	6400 3400 6800 3400
+Wire Wire Line
+	6800 3400 6800 3600
+$Comp
+L power:GND #PWR?
+U 1 1 5DB47834
+P 6800 4000
+F 0 "#PWR?" H 6800 3750 50  0001 C CNN
+F 1 "GND" H 6805 3827 50  0000 C CNN
+F 2 "" H 6800 4000 50  0001 C CNN
+F 3 "" H 6800 4000 50  0001 C CNN
+	1    6800 4000
+	1    0    0    -1
+$EndComp
+Wire Wire Line
+	6800 4000 6800 3900
+Wire Wire Line
+	4900 3500 4900 4000
+Text Notes 3200 1700 0    79   ~ 16
+Circuito acelerómetro MPU-6050\nProvee datos de:\n> Acelerómetro\n> Giróscopo\n> Temperatura
 $EndSCHEMATC

Commit message: Cambios en sch
Parts:
- gave numbers to parts that had none: 5
Other:
- note added: "Señal de interrupción programable\nsegún eventos (ver Datasheet MPU)"
Changed lines of the file:
@@
 $Descr A4 11693 8268
 encoding utf-8
-Sheet 3 7
+Sheet 3 8
 Title ""
 Date ""
@@
 $EndDescr
 $Comp
-L Sensor_Motion:MPU-6050 U?
+L Sensor_Motion:MPU-6050 U301
 U 1 1 5DB41454
 P 5700 3200
-F 0 "U?" H 5800 2650 50  0000 C CNN
+F 0 "U301" H 5800 2650 50  0000 C CNN
 F 1 "MPU-6050" H 5400 2650 50  0000 C CNN
 F 2 "Sensor_Motion:InvenSense_QFN-24_4x4mm_P0.5mm" H 5700 2400 50  0001 C CNN
@@
 P 5200 2100
 AR Path="/5BA56FC1/5DB41F13" Ref="C?"  Part="1"
-AR Path="/5BA57001/5DB41F13" Ref="C?"  Part="1"
-F 0 "C?" H 5200 2200 39  0000 L CNN
+AR Path="/5BA57001/5DB41F13" Ref="C301"  Part="1"
+F 0 "C301" H 5200 2200 39  0000 L CNN
 F 1 "100nF" H 5200 2000 39  0000 L CNN
 F 2 "" H 5238 1950 50  0001 C CNN
@@
 $EndComp
 $Comp
-L power:GND #PWR?
+L power:GND #PWR0302
 U 1 1 5DB41FBA
 P 5200 2350
-F 0 "#PWR?" H 5200 2100 50  0001 C CNN
+F 0 "#PWR0302" H 5200 2100 50  0001 C CNN
 F 1 "GND" H 5205 2177 50  0000 C CNN
 F 2 "" H 5200 2350 50  0001 C CNN
@@
 	5200 2250 5200 2350
 $Comp
-L power:GND #PWR?
+L power:GND #PWR0304
 U 1 1 5DB420BD
 P 5700 4000
-F 0 "#PWR?" H 5700 3750 50  0001 C CNN
+F 0 "#PWR0304" H 5700 3750 50  0001 C CNN
 F 1 "GND" H 5705 3827 50  0000 C CNN
 F 2 "" H 5700 4000 50  0001 C CNN
@@
 	5700 4000 5700 3900
 $Comp
-L power:GND #PWR?
+L power:GND #PWR0301
 U 1 1 5DB4256C
 P 4900 4000
-F 0 "#PWR?" H 4900 3750 50  0001 C CNN
+F 0 "#PWR0301" H 4900 3750 50  0001 C CNN
 F 1 "GND" H 4905 3827 50  0000 C CNN
 F 2 "" H 4900 4000 50  0001 C CNN
@@
 	5000 3000 4200 3000
 $Comp
-L power:+3.3V #PWR?
+L power:+3.3V #PWR0303
 U 1 1 5DB43AB6
 P 5600 1850
-F 0 "#PWR?" H 5600 1700 50  0001 C CNN
+F 0 "#PWR0303" H 5600 1700 50  0001 C CNN
 F 1 "+3.3V" H 5615 2023 50  0000 C CNN
 F 2 "" H 5600 1850 50  0001 C CNN
@@
 P 6200 2100
 AR Path="/5BA56FC1/5DB44A9E" Ref="C?"  Part="1"
-AR Path="/5BA57001/5DB44A9E" Ref="C?"  Part="1"
-F 0 "C?" H 6200 2200 39  0000 L CNN
+AR Path="/5BA57001/5DB44A9E" Ref="C302"  Part="1"
+F 0 "C302" H 6200 2200 39  0000 L CNN
 F 1 "100nF" H 6200 2000 39  0000 L CNN
 F 2 "" H 6238 1950 50  0001 C CNN
@@
 $EndComp
 $Comp
-L power:GND #PWR?
+L power:GND #PWR0305
 U 1 1 5DB44AE2
 P 6200 2350
-F 0 "#PWR?" H 6200 2100 50  0001 C CNN
+F 0 "#PWR0305" H 6200 2100 50  0001 C CNN
 F 1 "GND" H 6205 2177 50  0000 C CNN
 F 2 "" H 6200 2350 50  0001 C CNN
@@
 P 6500 3750
 AR Path="/5BA56FC1/5DB47214" Ref="C?"  Part="1"
-AR Path="/5BA57001/5DB47214" Ref="C?"  Part="1"
-F 0 "C?" H 6500 3850 39  0000 L CNN
+AR Path="/5BA57001/5DB47214" Ref="C303"  Part="1"
+F 0 "C303" H 6500 3850 39  0000 L CNN
 F 1 "100nF" H 6500 3650 39  0000 L CNN
 F 2 "" H 6538 3600 50  0001 C CNN
@@
 P 6800 3750
 AR Path="/5BA56FC1/5DB47258" Ref="C?"  Part="1"
-AR Path="/5BA57001/5DB47258" Ref="C?"  Part="1"
-F 0 "C?" H 6800 3850 39  0000 L CNN
+AR Path="/5BA57001/5DB47258" Ref="C304"  Part="1"
+F 0 "C304" H 6800 3850 39  0000 L CNN
 F 1 "2.2nF" H 6800 3650 39  0000 L CNN
 F 2 "" H 6838 3600 50  0001 C CNN
@@
 	6500 3500 6500 3600
 $Comp
-L power:GND #PWR?
+L power:GND #PWR0306
 U 1 1 5DB47429
 P 6500 4000
-F 0 "#PWR?" H 6500 3750 50  0001 C CNN
+F 0 "#PWR0306" H 6500 3750 50  0001 C CNN
 F 1 "GND" H 6505 3827 50  0000 C CNN
 F 2 "" H 6500 4000 50  0001 C CNN
@@
 	6800 3400 6800 3600
 $Comp
-L power:GND #PWR?
+L power:GND #PWR0307
 U 1 1 5DB47834
 P 6800 4000
-F 0 "#PWR?" H 6800 3750 50  0001 C CNN
+F 0 "#PWR0307" H 6800 3750 50  0001 C CNN
 F 1 "GND" H 6805 3827 50  0000 C CNN
 F 2 "" H 6800 4000 50  0001 C CNN
@@
 Text Notes 3200 1700 0    79   ~ 16
 Circuito acelerómetro MPU-6050\nProvee datos de:\n> Acelerómetro\n> Giróscopo\n> Temperatura
+Text Notes 7550 2900 0    59   ~ 0
+Señal de interrupción programable\nsegún eventos (ver Datasheet MPU)
+Wire Notes Line
+	7450 2900 9150 2900
 $EndSCHEMATC

Commit message: Cambios en sch
Parts:
- C301, C302, C303, C304: footprint (none) -> Capacitor_SMD:C_0805_2012Metric_Pad1.15x1.40mm_HandSolder
Changed lines of the file:
@@
 encoding utf-8
 Sheet 3 8
-Title ""
-Date ""
-Rev ""
+Title "Equipo AVL - vRaptor"
+Date "2018-10-30"
+Rev "1.0"
 Comp ""
-Comment1 ""
+Comment1 "Ing. Mauro Moreyra"
 Comment2 ""
 Comment3 ""
@@
 F 0 "C301" H 5200 2200 39  0000 L CNN
 F 1 "100nF" H 5200 2000 39  0000 L CNN
-F 2 "" H 5238 1950 50  0001 C CNN
+F 2 "Capacitor_SMD:C_0805_2012Metric_Pad1.15x1.40mm_HandSolder" H 5238 1950 50  0001 C CNN
 F 3 "~" H 5200 2100 50  0001 C CNN
 	1    5200 2100
@@
 F 0 "C302" H 6200 2200 39  0000 L CNN
 F 1 "100nF" H 6200 2000 39  0000 L CNN
-F 2 "" H 6238 1950 50  0001 C CNN
+F 2 "Capacitor_SMD:C_0805_2012Metric_Pad1.15x1.40mm_HandSolder" H 6238 1950 50  0001 C CNN
 F 3 "~" H 6200 2100 50  0001 C CNN
 	1    6200 2100
@@
 F 0 "C303" H 6500 3850 39  0000 L CNN
 F 1 "100nF" H 6500 3650 39  0000 L CNN
-F 2 "" H 6538 3600 50  0001 C CNN
+F 2 "Capacitor_SMD:C_0805_2012Metric_Pad1.15x1.40mm_HandSolder" H 6538 3600 50  0001 C CNN
 F 3 "~" H 6500 3750 50  0001 C CNN
 	1    6500 3750
@@
 F 0 "C304" H 6800 3850 39  0000 L CNN
 F 1 "2.2nF" H 6800 3650 39  0000 L CNN
-F 2 "" H 6838 3600 50  0001 C CNN
+F 2 "Capacitor_SMD:C_0805_2012Metric_Pad1.15x1.40mm_HandSolder" H 6838 3600 50  0001 C CNN
 F 3 "~" H 6800 3750 50  0001 C CNN
 	1    6800 3750

Commit message: Cambios menores en archivos
Parts:
- U301: footprint Sensor_Motion:InvenSense_QFN-24_4x4mm_P0.5mm -> Sensor_Motion:InvenSense_QFN-24_4x4mm_P0.5mm_HandSoldering
Changed lines of the file:
@@
 F 0 "U301" H 5800 2650 50  0000 C CNN
 F 1 "MPU-6050" H 5400 2650 50  0000 C CNN
-F 2 "Sensor_Motion:InvenSense_QFN-24_4x4mm_P0.5mm" H 5700 2400 50  0001 C CNN
+F 2 "Sensor_Motion:InvenSense_QFN-24_4x4mm_P0.5mm_HandSoldering" H 5700 2400 50  0001 C CNN
 F 3 "https://store.invensense.com/datasheets/invensense/MPU-6050_DataSheet_V3%204.pdf" H 5700 3050 50  0001 C CNN
 	1    5700 3200

Commit message: Generación de archivos gerber, drills, bom
Parts:
- added J301: Conn_01x08, Connector_PinHeader_2.54mm:PinHeader_1x08_P2.54mm_Vertical, symbol Connector_Generic:Conn_01x08
Connections:
- net +3V3: now also J301.1 (Pin_1)
- net GND: now also J301.2 (Pin_2), J301.7 (Pin_7)
- net I2C_SCL: now also J301.4 (Pin_4)
- net I2C_SDA: now also J301.3 (Pin_3)
- net INT: now also J301.8 (Pin_8)
- no-connect marks 2 -> 4
Other:
- note added: "Conector backup para PCB MPU-6050 Arduino"
Changed lines of the file:
@@
 Wire Notes Line
 	7450 2900 9150 2900
+$Comp
+L Connector_Generic:Conn_01x08 J301
+U 1 1 5BEF7FA3
+P 5700 5350
+F 0 "J301" H 5780 5342 50  0000 L CNN
+F 1 "Conn_01x08" H 5780 5251 50  0000 L CNN
+F 2 "Connector_PinHeader_2.54mm:PinHeader_1x08_P2.54mm_Vertical" H 5700 5350 50  0001 C CNN
+F 3 "~" H 5700 5350 50  0001 C CNN
+	1    5700 5350
+	1    0    0    -1
+$EndComp
+Text Notes 4300 4650 0    79   ~ 16
+Conector backup para PCB MPU-6050 Arduino
+$Comp
+L power:+3.3V #PWR0101
+U 1 1 5BEF90AF
+P 5400 4950
+F 0 "#PWR0101" H 5400 4800 50  0001 C CNN
+F 1 "+3.3V" H 5415 5123 50  0000 C CNN
+F 2 "" H 5400 4950 50  0001 C CNN
+F 3 "" H 5400 4950 50  0001 C CNN
+	1    5400 4950
+	1    0    0    -1
+$EndComp
+Wire Wire Line
+	5500 5050 5400 5050
+Wire Wire Line
+	5400 5050 5400 4950
+Text Label 4400 2900 0    50   ~ 0
+MPU_SCL
+Text Label 4400 3000 0    50   ~ 0
+MPU_SDA
+Text Label 4950 5250 0    50   ~ 0
+MPU_SCL
+Text Label 4950 5350 0    50   ~ 0
+MPU_SDA
+NoConn ~ 5500 5450
+NoConn ~ 5500 5550
+$Comp
+L power:GND #PWR0104
+U 1 1 5BEFD24B
+P 5400 5850
+F 0 "#PWR0104" H 5400 5600 50  0001 C CNN
+F 1 "GND" H 5405 5677 50  0000 C CNN
+F 2 "" H 5400 5850 50  0001 C CNN
+F 3 "" H 5400 5850 50  0001 C CNN
+	1    5400 5850
+	1    0    0    -1
+$EndComp
+Wire Wire Line
+	4950 5250 5500 5250
+Wire Wire Line
+	4950 5350 5500 5350
+Wire Wire Line
+	5500 5150 5400 5150
+Wire Wire Line
+	5400 5150 5400 5650
+Wire Wire Line
+	5500 5650 5400 5650
+Connection ~ 5400 5650
+Wire Wire Line
+	5400 5650 5400 5850
+Text Label 6600 2900 0    50   ~ 0
+MPU_INT
+Text Label 4950 5750 0    50   ~ 0
+MPU_INT
+Wire Wire Line
+	5500 5750 4950 5750
 $EndSCHEMATC
