File: TrackerAVL/io_ad.sch (KiCad schematic (older format))
At the start: 28 parts, among them Q801 2N7002P, Q802 2N7002P, Q803 2N7002P, Q804 DTC043ZEBTL

Commit message: Cambios en sch
Parts:
- added U701: 74HC244, symbol 74xx:74HC244
- renumbered C802 to C701, C805 to C702, C806 to C703, C807 to C704, C808 to C705, C809 to C706, D804 to D701, D805 to D702, D806 to D703, D807 to D704, D808 to D705, D809 to D706, D803 to D707, D810 to D708, D811 to D709, D812 to D710, Q801 to Q701, Q802 to Q702, Q803 to Q703, Q804 to Q704, R802 to R701, R803 to R702, R804 to R703, R805 to R704, R806 to R705, R807 to R706, R808 to R707, R809 to R708
Connections:
- net GND: now also U701.10 (GND)
- net in_DIG_IN_0: now also U701.18 (1Y0), U701.2 (1A0)
- net in_DIG_IN_1: now also U701.16 (1Y1), U701.4 (1A1)
- net in_DIG_IN_2: now also U701.14 (1Y2), U701.6 (1A2)
- new net +3V3: U701.20 (VCC)
- new net BUFFER_OE: U701.1 (1OE), U701.19 (2OE)
- new net in_TEC_0: U701.17 (2A0)
- new net in_TEC_1: U701.15 (2A1)
- new net in_TEC_2: U701.13 (2A2)
- new net in_TEC_3: U701.11 (2A3)
- new net out_TEC_0: U701.3 (2Y0)
- new net out_TEC_1: U701.5 (2Y1)
- new net out_TEC_2: U701.7 (2Y2)
- new net out_TEC_3: U701.9 (2Y3)
Other:
- note added: "Buffer de protección de IO"
- note added: "NM"
- moved on the sheet: D707, Q704, R704, R705

Commit message: Cambios en sch
Connections:
- no-connect marks 0 -> 2
Changed lines of the file:
@@
 Wire Wire Line
 	3800 6500 3500 6500
+NoConn ~ 2500 6100
+NoConn ~ 3500 6100
 $EndSCHEMATC

Commit message: Cambios en sch
Parts:
- C701, C702, C703, C704, C705, C706: footprint (none) -> Capacitor_SMD:C_0805_2012Metric_Pad1.15x1.40mm_HandSolder
- D704, D705, D706, D707, D708, D709, D710: footprint Diode_THT:D_DO-201AE_P15.24mm_Horizontal -> Diode_SMD:D_SOD-323_HandSoldering
- Q701, Q702, Q703: footprint Package_TO_SOT_SMD:SOT-23 -> Package_TO_SOT_SMD:SOT-23_Handsoldering
- R701, R702, R703, R704, R705, R706, R707, R708: footprint (none) -> Resistor_SMD:R_0805_2012Metric_Pad1.15x1.40mm_HandSolder
- U701: value 74HC244 -> 74LVC244APW; footprint (none) -> Package_SO:TSSOP-20_4.4x6.5mm_P0.65mm
Changed lines of the file:
@@
 encoding utf-8
 Sheet 7 8
-Title ""
-Date ""
-Rev ""
+Title "Equipo AVL - vRaptor"
+Date "2018-10-30"
+Rev "1.0"
 Comp ""
-Comment1 ""
+Comment1 "Ing. Mauro Moreyra"
 Comment2 ""
 Comment3 ""
@@
 F 0 "R701" V 2600 1950 50  0000 L CNN
 F 1 "10K" V 2500 1950 50  0000 L CNN
-F 2 "" V 2430 2050 50  0001 C CNN
+F 2 "Resistor_SMD:R_0805_2012Metric_Pad1.15x1.40mm_HandSolder" V 2430 2050 50  0001 C CNN
 F 3 "~" H 2500 2050 50  0001 C CNN
 	1    2500 2050
@@
 F 0 "Q701" H 3005 1846 50  0000 L CNN
 F 1 "2N7002P" H 3005 1755 50  0000 L CNN
-F 2 "Package_TO_SOT_SMD:SOT-23" H 3000 1725 50  0001 L CIN
+F 2 "Package_TO_SOT_SMD:SOT-23_Handsoldering" H 3000 1725 50  0001 L CIN
 F 3 "https://www.fairchildsemi.com/datasheets/2N/2N7002.pdf" H 2800 1800 50  0001 L CNN
 	1    2800 1800
@@
 F 0 "R702" V 2600 2950 50  0000 L CNN
 F 1 "10K" V 2500 2950 50  0000 L CNN
-F 2 "" V 2430 3050 50  0001 C CNN
+F 2 "Resistor_SMD:R_0805_2012Metric_Pad1.15x1.40mm_HandSolder" V 2430 3050 50  0001 C CNN
 F 3 "~" H 2500 3050 50  0001 C CNN
 	1    2500 3050
@@
 F 0 "Q702" H 3005 2846 50  0000 L CNN
 F 1 "2N7002P" H 3005 2755 50  0000 L CNN
-F 2 "Package_TO_SOT_SMD:SOT-23" H 3000 2725 50  0001 L CIN
+F 2 "Package_TO_SOT_SMD:SOT-23_Handsoldering" H 3000 2725 50  0001 L CIN
 F 3 "https://www.fairchildsemi.com/datasheets/2N/2N7002.pdf" H 2800 2800 50  0001 L CNN
 	1    2800 2800
@@
 F 0 "R703" V 2600 3950 50  0000 L CNN
 F 1 "10K" V 2500 3950 50  0000 L CNN
-F 2 "" V 2430 4050 50  0001 C CNN
+F 2 "Resistor_SMD:R_0805_2012Metric_Pad1.15x1.40mm_HandSolder" V 2430 4050 50  0001 C CNN
 F 3 "~" H 2500 4050 50  0001 C CNN
 	1    2500 4050
@@
 F 0 "Q703" H 3005 3846 50  0000 L CNN
 F 1 "2N7002P" H 3005 3755 50  0000 L CNN
-F 2 "Package_TO_SOT_SMD:SOT-23" H 3000 3725 50  0001 L CIN
+F 2 "Package_TO_SOT_SMD:SOT-23_Handsoldering" H 3000 3725 50  0001 L CIN
 F 3 "https://www.fairchildsemi.com/datasheets/2N/2N7002.pdf" H 2800 3800 50  0001 L CNN
 	1    2800 3800
@@
 F 0 "D704" V 5654 2129 50  0000 L CNN
 F 1 "PESD5V0L1UA" V 5745 2129 50  0000 L CNN
-F 2 "Diode_THT:D_DO-201AE_P15.24mm_Horizontal" H 5700 1850 50  0001 C CNN
+F 2 "Diode_SMD:D_SOD-323_HandSoldering" H 5700 1850 50  0001 C CNN
 F 3 "https://www.vishay.com/docs/88301/15ke.pdf" H 5650 2050 50  0001 C CNN
 	1    5700 2050
@@
 F 0 "C701" H 6515 2096 50  0000 L CNN
 F 1 "100nF" H 6515 2005 50  0000 L CNN
-F 2 "" H 6438 1900 50  0001 C CNN
+F 2 "Capacitor_SMD:C_0805_2012Metric_Pad1.15x1.40mm_HandSolder" H 6438 1900 50  0001 C CNN
 F 3 "~" H 6400 2050 50  0001 C CNN
 	1    6400 2050
@@
 F 0 "D705" V 5654 3129 50  0000 L CNN
 F 1 "PESD5V0L1UA" V 5745 3129 50  0000 L CNN
-F 2 "Diode_THT:D_DO-201AE_P15.24mm_Horizontal" H 5700 2850 50  0001 C CNN
+F 2 "Diode_SMD:D_SOD-323_HandSoldering" H 5700 2850 50  0001 C CNN
 F 3 "https://www.vishay.com/docs/88301/15ke.pdf" H 5650 3050 50  0001 C CNN
 	1    5700 3050
@@
 F 0 "C702" H 6515 3096 50  0000 L CNN
 F 1 "100nF" H 6515 3005 50  0000 L CNN
-F 2 "" H 6438 2900 50  0001 C CNN
+F 2 "Capacitor_SMD:C_0805_2012Metric_Pad1.15x1.40mm_HandSolder" H 6438 2900 50  0001 C CNN
 F 3 "~" H 6400 3050 50  0001 C CNN
 	1    6400 3050
@@
 F 0 "D706" V 5654 4129 50  0000 L CNN
 F 1 "PESD5V0L1UA" V 5745 4129 50  0000 L CNN
-F 2 "Diode_THT:D_DO-201AE_P15.24mm_Horizontal" H 5700 3850 50  0001 C CNN
+F 2 "Diode_SMD:D_SOD-323_HandSoldering" H 5700 3850 50  0001 C CNN
 F 3 "https://www.vishay.com/docs/88301/15ke.pdf" H 5650 4050 50  0001 C CNN
 	1    5700 4050
@@
 F 0 "C703" H 6515 4096 50  0000 L CNN
 F 1 "100nF" H 6515 4005 50  0000 L CNN
-F 2 "" H 6438 3900 50  0001 C CNN
+F 2 "Capacitor_SMD:C_0805_2012Metric_Pad1.15x1.40mm_HandSolder" H 6438 3900 50  0001 C CNN
 F 3 "~" H 6400 4050 50  0001 C CNN
 	1    6400 4050
@@
 F 0 "D708" V 8850 1800 50  0000 L CNN
 F 1 "PESD5V0L1UA" V 8950 1450 50  0000 L CNN
-F 2 "Diode_THT:D_DO-201AE_P15.24mm_Horizontal" H 8900 1850 50  0001 C CNN
+F 2 "Diode_SMD:D_SOD-323_HandSoldering" H 8900 1850 50  0001 C CNN
 F 3 "https://www.vishay.com/docs/88301/15ke.pdf" H 8850 2050 50  0001 C CNN
 	1    8900 2050
@@
 F 0 "C704" H 9315 2096 50  0000 L CNN
 F 1 "100nF" H 9315 2005 50  0000 L CNN
-F 2 "" H 9238 1900 50  0001 C CNN
+F 2 "Capacitor_SMD:C_0805_2012Metric_Pad1.15x1.40mm_HandSolder" H 9238 1900 50  0001 C CNN
 F 3 "~" H 9200 2050 50  0001 C CNN
 	1    9200 2050
@@
 F 0 "R706" V 8700 1700 50  0000 L CNN
 F 1 "1K2" V 8600 1700 50  0000 L CNN
-F 2 "" V 8530 1800 50  0001 C CNN
+F 2 "Resistor_SMD:R_0805_2012Metric_Pad1.15x1.40mm_HandSolder" V 8530 1800 50  0001 C CNN
 F 3 "~" H 8600 1800 50  0001 C CNN
 	1    8600 1800
@@
 F 0 "D709" V 8850 2800 50  0000 L CNN
 F 1 "PESD5V0L1UA" V 8950 2450 50  0000 L CNN
-F 2 "Diode_THT:D_DO-201AE_P15.24mm_Horizontal" H 8900 2850 50  0001 C CNN
+F 2 "Diode_SMD:D_SOD-323_HandSoldering" H 8900 2850 50  0001 C CNN
 F 3 "https://www.vishay.com/docs/88301/15ke.pdf" H 8850 3050 50  0001 C CNN
 	1    8900 3050
@@
 F 0 "C705" H 9315 3096 50  0000 L CNN
 F 1 "100nF" H 9315 3005 50  0000 L CNN
-F 2 "" H 9238 2900 50  0001 C CNN
+F 2 "Capacitor_SMD:C_0805_2012Metric_Pad1.15x1.40mm_HandSolder" H 9238 2900 50  0001 C CNN
 F 3 "~" H 9200 3050 50  0001 C CNN
 	1    9200 3050
@@
 F 0 "R707" V 8700 2700 50  0000 L CNN
 F 1 "1K2" V 8600 2700 50  0000 L CNN
-F 2 "" V 8530 2800 50  0001 C CNN
+F 2 "Resistor_SMD:R_0805_2012Metric_Pad1.15x1.40mm_HandSolder" V 8530 2800 50  0001 C CNN
 F 3 "~" H 8600 2800 50  0001 C CNN
 	1    8600 2800
@@
 F 0 "D710" V 8850 3800 50  0000 L CNN
 F 1 "PESD5V0L1UA" V 8950 3450 50  0000 L CNN
-F 2 "Diode_THT:D_DO-201AE_P15.24mm_Horizontal" H 8900 3850 50  0001 C CNN
+F 2 "Diode_SMD:D_SOD-323_HandSoldering" H 8900 3850 50  0001 C CNN
 F 3 "https://www.vishay.com/docs/88301/15ke.pdf" H 8850 4050 50  0001 C CNN
 	1    8900 4050
@@
 F 0 "C706" H 9315 4096 50  0000 L CNN
 F 1 "100nF" H 9315 4005 50  0000 L CNN
-F 2 "" H 9238 3900 50  0001 C CNN
+F 2 "Capacitor_SMD:C_0805_2012Metric_Pad1.15x1.40mm_HandSolder" H 9238 3900 50  0001 C CNN
 F 3 "~" H 9200 4050 50  0001 C CNN
 	1    9200 4050
@@
 F 0 "R708" V 8700 3700 50  0000 L CNN
 F 1 "1K2" V 8600 3700 50  0000 L CNN
-F 2 "" V 8530 3800 50  0001 C CNN
+F 2 "Resistor_SMD:R_0805_2012Metric_Pad1.15x1.40mm_HandSolder" V 8530 3800 50  0001 C CNN
 F 3 "~" H 8600 3800 50  0001 C CNN
 	1    8600 3800
@@
 F 0 "R704" V 6100 5350 50  0000 L CNN
 F 1 "10K 1%" V 5900 5350 50  0000 L CNN
-F 2 "" V 5930 5450 50  0001 C CNN
+F 2 "Resistor_SMD:R_0805_2012Metric_Pad1.15x1.40mm_HandSolder" V 5930 5450 50  0001 C CNN
 F 3 "~" H 6000 5450 50  0001 C CNN
 	1    6000 5450
@@
 F 0 "R705" V 6100 5750 50  0000 L CNN
 F 1 "1210 1%" V 5900 5700 50  0000 L CNN
-F 2 "" V 5930 5850 50  0001 C CNN
+F 2 "Resistor_SMD:R_0805_2012Metric_Pad1.15x1.40mm_HandSolder" V 5930 5850 50  0001 C CNN
 F 3 "~" H 6000 5850 50  0001 C CNN
 	1    6000 5850
@@
 F 0 "D707" V 6404 5929 50  0000 L CNN
 F 1 "PESD5V0L1UA" V 6495 5929 50  0000 L CNN
-F 2 "Diode_THT:D_DO-201AE_P15.24mm_Horizontal" H 6450 5650 50  0001 C CNN
+F 2 "Diode_SMD:D_SOD-323_HandSoldering" H 6450 5650 50  0001 C CNN
 F 3 "https://www.vishay.com/docs/88301/15ke.pdf" H 6400 5850 50  0001 C CNN
 	1    6450 5850
@@
 P 3000 6300
 F 0 "U701" H 3100 7050 50  0000 C CNN
-F 1 "74HC244" H 3200 6950 50  0000 C CNN
-F 2 "" H 3000 6300 50  0001 C CNN
+F 1 "74LVC244APW" H 3300 6950 50  0000 C CNN
+F 2 "Package_SO:TSSOP-20_4.4x6.5mm_P0.65mm" H 3000 6300 50  0001 C CNN
 F 3 "http://www.nxp.com/documents/data_sheet/74HC_HCT244.pdf" H 3000 6300 50  0001 C CNN
 	1    3000 6300

Commit message: EquipoAVL-vRaptor1.0 sch-finalizado
Parts:
- Q704: footprint (none) -> EquipoAVL:SOT-523_(SOT-416)
Changed lines of the file:
@@
 F 0 "Q704" H 9087 5646 50  0000 L CNN
 F 1 "DTC043ZEBTL" H 9087 5555 50  0000 L CNN
-F 2 "" H 8900 5600 50  0001 L CNN
+F 2 "EquipoAVL:SOT-523_(SOT-416)" H 8900 5600 50  0001 L CNN
 F 3 "" H 8900 5600 50  0001 L CNN
 	1    8900 5600

Commit message: Cambios en pcb
Connections:
- net in_DIG_IN_0: no longer C701.1, D704.1 (A1), U701.18 (1Y0)
- net in_DIG_IN_1: no longer C702.1, D705.1 (A1), U701.16 (1Y1)
- net in_DIG_IN_2: no longer C703.1, D706.1 (A1), U701.14 (1Y2)
- new net out_DIG_IN_0: C701.1, D704.1 (A1), U701.18 (1Y0)
- new net out_DIG_IN_1: C702.1, D705.1 (A1), U701.16 (1Y1)
- new net out_DIG_IN_2: C703.1, D706.1 (A1), U701.14 (1Y2)
Changed lines of the file:
@@
 	2200 6000 2500 6000
 Text Label 4000 5800 2    50   ~ 0
-in_DIG_IN_0
+in_DIG_IN_0_a
 Wire Wire Line
 	3500 5800 4000 5800
@@
 	3500 6000 4000 6000
 Text Label 4000 5900 2    50   ~ 0
-in_DIG_IN_1
+in_DIG_IN_1_b
 Text Label 4000 6000 2    50   ~ 0
-in_DIG_IN_2
+in_DIG_IN_2_c
 Text Label 5150 1800 0    50   ~ 0
-in_DIG_IN_0
+in_DIG_IN_0_a
 Wire Wire Line
 	5150 1800 5700 1800
 Text Label 5150 2800 0    50   ~ 0
-in_DIG_IN_1
+in_DIG_IN_1_b
 Wire Notes Line
 	5050 2250 5650 2250
@@
 	5150 3800 5700 3800
 Text Label 5150 3800 0    50   ~ 0
-in_DIG_IN_2
+in_DIG_IN_2_c
 Text Notes 5450 4100 0    59   ~ 12
 NM
